File: pcbs/amp ctrl/amp ctrl.kicad_sch (KiCad schematic)
At the start: 59 parts

Commit message: Schematic file fix, misc. PCB
Fixed issue with KiCAD's automatic V5→V6 migration (corrected in 6.0.11) that caused problems with component references in multi-channel schematic sheets
Finished migration in amp ctrl PCB, inc. re-assigning "exclude from BOM" attributes to testpoints, solder jumpers
Added mounting hole to amp ctrl PCB for addl support to Ethernet jacks, power connector through stiffener
Parts:
- added H13: #4/M3, MountingHole:MountingHole_3.2mm_M3_Pad_Via, symbol Mechanical:MountingHole_Pad
- H1, H2, H3, H4, H7, H8, JP74, JP75, JP77, JP78, JP79, JP80, TP1, TP19: renamed from ?; now left out of the parts list
- H10, H11, H12, H5, H6, H9: now left out of the parts list
- gave numbers to parts that had none: 39
Connections:
- net GND: now also H13.1
Other:
- moved on the sheet: H10, H11, H12, H5, H6, H9

Commit message: Misc. mfg
Marked top-side testpoints on amp control board as DNP
Updated serial interface board's BOM-placement-help file
Exported stiffener file for amp control board
Parts:
- TP13, TP3, TP33, TP4, TP5: DNP (none) -> DNP
Changed lines of the file:
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@@
+      (effects (font (size 1.27 1.27)) hide)
+    )
+    (property "DNP" "DNP" (id 7) (at 67.31 74.93 0)
       (effects (font (size 1.27 1.27)) hide)
     )
@@
       (effects (font (size 1.27 1.27)) hide)
     )
+    (property "DNP" "DNP" (id 7) (at 40.64 217.17 0)
+      (effects (font (size 1.27 1.27)) hide)
+    )
     (pin "1")
   )
@@
       (effects (font (size 1.27 1.27)) hide)
     )
+    (property "DNP" "DNP" (id 7) (at 49.53 217.17 0)
+      (effects (font (size 1.27 1.27)) hide)
+    )
     (pin "1")
   )
@@
     )
     (property "Part Number" "5019" (id 6) (at 58.42 217.17 0)
+      (effects (font (size 1.27 1.27)) hide)
+    )
+    (property "DNP" "DNP" (id 7) (at 58.42 217.17 0)
       (effects (font (size 1.27 1.27)) hide)
     )
@@
       (effects (font (size 1.27 1.27)) hide)
     )
+    (property "DNP" "DNP" (id 7) (at 68.58 149.86 0)
+      (effects (font (size 1.27 1.27)) hide)
+    )
