File: pcbs/amp ctrl/amp ctrl.kicad_sch (KiCad schematic)
At the start: 60 parts, among them J1 Conn_02x25_Odd_Even, J13 Conn_02x02, J4 Conn_01x02, U10 ADA4004-1, U70 MCP1754ST-3302

Commit message: Moved all project-specific symbols & footprints into new "shim" libraries Updated projects to reference the new "shim" library
Parts:
- D1, D3, D4: footprint Martinos:LED_Kingbright_APA3010_3x2mm_Horizontal -> shim:LED_Kingbright_APA3010_3x2mm_Horizontal
- D2: footprint Martinos_std:D_SMC -> shim:D_SMC
- F1: footprint Martinos:Fuse_12.4x4.5mm_SMT -> shim:Fuse_12.4x4.5mm_SMT
- J1: footprint Martinos_std:PinHeader_2x25_P2.54mm_Vertical_Shrouded -> shim:PinHeader_2x25_P2.54mm_Vertical_Shrouded
- J13: footprint Martinos:PinSocket_2x02_P2.54mm_Vertical_SMD_BotEntry_Pin -> shim:PinSocket_2x02_P2.54mm_Vertical_SMD_BotEntry_Pin
- J4: footprint Martinos:Connector_Combo_Molex_386608802_Phoenix_1792229 -> shim:Connector_Combo_Molex_386608802_Phoenix_1792229
- JP1, JP10, JP11, JP12, JP13, JP14, JP2, JP3, JP4, JP5, JP6, JP7, JP8, JP9: footprint Martinos:Jumper_SMT_Gap-3mm -> shim:Jumper_SMT_Gap-3mm
- TP13, TP3, TP33, TP4, TP5: footprint Don_std:TestPoint_Keystone_5019_Minature -> TestPoint:TestPoint_Keystone_5019_Minature
- U10: footprint Martinos_std:SOT-23-5 -> Package_TO_SOT_SMD:SOT-23-5
- U70: footprint Martinos_std:SOT-23 -> Package_TO_SOT_SMD:SOT-23
Changed lines of the file:
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@@
 			)
 		)
-		(property "Footprint" "Martinos:Connector_Combo_Molex_386608802_Phoenix_1792229"
+		(property "Footprint" "shim:Connector_Combo_Molex_386608802_Phoenix_1792229"
 			(at 34.29 41.91 0)
 			(effects
@@
 			)
 		)
-		(property "Footprint" "Martinos:LED_Kingbright_APA3010_3x2mm_Horizontal"
+		(property "Footprint" "shim:LED_Kingbright_APA3010_3x2mm_Horizontal"
 			(at 55.88 121.92 0)
 			(effects
@@
 			)
 		)
-		(property "Footprint" "Martinos:LED_Kingbright_APA3010_3x2mm_Horizontal"
+		(property "Footprint" "shim:LED_Kingbright_APA3010_3x2mm_Horizontal"
 			(at 39.37 121.92 0)
 			(effects
@@
 			)
 		)
-		(property "Footprint" "Don_std:TestPoint_Keystone_5019_Minature"
+		(property "Footprint" "TestPoint:TestPoint_Keystone_5019_Minature"
 			(at 72.39 74.93 0)
 			(effects
@@
 			)
 		)
-		(property "Footprint" "Don_std:TestPoint_Keystone_5019_Minature"
+		(property "Footprint" "TestPoint:TestPoint_Keystone_5019_Minature"
 			(at 45.72 217.17 0)
 			(effects
@@
 			)
 		)
-		(property "Footprint" "Don_std:TestPoint_Keystone_5019_Minature"
+		(property "Footprint" "TestPoint:TestPoint_Keystone_5019_Minature"
 			(at 54.61 217.17 0)
 			(effects
@@
 			)
 		)
-		(property "Footprint" "Don_std:TestPoint_Keystone_5019_Minature"
+		(property "Footprint" "TestPoint:TestPoint_Keystone_5019_Minature"
 			(at 63.5 217.17 0)
 			(effects
@@
 			)
 		)
-		(property "Footprint" "Martinos_std:SOT-23-5"
+		(property "Footprint" "Package_TO_SOT_SMD:SOT-23-5"
 			(at 365.76 60.96 0)
 			(effects
@@
 			)
 		)
-		(property "Footprint" "Martinos_std:PinHeader_2x25_P2.54mm_Vertical_Shrouded"
+		(property "Footprint" "shim:PinHeader_2x25_P2.54mm_Vertical_Shrouded"
 			(at 331.47 158.75 0)
 			(effects
@@
 			)
 		)
-		(property "Footprint" "Martinos:PinSocket_2x02_P2.54mm_Vertical_SMD_BotEntry_Pin"
+		(property "Footprint" "shim:PinSocket_2x02_P2.54mm_Vertical_SMD_BotEntry_Pin"
 			(at 49.53 74.93 0)
 			(effects
@@
 			)
 		)
-		(property "Footprint" "Martinos:Fuse_12.4x4.5mm_SMT"
+		(property "Footprint" "shim:Fuse_12.4x4.5mm_SMT"
 			(at 45.72 37.592 90)
 			(effects
@@
 			)
 		)
-		(property "Footprint" "Martinos_std:D_SMC"
+		(property "Footprint" "shim:D_SMC"
 			(at 58.42 40.64 0)
 			(effects
@@
 			)
 		)
-		(property "Footprint" "Martinos:Jumper_SMT_Gap-3mm"
+		(property "Footprint" "shim:Jumper_SMT_Gap-3mm"
 			(at 256.54 57.15 0)
 			(effects
@@
 			)
 		)
-		(property "Footprint" "Martinos:Jumper_SMT_Gap-3mm"
+		(property "Footprint" "shim:Jumper_SMT_Gap-3mm"
 			(at 262.89 57.15 0)
 			(effects
@@
 			)
 		)
-		(property "Footprint" "Martinos:Jumper_SMT_Gap-3mm"
+		(property "Footprint" "shim:Jumper_SMT_Gap-3mm"
 			(at 256.54 85.09 0)
 			(effects
@@
 			)
 		)
-		(property "Footprint" "Martinos:Jumper_SMT_Gap-3mm"
+		(property "Footprint" "shim:Jumper_SMT_Gap-3mm"
 			(at 262.89 85.09 0)
 			(effects
@@
 			)
 		)
-		(property "Footprint" "Martinos:Jumper_SMT_Gap-3mm"
+		(property "Footprint" "shim:Jumper_SMT_Gap-3mm"
 			(at 256.54 114.3 0)
 			(effects
@@
 			)
 		)
-		(property "Footprint" "Martinos:Jumper_SMT_Gap-3mm"
+		(property "Footprint" "shim:Jumper_SMT_Gap-3mm"
 			(at 262.89 114.3 0)
 			(effects
@@
 			)
 		)
-		(property "Footprint" "Martinos:Jumper_SMT_Gap-3mm"
+		(property "Footprint" "shim:Jumper_SMT_Gap-3mm"
 			(at 256.54 142.24 0)
 			(effects
@@
 			)
 		)
-		(property "Footprint" "Martinos:Jumper_SMT_Gap-3mm"
+		(property "Footprint" "shim:Jumper_SMT_Gap-3mm"
 			(at 262.89 142.24 0)
 			(effects
@@
 			)
 		)
-		(property "Footprint" "Martinos:Jumper_SMT_Gap-3mm"
+		(property "Footprint" "shim:Jumper_SMT_Gap-3mm"
 			(at 256.54 170.18 0)
 			(effects
@@
 			)
 		)
-		(property "Footprint" "Martinos:Jumper_SMT_Gap-3mm"
+		(property "Footprint" "shim:Jumper_SMT_Gap-3mm"
 			(at 262.89 170.18 0)
 			(effects
@@
 			)
 		)
-		(property "Footprint" "Martinos:Jumper_SMT_Gap-3mm"
+		(property "Footprint" "shim:Jumper_SMT_Gap-3mm"
 			(at 256.54 198.12 0)
 			(effects
@@
 			)
 		)
-		(property "Footprint" "Martinos:Jumper_SMT_Gap-3mm"
+		(property "Footprint" "shim:Jumper_SMT_Gap-3mm"
 			(at 262.89 198.12 0)
 			(effects
@@
 			)
 		)
-		(property "Footprint" "Martinos:Jumper_SMT_Gap-3mm"
+		(property "Footprint" "shim:Jumper_SMT_Gap-3mm"
 			(at 256.54 226.06 0)
 			(effects
@@
 			)
 		)
-		(property "Footprint" "Martinos:Jumper_SMT_Gap-3mm"
+		(property "Footprint" "shim:Jumper_SMT_Gap-3mm"
 			(at 262.89 226.06 0)
 			(effects
@@
 			)
 		)
-		(property "Footprint" "Martinos_std:SOT-23"
+		(property "Footprint" "Package_TO_SOT_SMD:SOT-23"
 			(at 48.26 151.13 0)
 			(effects
@@
 			)
 		)
-		(property "Footprint" "Don_std:TestPoint_Keystone_5019_Minature"
+		(property "Footprint" "TestPoint:TestPoint_Keystone_5019_Minature"
 			(at 73.66 149.86 0)
 			(effects
@@
 			)
 		)
-		(property "Footprint" "Martinos:LED_Kingbright_APA3010_3x2mm_Horizontal"
+		(property "Footprint" "shim:LED_Kingbright_APA3010_3x2mm_Horizontal"
 			(at 71.12 121.92 0)
 			(effects

Commit message: Finished migrating footprint names
Parts:
- TP13, TP3, TP33, TP4, TP5: footprint TestPoint:TestPoint_Keystone_5019_Minature -> TestPoint:TestPoint_Keystone_5019_Miniature
Changed lines of the file:
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@@
 			)
 		)
-		(property "Footprint" "TestPoint:TestPoint_Keystone_5019_Minature"
+		(property "Footprint" "TestPoint:TestPoint_Keystone_5019_Miniature"
 			(at 72.39 74.93 0)
 			(effects
@@
 			)
 		)
-		(property "Footprint" "TestPoint:TestPoint_Keystone_5019_Minature"
+		(property "Footprint" "TestPoint:TestPoint_Keystone_5019_Miniature"
 			(at 45.72 217.17 0)
 			(effects
@@
 			)
 		)
-		(property "Footprint" "TestPoint:TestPoint_Keystone_5019_Minature"
+		(property "Footprint" "TestPoint:TestPoint_Keystone_5019_Miniature"
 			(at 54.61 217.17 0)
 			(effects
@@
 			)
 		)
-		(property "Footprint" "TestPoint:TestPoint_Keystone_5019_Minature"
+		(property "Footprint" "TestPoint:TestPoint_Keystone_5019_Miniature"
 			(at 63.5 217.17 0)
 			(effects
@@
 			)
 		)
-		(property "Footprint" "TestPoint:TestPoint_Keystone_5019_Minature"
+		(property "Footprint" "TestPoint:TestPoint_Keystone_5019_Miniature"
 			(at 73.66 149.86 0)
 			(effects

Commit message: BOM & reset fixes
Amp ctrl: changed name of "Manufacturer" field to "MPN" to work with Aisler
Amp ctrl: added part number to logic inverter, corrected various typos and part number problems
Backplane: added pull-down to Shutdown_Reset signal (#35)
Backplane: rethought Shutdown_Force circuit to make fail-safe (broken connections->shutdown), make work correctly (fixes #35)
Backplane: updated/corrected various schematic annotations
Parts:
- C2: MPN (none) -> GCM32EC71H106KA03L; MPN Alt. (none) -> GRM32EC72A106KE05L; Part Number GCM32EC71H106KA03L -> (none); Part Number Alt. GRM32EC72A106KE05L -> (none)
- C231, C232: MPN (none) -> C0603C105K4RACTU; Part Number C0603C105K4RACTU -> (none)
- C30: MPN (none) -> C0805C105K3RACTU; Part Number C0805C105K3RACTU -> (none)
- D1: MPN (none) -> APA3010SYCK-GX; Part Number APA3010SYCK-GX -> (none)
- D2: MPN (none) -> SMDJ30A; Part Number SMDJ30A -> (none)
- D3, D4: MPN (none) -> APA3010ZGC-GX; Part Number APA3010ZGC-GX -> (none)
- F1: MPN (none) -> 0456040.DR; Part Number 0456040.DR -> (none)
- J1: MPN (none) -> SBH11-PBPC-D25-ST-BK; MPN Alt. (none) -> 30350-6002HB; Part Number SBH11-PBPC-D25-ST-BK -> (none); Part Number Alt. 30350-6002HB -> (none)
- J13: MPN (none) -> M20-7810245 / M20-7810245R; MPN Alt. (none) -> HLE-102-02-L-DV / HLE-102-02-F-DV / HLE-102-02-G-DV / HLE-1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; Part Number M20-7810245 / M20-7810245R -> (none); Part Number Alt. HLE-102-02-L-DV / HLE-102-02-F-DV / HLE-102-02-G-DV / HLE-1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 -> (none)
- JP1, JP10, JP11, JP12, JP13, JP14, JP2, JP3, JP4, JP5, JP6, JP7, JP8, JP9: DNP DNP -> (none); MPN (none) -> 5100TR; Part Number 5100TR -> (none)
- R16, R34, R35: MPN (none) -> RK73H2ATTD1002F; Part Number RK73H2ATTE1002F -> (none)
- R20: MPN (none) -> RK73H2ATTD1001F; Part Number RK73H2ATTDD1001F -> (none)
- R25, R41: MPN (none) -> RK73H2ATTD3301F; Part Number RK73H2ATTD3301F -> (none)
- TP13, TP3, TP33, TP4, TP5: DNP DNP -> (none); MPN (none) -> 5019; Part Number 5019 -> (none)
- U10: MPN (none) -> ADA4004-1ARJZ-R7; MPN Alt. (none) -> ADA4004-1ARJZ-R2; Part Number ADA4004-1ARJZ-R7 -> (none); Part Number Alt. ADA4004-1ARJZ-R2 -> (none)
- U70: MPN (none) -> MCP1754ST-3302E/CB; Part Number MCP1754ST-3302E/CB -> (none)
