File: pcbs/amp ctrl/channel.kicad_sch (KiCad schematic)
At the start: 98 parts, among them J11 Conn_01x02, J6 Conn_02x02, J8 Conn_02x10_Odd_Even, J9 Conn_02x02, J92 Conn_01x02, Q1 MMBT3904, Q2 MMBT3906, Q3 MMBT3904, Q36 MMBT3904, Q37 2N7002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

Commit message: Misc. cleanup for mfg & improvements
Minor backplane pinout doc corrections (SCKO5 polarity, clarified some descriptions)
Backplane: Added differential- and common-mode (to standoffs) power filtering, for EMI escaping over power wiring
Amp ctrl: Changed DAC testpoints from individual pads to Keystone 5019 for easier probing
Corrected part numbers, DNP vs. non-BOM-item indications, other misc. BOM issues
Parts:
- C235, C265, C273, D31, J11, J2, J3, J5, J92, R236, R237, R335, R343, R4, RN5, RN6, U3, U73: now not fitted
- TP18, TP2, TP20, TP52: footprint TestPoint:TestPoint_Keystone_5019_Minature -> Don_std:TestPoint_Keystone_5019_Minature; now not fitted
Changed lines of the file:
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@@
 		(in_bom yes)
 		(on_board yes)
-		(dnp no)
+		(dnp yes)
 		(property "Reference" "U3"
 			(at 167.64 52.07 0)
@@
 		(in_bom yes)
 		(on_board yes)
-		(dnp no)
+		(dnp yes)
 		(property "Reference" "J2"
 			(at 17.78 36.83 0)
@@
 			)
 		)
-		(property "Datasheet" " ~"
+		(property "Datasheet" "~"
 			(at 21.59 36.83 0)
 			(effects
@@
 		(in_bom yes)
 		(on_board yes)
-		(dnp no)
+		(dnp yes)
 		(property "Reference" "J3"
 			(at 96.52 153.67 0)
@@
 			)
 		)
-		(property "Datasheet" " ~"
+		(property "Datasheet" "~"
 			(at 96.52 157.48 0)
 			(effects
@@
 		(in_bom yes)
 		(on_board yes)
-		(dnp no)
+		(dnp yes)
 		(property "Reference" "R4"
 			(at 133.35 152.2222 90)
@@
 		(in_bom yes)
 		(on_board yes)
-		(dnp no)
+		(dnp yes)
 		(property "Reference" "TP2"
 			(at 93.98 72.39 0)
@@
 			)
 		)
-		(property "Footprint" "TestPoint:TestPoint_Keystone_5019_Minature"
+		(property "Footprint" "Don_std:TestPoint_Keystone_5019_Minature"
 			(at 99.06 76.2 0)
 			(effects
@@
 		(in_bom yes)
 		(on_board yes)
-		(dnp no)
+		(dnp yes)
 		(property "Reference" "J5"
 			(at 121.92 125.73 0)
@@
 			)
 		)
-		(property "Datasheet" " ~"
+		(property "Datasheet" "~"
 			(at 121.92 129.54 0)
 			(effects
@@
 		(in_bom yes)
 		(on_board yes)
-		(dnp no)
+		(dnp yes)
 		(property "Reference" "J11"
 			(at 373.38 88.9 90)
@@
 		(in_bom yes)
 		(on_board yes)
-		(dnp no)
+		(dnp yes)
 		(property "Reference" "J92"
 			(at 392.43 100.33 0)
@@
 		(at 118.11 76.2 0)
 		(unit 1)
-		(exclude_from_sim no)
+		(exclude_from_sim yes)
 		(in_bom no)
 		(on_board yes)
@@
 		(at 118.11 68.58 0)
 		(unit 1)
-		(exclude_from_sim no)
+		(exclude_from_sim yes)
 		(in_bom no)
 		(on_board yes)
@@
 		(in_bom yes)
 		(on_board yes)
-		(dnp no)
+		(dnp yes)
 		(property "Reference" "R237"
 			(at 109.22 66.04 90)
@@
 		(in_bom yes)
 		(on_board yes)
-		(dnp no)
+		(dnp yes)
 		(property "Reference" "R236"
 			(at 34.29 46.99 0)
@@
 		(in_bom yes)
 		(on_board yes)
-		(dnp no)
+		(dnp yes)
 		(property "Reference" "C235"
 			(at 140.97 190.5 0)
@@
 		(in_bom yes)
 		(on_board yes)
-		(dnp no)
+		(dnp yes)
 		(property "Reference" "TP18"
 			(at 405.13 209.55 0)
@@
 			)
 		)
-		(property "Footprint" "TestPoint:TestPoint_Keystone_5019_Minature"
+		(property "Footprint" "Don_std:TestPoint_Keystone_5019_Minature"
 			(at 410.21 213.36 0)
 			(effects
@@
 		(in_bom yes)
 		(on_board yes)
-		(dnp no)
+		(dnp yes)
 		(property "Reference" "TP20"
 			(at 405.13 222.25 0)
@@
 			)
 		)
-		(property "Footprint" "TestPoint:TestPoint_Keystone_5019_Minature"
+		(property "Footprint" "Don_std:TestPoint_Keystone_5019_Minature"
 			(at 410.21 226.06 0)
 			(effects
@@
 		(in_bom yes)
 		(on_board yes)
-		(dnp no)
+		(dnp yes)
 		(property "Reference" "TP52"
 			(at 116.84 153.67 0)
@@
 			)
 		)
-		(property "Footprint" "TestPoint:TestPoint_Keystone_5019_Minature"
+		(property "Footprint" "Don_std:TestPoint_Keystone_5019_Minature"
 			(at 111.76 157.48 0)
 			(effects
@@
 		(in_bom yes)
 		(on_board yes)
-		(dnp no)
+		(dnp yes)
 		(property "Reference" "RN5"
 			(at 65.532 49.7586 0)
@@
 		(in_bom yes)
 		(on_board yes)
-		(dnp no)
+		(dnp yes)
 		(property "Reference" "RN6"
 			(at 93.98 60.96 90)
@@
 		(in_bom yes)
 		(on_board yes)
-		(dnp no)
+		(dnp yes)
 		(property "Reference" "U73"
 			(at 55.88 30.48 0)
@@
 		(in_bom yes)
 		(on_board yes)
-		(dnp no)
+		(dnp yes)
 		(property "Reference" "U73"
 			(at 92.71 27.7622 0)
@@
 		(in_bom yes)
 		(on_board yes)
-		(dnp no)
+		(dnp yes)
 		(property "Reference" "U73"
 			(at 114.5032 38.3286 0)
@@
 		(in_bom yes)
 		(on_board yes)
-		(dnp no)
+		(dnp yes)
 		(property "Reference" "C265"
 			(at 119.38 26.67 90)
@@
 		(at 67.31 68.58 0)
 		(unit 1)
-		(exclude_from_sim no)
+		(exclude_from_sim yes)
 		(in_bom no)
 		(on_board yes)
@@
 		(in_bom yes)
 		(on_board yes)
-		(dnp no)
+		(dnp yes)
 		(property "Reference" "R335"
 			(at 41.91 39.37 90)
@@
 		(in_bom yes)
 		(on_board yes)
-		(dnp no)
+		(dnp yes)
 		(property "Reference" "D31"
 			(at 45.72 250.19 90)
@@
 		(in_bom yes)
 		(on_board yes)
-		(dnp no)
+		(dnp yes)
 		(property "Reference" "R343"
 			(at 67.31 44.45 0)
@@
 		(in_bom yes)
 		(on_board yes)
-		(dnp no)
+		(dnp yes)
 		(property "Reference" "C273"
 			(at 93.98 44.45 90)

Commit message: Moved all project-specific symbols & footprints into new "shim" libraries Updated projects to reference the new "shim" library
Parts:
- D31, D32, D33, D34: footprint Don_std:D_SOD-323F -> shim:D_SOD-323F
- D5: footprint Martinos_std:D_SOD-123 -> shim:D_SOD-123
- J6, J9: footprint Martinos:PinSocket_2x02_P2.54mm_Vertical_SMD_BotEntry_Pin -> shim:PinSocket_2x02_P2.54mm_Vertical_SMD_BotEntry_Pin
- J8: footprint Martinos:PinSocket_2x10_P2.54mm_Vertical_SMD_BotEntry_Pin -> shim:PinSocket_2x10_P2.54mm_Vertical_SMD_BotEntry_Pin
- Q1, Q2, Q3, Q36, Q4, U7, U9: footprint Martinos_std:SOT-23 -> Package_TO_SOT_SMD:SOT-23
- Q37: footprint Don_std:SOT-563 -> Package_TO_SOT_SMD:SOT-563
- RN5, RN6: footprint Don_std:R_Array_Convex_2x0606 -> Resistor_SMD:R_Array_Convex_2x0606
- TP18, TP2, TP20, TP52: footprint Don_std:TestPoint_Keystone_5019_Minature -> TestPoint:TestPoint_Keystone_5019_Minature
- TP41, TP8: footprint Martinos:TestPoint_2Pads_Pitch4mm_Drill1mm0.7mm -> shim:TestPoint_2Pads_Pitch4mm_Drill1mm0.7mm
- U1: footprint Don_std:SOIC-8_3.9x4.9mm_P1.27mm -> Package_SO:SOIC-8_3.9x4.9mm_P1.27mm; symbol Don:INA821_INA819 -> shim:INA821_INA819
- U2, U73: footprint Don_std:SOIC-8_3.9x4.9mm_P1.27mm -> Package_SO:SOIC-8_3.9x4.9mm_P1.27mm
- U3: footprint Martinos_std:SOT-23-5 -> Package_TO_SOT_SMD:SOT-23-5
Changed lines of the file:
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@@
 			)
 		)
-		(property "Footprint" "Martinos_std:SOT-23-5"
+		(property "Footprint" "Package_TO_SOT_SMD:SOT-23-5"
 			(at 167.64 59.69 0)
 			(effects
@@
 	)
 	(symbol
-		(lib_id "Don:INA821_INA819")
+		(lib_id "shim:INA821_INA819")
 		(at 156.21 175.26 0)
 		(mirror y)
@@
 			)
 		)
-		(property "Footprint" "Don_std:SOIC-8_3.9x4.9mm_P1.27mm"
+		(property "Footprint" "Package_SO:SOIC-8_3.9x4.9mm_P1.27mm"
 			(at 153.67 175.26 0)
 			(effects
@@
 			)
 		)
-		(property "Footprint" "Martinos:PinSocket_2x02_P2.54mm_Vertical_SMD_BotEntry_Pin"
+		(property "Footprint" "shim:PinSocket_2x02_P2.54mm_Vertical_SMD_BotEntry_Pin"
 			(at 303.53 181.61 0)
 			(effects
@@
 			)
 		)
-		(property "Footprint" "Martinos:PinSocket_2x10_P2.54mm_Vertical_SMD_BotEntry_Pin"
+		(property "Footprint" "shim:PinSocket_2x10_P2.54mm_Vertical_SMD_BotEntry_Pin"
 			(at 303.53 161.29 0)
 			(effects
@@
 			)
 		)
-		(property "Footprint" "Martinos:TestPoint_2Pads_Pitch4mm_Drill1mm0.7mm"
+		(property "Footprint" "shim:TestPoint_2Pads_Pitch4mm_Drill1mm0.7mm"
 			(at 186.69 68.58 0)
 			(effects
@@
 			)
 		)
-		(property "Footprint" "Don_std:TestPoint_Keystone_5019_Minature"
+		(property "Footprint" "TestPoint:TestPoint_Keystone_5019_Minature"
 			(at 99.06 76.2 0)
 			(effects
@@
 			)
 		)
-		(property "Footprint" "Don_std:SOIC-8_3.9x4.9mm_P1.27mm"
+		(property "Footprint" "Package_SO:SOIC-8_3.9x4.9mm_P1.27mm"
 			(at 161.29 78.74 0)
 			(effects
@@
 			)
 		)
-		(property "Footprint" "Martinos:PinSocket_2x02_P2.54mm_Vertical_SMD_BotEntry_Pin"
+		(property "Footprint" "shim:PinSocket_2x02_P2.54mm_Vertical_SMD_BotEntry_Pin"
 			(at 142.24 111.76 0)
 			(effects
@@
 			)
 		)
-		(property "Footprint" "Martinos:TestPoint_2Pads_Pitch4mm_Drill1mm0.7mm"
+		(property "Footprint" "shim:TestPoint_2Pads_Pitch4mm_Drill1mm0.7mm"
 			(at 290.83 68.58 0)
 			(effects
@@
 			)
 		)
-		(property "Footprint" "Martinos_std:SOT-23"
+		(property "Footprint" "Package_TO_SOT_SMD:SOT-23"
 			(at 226.06 75.565 0)
 			(effects
@@
 			)
 		)
-		(property "Footprint" "Martinos_std:SOT-23"
+		(property "Footprint" "Package_TO_SOT_SMD:SOT-23"
 			(at 262.89 75.565 0)
 			(effects
@@
 			)
 		)
-		(property "Footprint" "Martinos_std:SOT-23"
+		(property "Footprint" "Package_TO_SOT_SMD:SOT-23"
 			(at 262.89 81.915 0)
 			(effects
@@
 			)
 		)
-		(property "Footprint" "Martinos_std:SOT-23"
+		(property "Footprint" "Package_TO_SOT_SMD:SOT-23"
 			(at 226.06 81.915 0)
 			(effects
@@
 			)
 		)
-		(property "Footprint" "Martinos_std:SOT-23"
+		(property "Footprint" "Package_TO_SOT_SMD:SOT-23"
 			(at 256.54 60.96 0)
 			(effects
@@
 			)
 		)
-		(property "Footprint" "Martinos_std:SOT-23"
+		(property "Footprint" "Package_TO_SOT_SMD:SOT-23"
 			(at 256.54 96.52 0)
 			(effects
@@
 			)
 		)
-		(property "Footprint" "Martinos_std:D_SOD-123"
+		(property "Footprint" "shim:D_SOD-123"
 			(at 101.6 179.07 0)
 			(effects
@@
 			)
 		)
-		(property "Footprint" "Don_std:TestPoint_Keystone_5019_Minature"
+		(property "Footprint" "TestPoint:TestPoint_Keystone_5019_Minature"
 			(at 410.21 213.36 0)
 			(effects
@@
 			)
 		)
-		(property "Footprint" "Don_std:TestPoint_Keystone_5019_Minature"
+		(property "Footprint" "TestPoint:TestPoint_Keystone_5019_Minature"
 			(at 410.21 226.06 0)
 			(effects
@@
 			)
 		)
-		(property "Footprint" "Don_std:TestPoint_Keystone_5019_Minature"
+		(property "Footprint" "TestPoint:TestPoint_Keystone_5019_Minature"
 			(at 111.76 157.48 0)
 			(effects
@@
 			)
 		)
-		(property "Footprint" "Don_std:SOT-563"
+		(property "Footprint" "Package_TO_SOT_SMD:SOT-563"
 			(at 177.8 228.6 0)
 			(effects
@@
 			)
 		)
-		(property "Footprint" "Don_std:SOT-563"
+		(property "Footprint" "Package_TO_SOT_SMD:SOT-563"
 			(at 157.48 228.6 0)
 			(effects
@@
 			)
 		)
-		(property "Footprint" "Don_std:R_Array_Convex_2x0606"
+		(property "Footprint" "Resistor_SMD:R_Array_Convex_2x0606"
 			(at 56.515 52.07 90)
 			(effects
@@
 			)
 		)
-		(property "Footprint" "Don_std:R_Array_Convex_2x0606"
+		(property "Footprint" "Resistor_SMD:R_Array_Convex_2x0606"
 			(at 93.98 51.435 90)
 			(effects
@@
 			)
 		)
-		(property "Footprint" "Don_std:SOIC-8_3.9x4.9mm_P1.27mm"
+		(property "Footprint" "Package_SO:SOIC-8_3.9x4.9mm_P1.27mm"
 			(at 53.34 39.37 0)
 			(effects
@@
 			)
 		)
-		(property "Footprint" "Don_std:SOIC-8_3.9x4.9mm_P1.27mm"
+		(property "Footprint" "Package_SO:SOIC-8_3.9x4.9mm_P1.27mm"
 			(at 92.71 39.37 0)
 			(effects
@@
 			)
 		)
-		(property "Footprint" "Don_std:SOIC-8_3.9x4.9mm_P1.27mm"
+		(property "Footprint" "Package_SO:SOIC-8_3.9x4.9mm_P1.27mm"
 			(at 115.57 40.64 0)
 			(effects
@@
 			)
 		)
-		(property "Footprint" "Don_std:D_SOD-323F"
+		(property "Footprint" "shim:D_SOD-323F"
 			(at 172.72 214.63 0)
 			(effects
@@
 			)
 		)
-		(property "Footprint" "Martinos_std:SOT-23"
+		(property "Footprint" "Package_TO_SOT_SMD:SOT-23"
 			(at 44.45 236.855 0)
 			(effects
@@
 			)
 		)
-		(property "Footprint" "Don_std:D_SOD-323F"
+		(property "Footprint" "shim:D_SOD-323F"
 			(at 48.26 243.84 0)
 			(effects
@@
 			)
 		)
-		(property "Footprint" "Don_std:D_SOD-323F"
+		(property "Footprint" "shim:D_SOD-323F"
 			(at 41.91 250.19 0)
 			(effects
@@
 			)
 		)
-		(property "Footprint" "Don_std:D_SOD-323F"
+		(property "Footprint" "shim:D_SOD-323F"
 			(at 172.72 222.25 0)
 			(effects

Commit message: Finished migrating footprint names
Parts:
- TP18, TP2, TP20, TP52: footprint TestPoint:TestPoint_Keystone_5019_Minature -> TestPoint:TestPoint_Keystone_5019_Miniature
Changed lines of the file:
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@@
 			)
 		)
-		(property "Footprint" "TestPoint:TestPoint_Keystone_5019_Minature"
+		(property "Footprint" "TestPoint:TestPoint_Keystone_5019_Miniature"
 			(at 99.06 76.2 0)
 			(effects
@@
 			)
 		)
-		(property "Footprint" "TestPoint:TestPoint_Keystone_5019_Minature"
+		(property "Footprint" "TestPoint:TestPoint_Keystone_5019_Miniature"
 			(at 410.21 213.36 0)
 			(effects
@@
 			)
 		)
-		(property "Footprint" "TestPoint:TestPoint_Keystone_5019_Minature"
+		(property "Footprint" "TestPoint:TestPoint_Keystone_5019_Miniature"
 			(at 410.21 226.06 0)
 			(effects
@@
 			)
 		)
-		(property "Footprint" "TestPoint:TestPoint_Keystone_5019_Minature"
+		(property "Footprint" "TestPoint:TestPoint_Keystone_5019_Miniature"
 			(at 111.76 157.48 0)
 			(effects

Commit message: BOM & reset fixes
Amp ctrl: changed name of "Manufacturer" field to "MPN" to work with Aisler
Amp ctrl: added part number to logic inverter, corrected various typos and part number problems
Backplane: added pull-down to Shutdown_Reset signal (#35)
Backplane: rethought Shutdown_Force circuit to make fail-safe (broken connections->shutdown), make work correctly (fixes #35)
Backplane: updated/corrected various schematic annotations
Parts:
- C10, C12, C19, C273, C5, C7, J11, R14, R236, R237, R3, R335, R343, R5, U3, U73: DNP DNP -> (none)
- C11, C21, C23, C3: MPN (none) -> C0603C101J5GACTU; Part Number C0603C101J5GACTU -> (none)
- C13: MPN (none) -> C0603C221J5GACTU; Part Number C0603C221J5GACTU -> (none)
- C16, C215, C216: MPN (none) -> GCM32EC71H106KA03L; MPN Alt. (none) -> GRM32EC72A106KE05L; Part Number GCM32EC71H106KA03L -> (none); Part Number Alt. GRM32EC72A106KE05L -> (none)
- C235: DNP DNP -> (none); MPN (none) -> C0805C475K4RACTU; Part Number C0805C475K4RACTU -> (none)
- C257: DNP DNP -> (none); MPN (none) -> C0603C101J5GACTU; Part Number C0603C101J5GACTU -> (none)
- C265: DNP DNP -> (none); MPN (none) -> C0805C105K3RACTU; Part Number C0805C105K3RACTU -> (none)
- C4: MPN (none) -> C0603C102J5GACTU; Part Number C0603C102J5GACTU -> (none)
- C58: MPN (none) -> C0603C105K4RACTU; Part Number C0603C105K4RACTU -> (none)
- C6, C8: MPN (none) -> C0805C105K3RACTU; Part Number C0805C105K3RACTU -> (none)
- C9: MPN (none) -> C0603C820J5GACTU; Part Number C0603C820J5GACTU -> (none)
- D31: DNP DNP -> (none); MPN (none) -> BAS16J,115 / BAS16J,135; MPN Alt. (none) -> 1N4448WSF-7 / 1N4448WSFQ-7, 1N4448WS; Part Number BAS16J,115 / BAS16J,135 -> (none); Part Number Alt. 1N4448WSF-7 / 1N4448WSFQ-7, 1N4448WS -> (none)
- D32: MPN (none) -> BAS16J,115 / BAS16J,135; MPN Alt. (none) -> 1N4448WSF-7 / 1N4448WSFQ-7, 1N4448WS; Part Number BAS16J,115 / BAS16J,135 -> (none); Part Number Alt. 1N4448WSF-7 / 1N4448WSFQ-7, 1N4448WS -> (none)
- D33, D34: MPN (none) -> UDZVTE-1716B; MPN Alt. (none) -> MM3Z16VB; Part Number UDZVTE-1716B -> (none); Part Number Alt. MM3Z16VB -> (none)
- D5: DNP DNP -> (none); MPN (none) -> BZT52C6V2-7-F; Part Number BZT52C6V2-7-F -> (none)
- F2, F3: MPN (none) -> 3413.0223.22; MPN Alt. (none) -> C1Q 5; Part Number 3413.0223.22 -> (none); Part Number Alt. C1Q 5 -> (none)
- J2, J3, J5: DNP DNP -> (none); MPN (none) -> 132134; Part Number 132134 -> (none)
- J6: MPN (none) -> M20-7810245 / M20-7810245R; MPN Alt. (none) -> HLE-102-02-G-DV-BE / HLE-102-02-F-DV-BE / HLE-102-02-L-DV-B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; Part Number M20-7810245 / M20-7810245R -> (none); Part Number Alt. HLE-102-02-G-DV-BE / HLE-102-02-F-DV-BE / HLE-102-02-L-DV-B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 -> (none)
- J8: MPN (none) -> M20-7811045 / M20-7811045R; MPN Alt. (none) -> HLE-110-02-S-DV-A-K / HLE-110-02-L-DV-A-K / HLE-110-02-SM-D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; Part Number M20-7811045 / M20-7811045R -> (none); Part Number Alt. HLE-110-02-S-DV-A-K / HLE-110-02-L-DV-A-K / HLE-110-02-SM-D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 -> (none)
- J9: MPN (none) -> M20-7810245 / M20-7810245R; MPN Alt. (none) -> HLE-102-02-L-DV / HLE-102-02-F-DV / HLE-102-02-G-DV / HLE-1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; Part Number M20-7810245 / M20-7810245R -> (none); Part Number Alt. HLE-102-02-L-DV / HLE-102-02-F-DV / HLE-102-02-G-DV / HLE-1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 -> (none)
- J92: DNP DNP -> (none); MPN (none) -> 39281023; MPN Alt. (none) -> 39288020, 39293026, 39310020; Part Number 39281023 -> (none); Part Number Alt. 39288020, 39293026, 39310020 -> (none)
- Q1, Q3, Q36: MPN (none) -> MMBT3904-7-F; MPN Alt. (none) -> MMBT3904,215; Part Number MMBT3904-7-F -> (none); Part Number Alt. MMBT3904,215 -> (none)
- Q2, Q4: MPN (none) -> MMBT3906-7-F; MPN Alt. (none) -> MMBT3906,215; Part Number MMBT3906-7-F -> (none); Part Number Alt. MMBT3906,215 -> (none)
- Q37: MPN (none) -> 2N7002VC-7; MPN Alt. (none) -> 2N7002V, CMLDM7002AJ TR PBFREE; Part Number 2N7002VC-7 -> (none); Part Number Alt. 2N7002V, CMLDM7002AJ TR PBFREE -> (none)
- R1, R10, R11, R8, R9: MPN (none) -> RK73H2ATTD1000F; Part Number RK73H2ATTD1000F -> (none)
- R15, R162, R17, R18, R19, R61: MPN (none) -> RK73H2ATTD1002F; Part Number RK73H2ATTE1002F -> (none)
- R163, R62: MPN (none) -> RK73H2ATTD8201F; Part Number RK73H2ATTD8201F -> (none)
- R164: MPN (none) -> RK73H2ATTD1302F; Part Number RK73H2ATTE1302F -> (none)
- R192: MPN (none) -> RK73H2ATTD4641F; Part Number RK73H2ATTD4641F -> (none)
- R2: MPN (none) -> MCU08050D1001BP500; Part Number MCU08050D1001BP500 -> (none)
- R291: MPN (none) -> RK73H2ATTD1003F; Part Number RK73H2ATTE1003F -> (none)
- R292: MPN (none) -> RK73H2ATTD4703F; Part Number RK73H2ATTD4703F -> (none)
- R4: DNP DNP -> (none); MPN (none) -> RK73H2ATTD1000F; Part Number RK73H2ATTD1000F -> (none)
- R58: MPN (none) -> RK73H2ATTD4700F; Part Number RK73H2ATTD4700F -> (none)
- R6: MPN (none) -> RK73H2ATTE2002F; Part Number RK73H2ATTE2002F -> (none)
- R7: MPN (none) -> TNPW080516K2BEEA; MPN Alt. (none) -> TNPW080516K2BEEN; Manufacturer Alt. (none) -> Vishay; Part Number TNPW080516K2BEEN -> (none)
- RN5, RN6: DNP DNP -> (none); MPN (none) -> ACASN1002S1002P1AT; MPN Alt. (none) -> ACASN5002S5002P1AT, ACASN2002S2002P1AT, ACASN1003E1003P1AT; Part Number ACASN1002S1002P1AT -> (none); Part Number Alt. ACASN5002S5002P1AT, ACASN2002S2002P1AT, ACASN1003E1003P1AT -> (none)
- TP18, TP2, TP20, TP52: DNP DNP -> (none); MPN (none) -> 5019; Part Number 5019 -> (none)
- U1: MPN (none) -> INA821ID; MPN Alt. (none) -> INA821IDR, INA819ID, INA819IDR; Part Number INA821ID -> (none); Part Number Alt. INA821IDR, INA819ID, INA819IDR -> (none)
- U2: MPN (none) -> OPA37GU/2K5; MPN Alt. (none) -> OPA37GU; Part Number OPA37GU/2K5 -> (none); Part Number Alt. OPA37GU -> (none)
- U7, U9: MPN (none) -> TLVH431IDBZR; MPN Alt. (none) -> TLVH431QDBZR, TLVH431CDBZR; Part Number TLVH431IDBZR -> (none); Part Number Alt. TLVH431QDBZR, TLVH431CDBZR -> (none)
