File: pcbs/amp ctrl/shutdown_logic_per-chan.kicad_sch (KiCad schematic)
At the start: 24 parts, among them U17 74LVC2G17, U4 74HC02, U5 74LVC2G06

Commit message: BOM & reset fixes
Amp ctrl: changed name of "Manufacturer" field to "MPN" to work with Aisler
Amp ctrl: added part number to logic inverter, corrected various typos and part number problems
Backplane: added pull-down to Shutdown_Reset signal (#35)
Backplane: rethought Shutdown_Force circuit to make fail-safe (broken connections->shutdown), make work correctly (fixes #35)
Backplane: updated/corrected various schematic annotations
Parts:
- C14, C15, C17: MPN (none) -> C0603C105K4RACTU; Part Number C0603C105K4RACTU -> (none)
- C18, C79: MPN (none) -> C0603C104K5RACTU; Part Number C0603C104K5RACTU -> (none)
- D13, D14, D35, D36: MPN (none) -> BAS16J,115 / BAS16J,135; MPN Alt. (none) -> 1N4448WSF-7 / 1N4448WSFQ-7, 1N4448WS; Part Number BAS16J,115 / BAS16J,135 -> (none); Part Number Alt. 1N4448WSF-7 / 1N4448WSFQ-7, 1N4448WS -> (none)
- JP21, JP72: DNP DNP -> (none)
- R12, R13: MPN (none) -> RK73H2ATTD4703F; Part Number RK73H2ATTD4703F -> (none)
- R53, R54: MPN (none) -> RK73H2ATTD1002F; Part Number RK73H2ATTE1002F -> (none)
- U17: MPN (none) -> 74LVC2G17GV,125; MPN Alt. (none) -> SN74LVC2G17DBVR / SN74LVC2G17DBVT, 74LVC2G17W6-7; Part Number 74LVC2G17GV,125 -> (none); Part Number Alt. SN74LVC2G17DBVR / SN74LVC2G17DBVT, 74LVC2G17W6-7 -> (none)
- U4: MPN (none) -> 74VHC02FT; MPN Alt. (none) -> 74LV02APWJ, SN74LVC02APWR / SN74LVC02APWT; Part Number 74VHC02FT -> (none); Part Number Alt. 74LV02APWJ, SN74LVC02APWR / SN74LVC02APWT -> (none)
- U5: MPN (none) -> 74LVC2G06GV,125; MPN Alt. (none) -> SN74LVC2G06DBVR / SN74LVC2G06DBVT, 74LVC2G06W6-7; Part Number 74LVC2G06GV,125 -> (none); Part Number Alt. SN74LVC2G06DBVR / SN74LVC2G06DBVT, 74LVC2G06W6-7 -> (none)
Changed lines of the file:
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@@
 			)
 		)
-		(property "Part Number" "RK73H2ATTD4703F"
+		(property "MPN" "RK73H2ATTD4703F"
 			(at 133.35 96.52 0)
 			(effects
@@
 			)
 		)
-		(property "Part Number" "C0603C105K4RACTU"
+		(property "Type" "SMT"
 			(at 148.59 160.02 0)
 			(effects
@@
 			)
 		)
-		(property "Type" "SMT"
-			(at 148.59 160.02 0)
+		(property "MPN" "C0603C105K4RACTU"
+			(at 148.59 160.02 90)
 			(effects
 				(font
@@
 			)
 		)
-		(property "Part Number" "C0603C105K4RACTU"
+		(property "Type" "SMT"
 			(at 111.76 48.26 0)
 			(effects
@@
 			)
 		)
-		(property "Type" "SMT"
-			(at 111.76 48.26 0)
+		(property "MPN" "C0603C105K4RACTU"
+			(at 111.76 48.26 90)
 			(effects
 				(font
@@
 			)
 		)
-		(property "Part Number" "74LVC2G06GV,125"
+		(property "Type" "SMT"
 			(at 105.41 92.71 0)
 			(effects
@@
 			)
 		)
-		(property "Type" "SMT"
+		(property "Manufacturer Alt." "Texas Instruments, Diodes Inc."
 			(at 105.41 92.71 0)
 			(effects
@@
 			)
 		)
-		(property "Manufacturer Alt." "Texas Instruments, Diodes Inc."
+		(property "MPN" "74LVC2G06GV,125"
 			(at 105.41 92.71 0)
 			(effects
@@
 			)
 		)
-		(property "Part Number Alt." "SN74LVC2G06DBVR / SN74LVC2G06DBVT, 74LVC2G06W6-7"
+		(property "MPN Alt." "SN74LVC2G06DBVR / SN74LVC2G06DBVT, 74LVC2G06W6-7"
 			(at 105.41 92.71 0)
 			(effects
@@
 			)
 		)
-		(property "Part Number" "74LVC2G17GV,125"
+		(property "Type" "SMT"
 			(at 156.21 92.71 0)
 			(effects
@@
 			)
 		)
-		(property "Type" "SMT"
+		(property "Manufacturer Alt." "Texas Instruments, Diodes Inc."
 			(at 156.21 92.71 0)
 			(effects
@@
 			)
 		)
-		(property "Manufacturer Alt." "Texas Instruments, Diodes Inc."
+		(property "MPN" "74LVC2G17GV,125"
 			(at 156.21 92.71 0)
 			(effects
@@
 			)
 		)
-		(property "Part Number Alt." "SN74LVC2G17DBVR / SN74LVC2G17DBVT, 74LVC2G17W6-7"
+		(property "MPN Alt." "SN74LVC2G17DBVR / SN74LVC2G17DBVT, 74LVC2G17W6-7"
 			(at 156.21 92.71 0)
 			(effects
@@
 			)
 		)
-		(property "Part Number" "74LVC2G17GV,125"
+		(property "Type" "SMT"
 			(at 156.21 55.88 0)
 			(effects
@@
 			)
 		)
-		(property "Type" "SMT"
+		(property "Manufacturer Alt." "Texas Instruments, Diodes Inc."
 			(at 156.21 55.88 0)
 			(effects
@@
 			)
 		)
-		(property "Manufacturer Alt." "Texas Instruments, Diodes Inc."
+		(property "MPN" "74LVC2G17GV,125"
 			(at 156.21 55.88 0)
 			(effects
@@
 			)
 		)
-		(property "Part Number Alt." "SN74LVC2G17DBVR / SN74LVC2G17DBVT, 74LVC2G17W6-7"
+		(property "MPN Alt." "SN74LVC2G17DBVR / SN74LVC2G17DBVT, 74LVC2G17W6-7"
 			(at 156.21 55.88 0)
 			(effects
@@
 			)
 		)
-		(property "Part Number" "C0603C105K4RACTU"
+		(property "Type" "SMT"
 			(at 161.29 48.26 0)
 			(effects
@@
 			)
 		)
-		(property "Type" "SMT"
-			(at 161.29 48.26 0)
+		(property "MPN" "C0603C105K4RACTU"
+			(at 161.29 48.26 90)
 			(effects
 				(font
@@
 			)
 		)
-		(property "DNP" "DNP"
-			(at 68.58 156.21 0)
-			(effects
-				(font
-					(size 1.27 1.27)
-				)
-			)
-		)
 		(property "Type" "Through-hole"
 			(at 68.58 153.67 0)
@@
 			)
 		)
-		(property "Part Number" "RK73H2ATTD4703F"
+		(property "MPN" "RK73H2ATTD4703F"
 			(at 133.35 59.69 0)
 			(effects
@@
 			)
 		)
-		(property "Part Number" "74VHC02FT"
+		(property "Type" "SMT"
 			(at 88.9 92.71 0)
 			(effects
@@
 			)
 		)
-		(property "Part Number Alt." "74LV02APWJ, SN74LVC02APWR / SN74LVC02APWT"
+		(property "MPN" "74VHC02FT"
 			(at 88.9 92.71 0)
 			(effects
@@
 			)
 		)
-		(property "Type" "SMT"
+		(property "MPN Alt." "74LV02APWJ, SN74LVC02APWR / SN74LVC02APWT"
 			(at 88.9 92.71 0)
 			(effects
@@
 			)
 		)
-		(property "Part Number" "74VHC02FT"
+		(property "Type" "SMT"
 			(at 90.17 55.88 0)
 			(effects
@@
 			)
 		)
-		(property "Part Number Alt." "74LV02APWJ, SN74LVC02APWR / SN74LVC02APWT"
+		(property "MPN" "74VHC02FT"
 			(at 90.17 55.88 0)
 			(effects
@@
 			)
 		)
-		(property "Type" "SMT"
+		(property "MPN Alt." "74LV02APWJ, SN74LVC02APWR / SN74LVC02APWT"
 			(at 90.17 55.88 0)
 			(effects
@@
 			)
 		)
-		(property "Part Number" "74VHC02FT"
+		(property "Type" "SMT"
 			(at 179.07 58.42 0)
 			(effects
@@
 			)
 		)
-		(property "Part Number Alt." "74LV02APWJ, SN74LVC02APWR / SN74LVC02APWT"
+		(property "MPN" "74VHC02FT"
 			(at 179.07 58.42 0)
 			(effects
@@
 			)
 		)
-		(property "Type" "SMT"
+		(property "MPN Alt." "74LV02APWJ, SN74LVC02APWR / SN74LVC02APWT"
 			(at 179.07 58.42 0)
 			(effects
@@
 			)
 		)
-		(property "Part Number" "74VHC02FT"
+		(property "Type" "SMT"
 			(at 179.07 95.25 0)
 			(effects
@@
 			)
 		)
-		(property "Part Number Alt." "74LV02APWJ, SN74LVC02APWR / SN74LVC02APWT"
+		(property "MPN" "74VHC02FT"
 			(at 179.07 95.25 0)
 			(effects
@@
 			)
 		)
-		(property "Type" "SMT"
+		(property "MPN Alt." "74LV02APWJ, SN74LVC02APWR / SN74LVC02APWT"
 			(at 179.07 95.25 0)
 			(effects
@@
 			)
 		)
-		(property "Part Number" "74VHC02FT"
+		(property "Type" "SMT"
 			(at 143.51 177.8 0)
 			(effects
@@
 			)
 		)
-		(property "Part Number Alt." "74LV02APWJ, SN74LVC02APWR / SN74LVC02APWT"
+		(property "MPN" "74VHC02FT"
 			(at 143.51 177.8 0)
 			(effects
@@
 			)
 		)
-		(property "Type" "SMT"
+		(property "MPN Alt." "74LV02APWJ, SN74LVC02APWR / SN74LVC02APWT"
 			(at 143.51 177.8 0)
 			(effects
@@
 			)
 		)
-		(property "Part Number" "RK73H2ATTE1002F"
-			(at 193.04 58.42 0)
+		(property "MPN" "RK73H2ATTD1002F"
+			(at 193.04 58.42 90)
 			(effects
 				(font
@@
 			)
 		)
-		(property "Part Number" "RK73H2ATTE1002F"
-			(at 193.04 95.25 0)
+		(property "MPN" "RK73H2ATTD1002F"
+			(at 193.04 95.25 90)
 			(effects
 				(font
@@
 			)
 		)
-		(property "Part Number" "C0603C104K5RACTU"
+		(property "MPN" "C0603C104K5RACTU"
 			(at 198.12 62.23 0)
 			(effects
@@
 			)
 		)
-		(property "Part Number" "C0603C104K5RACTU"
+		(property "MPN" "C0603C104K5RACTU"
 			(at 198.12 99.06 0)
 			(effects
@@
 			)
 		)
-		(property "Part Number" "74LVC2G06GV,125"
+		(property "Type" "SMT"
 			(at 106.68 55.88 0)
 			(effects
@@
 			)
 		)
-		(property "Type" "SMT"
+		(property "Manufacturer Alt." "Texas Instruments, Diodes Inc."
 			(at 106.68 55.88 0)
 			(effects
@@
 			)
 		)
-		(property "Manufacturer Alt." "Texas Instruments, Diodes Inc."
+		(property "MPN" "74LVC2G06GV,125"
 			(at 106.68 55.88 0)
 			(effects
@@
 			)
 		)
-		(property "Part Number Alt." "SN74LVC2G06DBVR / SN74LVC2G06DBVT, 74LVC2G06W6-7"
+		(property "MPN Alt." "SN74LVC2G06DBVR / SN74LVC2G06DBVT, 74LVC2G06W6-7"
 			(at 106.68 55.88 0)
 			(effects
@@
 			)
 		)
-		(property "Part Number" "BAS16J,115 / BAS16J,135"
+		(property "Type" "SMT"
 			(at 209.55 58.42 0)
 			(effects
@@
 			)
 		)
-		(property "Part Number Alt." "1N4448WSF-7 / 1N4448WSFQ-7, 1N4448WS"
+		(property "MPN" "BAS16J,115 / BAS16J,135"
 			(at 209.55 58.42 0)
 			(effects
@@
 			)
 		)
-		(property "Type" "SMT"
+		(property "MPN Alt." "1N4448WSF-7 / 1N4448WSFQ-7, 1N4448WS"
 			(at 209.55 58.42 0)
 			(effects
@@
 			)
 		)
-		(property "Part Number" "BAS16J,115 / BAS16J,135"
+		(property "Type" "SMT"
 			(at 209.55 95.25 0)
 			(effects
@@
 			)
 		)
-		(property "Part Number Alt." "1N4448WSF-7 / 1N4448WSFQ-7, 1N4448WS"
+		(property "MPN" "BAS16J,115 / BAS16J,135"
 			(at 209.55 95.25 0)
 			(effects
@@
 			)
 		)
-		(property "Type" "SMT"
+		(property "MPN Alt." "1N4448WSF-7 / 1N4448WSFQ-7, 1N4448WS"
 			(at 209.55 95.25 0)
 			(effects
@@
 			)
 		)
-		(property "DNP" "DNP"
-			(at 68.58 167.64 0)
-			(effects
-				(font
-					(size 1.27 1.27)
-				)
-			)
-		)
 		(property "Type" "Through-hole"
 			(at 68.58 165.1 0)
@@
 			)
 		)
-		(property "Part Number" "BAS16J,115 / BAS16J,135"
+		(property "Type" "SMT"
 			(at 209.55 33.02 0)
 			(effects
@@
 			)
 		)
-		(property "Part Number Alt." "1N4448WSF-7 / 1N4448WSFQ-7, 1N4448WS"
+		(property "MPN" "BAS16J,115 / BAS16J,135"
 			(at 209.55 33.02 0)
 			(effects
@@
 			)
 		)
-		(property "Type" "SMT"
+		(property "MPN Alt." "1N4448WSF-7 / 1N4448WSFQ-7, 1N4448WS"
 			(at 209.55 33.02 0)
 			(effects
@@
 			)
 		)
-		(property "Part Number" "BAS16J,115 / BAS16J,135"
+		(property "Type" "SMT"
 			(at 209.55 81.28 0)
 			(effects
@@
 			)
 		)
-		(property "Part Number Alt." "1N4448WSF-7 / 1N4448WSFQ-7, 1N4448WS"
+		(property "MPN" "BAS16J,115 / BAS16J,135"
 			(at 209.55 81.28 0)
 			(effects
@@
 			)
 		)
-		(property "Type" "SMT"
+		(property "MPN Alt." "1N4448WSF-7 / 1N4448WSFQ-7, 1N4448WS"
 			(at 209.55 81.28 0)
 			(effects
