File: pcbs/amp ctrl/shutdown_logic_per-chan.kicad_sch (KiCad schematic)
At the start: 24 parts, among them U17 74LVC2G17, U4 74HC02, U5 74LVC2G06

Commit message: Backplane comms updates, manufacturing renaming
Removed misspelled "maunfacturing" folder, fixed gitignore rule to remove manufacturing folders within individual PCB folders too
Changed SCKI/SCKO terminology to SCK, SCK_LB (loopback) for clarity
Added ADC_CS loopback signal between amp ctrl board & backplane for better fast-clock timing (#38)
Backplane: changed LVDS FPGA outputs to single-ended FPGA outputs to gain more I/O pins, added external LVDS transceivers (#38)
Backplane: replaced global clock & ~LDAC buffers with a separate FPGA pin for each amp ctrl board (#38)
Backplane: removed +2.5V power supply and level translations, no longer needed without FPGA I/O pins using LVDS_25 I/O configuration
Backplane: replaced +VDC-input resistor with solder jumper (on by default)
Backplane: changed field names (Part Number to MPN) to match Aisler's naming convention for automatic recognition
Amp ctrl: fixed optional level-shifter circuit on each channel for voltage inputs (#9) schematic & channel-1 layout
Parts:
- JP21, JP72: value ~ -> (none)

Commit message: Amp ctrl layout for spring pins
Copied layout to all channels & cleaned up inter-channel routing
Updated footprints to latest copies from libraries
Added new SOT-563 footprint for wider clearance between pads, as KiCAD library now has boundary-pushing 0.15 mm (vs. 0.2 mm recc. in 2N7002 datasheet)
Fixed DRC errors
Marked former inter-board connectors (now alternates for spring pins) as DNP
Parts:
- JP21, JP72: now in the parts list
Changed lines of the file:
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@@
 		(in_bom no)
 		(on_board yes)
-		(in_pos_files yes)
+		(in_pos_files no)
 		(dnp no)
 		(property "Reference" "TP12"
@@
 		(in_bom no)
 		(on_board yes)
-		(in_pos_files yes)
+		(in_pos_files no)
 		(dnp no)
 		(property "Reference" "TP7"
@@
 		(in_bom no)
 		(on_board yes)
-		(in_pos_files yes)
+		(in_pos_files no)
 		(dnp no)
 		(property "Reference" "TP11"
@@
 		(in_bom no)
 		(on_board yes)
-		(in_pos_files yes)
+		(in_pos_files no)
 		(dnp no)
 		(property "Reference" "TP15"
@@
 		(body_style 1)
 		(exclude_from_sim no)
-		(in_bom no)
+		(in_bom yes)
 		(on_board yes)
-		(in_pos_files yes)
+		(in_pos_files no)
 		(dnp yes)
 		(property "Reference" "JP21"
@@
 		(in_bom no)
 		(on_board yes)
-		(in_pos_files yes)
+		(in_pos_files no)
 		(dnp no)
 		(property "Reference" "TP14"
@@
 		(in_bom no)
 		(on_board yes)
-		(in_pos_files yes)
+		(in_pos_files no)
 		(dnp no)
 		(property "Reference" "TP140"
@@
 		(body_style 1)
 		(exclude_from_sim no)
-		(in_bom no)
+		(in_bom yes)
 		(on_board yes)
-		(in_pos_files yes)
+		(in_pos_files no)
 		(dnp yes)
 		(property "Reference" "JP72"
