File: pcbs/amp ctrl/amp ctrl.kicad_pcb (KiCad board)
At the start: 4 copper layers, 343.2 x 120 mm, 1251 parts, among them J1 Conn_02x25_Odd_Even, J11 Conn_01x02, J13 Conn_02x02, J14 RF_Shield_Two_Pieces, J15 RJ45_Shielded, J17 RJ45_Shielded, J21 Conn_02x02, J23 Conn_02x10_Odd_Even, J24 Conn_02x02, J26 Conn_01x02, J31 Conn_02x02, J33 Conn_02x10_Odd_Even, J34 Conn_02x02, J36 Conn_01x02, J4 Conn_01x02, J41 Conn_02x02, J43 Conn_02x10_Odd_Even, J44 Conn_02x02, J46 Conn_01x02, J51 Conn_02x02, J53 Conn_02x10_Odd_Even, J54 Conn_02x02, J56 Conn_01x02, J6 Conn_02x02, J61 Conn_02x02, J63 Conn_02x10_Odd_Even, J64 Conn_02x02, J66 Conn_01x02, J7 Conn_02x08_Odd_Even, J71 Conn_02x02, J73 Conn_02x10_Odd_Even, J74 Conn_02x02, J76 Conn_01x02, J8 Conn_02x10_Odd_Even, J81 Conn_02x02, J83 Conn_02x10_Odd_Even, J84 Conn_02x02, J86 Conn_01x02, J88 RJ45_Shielded, J89 Conn_02x02, J9 Conn_02x02, J90 Conn_02x02, J91 Conn_02x02, J92 Conn_01x02, J93 Conn_01x02, J94 Conn_01x02, J95 Conn_01x02, J96 Conn_01x02, J97 Conn_01x02, J98 Conn_01x02, J99 Conn_01x02, Q1 MMBT3904, Q10 MMBT3906, Q11 MMBT3904, Q12 MMBT3906, Q13 MMBT3904, Q14 MMBT3906, Q15 MMBT3904, Q16 MMBT3906, Q17 MMBT3904, Q18 MMBT3906, Q19 MMBT3904, Q2 MMBT3906, Q20 MMBT3906, Q21 MMBT3904, Q22 MMBT3906, Q23 MMBT3904, Q24 MMBT3906, Q25 MMBT3904, Q26 MMBT3906, Q27 MMBT3904, Q28 MMBT3906, Q29 MMBT3904, Q3 MMBT3904, Q30 MMBT3906, Q31 MMBT3904, Q32 MMBT3906, Q33 MMBT3904, Q34 MMBT3904, Q35 MMBT3906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

Commit message: Added footprints and started layout of interposer board
Parts:
- moved Q37 5.68 mm to (127.2, 51.2)
- moved H10 5.68 mm to (298.0, 151.6)
- moved H2 5.68 mm to (100.0, 151.6)
- moved H4 5.68 mm to (364.0, 151.6)
- moved H6 5.68 mm to (166.0, 151.6)
- moved H8 5.68 mm to (232.0, 151.6)
- moved C1 5.68 mm to (59.0, 86.8)
- moved C10 5.68 mm to (132.0, 57.3)
- moved C101 5.68 mm to (174.2, 111.0)
- moved C102 5.68 mm to (180.8, 90.8)
- moved C103 5.68 mm to (211.0, 61.0)
- moved C104 5.68 mm to (208.2, 65.5)
- moved C105 5.68 mm to (209.8, 76.0)
- moved C106 5.68 mm to (208.2, 71.3)
- moved C107 5.68 mm to (212.2, 53.0)
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