File: pcbs/amp ctrl/amp ctrl.kicad_pcb (KiCad board)
At the start: 4 copper layers, 343.2 x 120 mm, 1251 parts, among them J1 Conn_02x25_Odd_Even, J11 Conn_01x02, J13 Conn_02x02, J14 RF_Shield_Two_Pieces, J15 RJ45_Shielded, J17 RJ45_Shielded, J21 Conn_02x02, J23 Conn_02x10_Odd_Even, J24 Conn_02x02, J26 Conn_01x02, J31 Conn_02x02, J33 Conn_02x10_Odd_Even, J34 Conn_02x02, J36 Conn_01x02, J4 Conn_01x02, J41 Conn_02x02, J43 Conn_02x10_Odd_Even, J44 Conn_02x02, J46 Conn_01x02, J51 Conn_02x02, J53 Conn_02x10_Odd_Even, J54 Conn_02x02, J56 Conn_01x02, J6 Conn_02x02, J61 Conn_02x02, J63 Conn_02x10_Odd_Even, J64 Conn_02x02, J66 Conn_01x02, J7 Conn_02x08_Odd_Even, J71 Conn_02x02, J73 Conn_02x10_Odd_Even, J74 Conn_02x02, J76 Conn_01x02, J8 Conn_02x10_Odd_Even, J81 Conn_02x02, J83 Conn_02x10_Odd_Even, J84 Conn_02x02, J86 Conn_01x02, J88 RJ45_Shielded, J89 Conn_02x02, J9 Conn_02x02, J90 Conn_02x02, J91 Conn_02x02, J92 Conn_01x02, J93 Conn_01x02, J94 Conn_01x02, J95 Conn_01x02, J96 Conn_01x02, J97 Conn_01x02, J98 Conn_01x02, J99 Conn_01x02, Q1 MMBT3904, Q10 MMBT3906, Q11 MMBT3904, Q12 MMBT3906, Q13 MMBT3904, Q14 MMBT3906, Q15 MMBT3904, Q16 MMBT3906, Q17 MMBT3904, Q18 MMBT3906, Q19 MMBT3904, Q2 MMBT3906, Q20 MMBT3906, Q21 MMBT3904, Q22 MMBT3906, Q23 MMBT3904, Q24 MMBT3906, Q25 MMBT3904, Q26 MMBT3906, Q27 MMBT3904, Q28 MMBT3906, Q29 MMBT3904, Q3 MMBT3904, Q30 MMBT3906, Q31 MMBT3904, Q32 MMBT3906, Q33 MMBT3904, Q34 MMBT3904, Q35 MMBT3906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

Commit message: Library & amp ctrl updates for spring connectors
Library: added footprints for spring connector bare pads (both 70AAJ & SIB)
Library: added SIB contact point markers to all footprints
Library: corrected 70AAJ outline size
Amp ctrl: started layout change on channel 2
Parts:
- added J10: Conn_01x05, shim:Conn_70AAJ-M_SIB_1x05_P2.54mm_F_bare, F.Cu at (-105.0, 115.8)
- added J100: Conn_01x05, shim:Conn_70AAJ-M_SIB_1x05_P2.54mm_F_bare, F.Cu at (-105.0, 189.8)
- added J101: Conn_01x05, shim:Conn_70AAJ-M_SIB_1x05_P2.54mm_F_bare, F.Cu at (-105.0, 201.8)
- added J102: Conn_01x05, shim:Conn_70AAJ-M_SIB_1x05_P2.54mm_F_bare, F.Cu at (-88.8, 189.8)
- added J103: Conn_01x05, shim:Conn_70AAJ-M_SIB_1x05_P2.54mm_F_bare, F.Cu at (-88.8, 201.8)
- added J104: Conn_01x05, shim:Conn_70AAJ-M_SIB_1x05_P2.54mm_F_bare, F.Cu at (-72.5, 189.8)
- added J105: Conn_01x05, shim:Conn_70AAJ-M_SIB_1x05_P2.54mm_F_bare, F.Cu at (-72.5, 201.8)
- added J106: Conn_01x05, shim:Conn_70AAJ-M_SIB_1x05_P2.54mm_F_bare, F.Cu at (-56.3, 189.8)
- added J107: Conn_01x05, shim:Conn_70AAJ-M_SIB_1x05_P2.54mm_F_bare, F.Cu at (-56.3, 201.8)
- added J12: Conn_01x05, shim:Conn_70AAJ-M_SIB_1x05_P2.54mm_F_bare, B.Cu at (146.2, 110.8)
- added J16: Conn_01x05, shim:Conn_70AAJ-M_SIB_1x05_P2.54mm_F_bare, F.Cu at (-72.5, 115.8)
- added J22: Conn_01x05, shim:Conn_70AAJ-M_SIB_1x05_P2.54mm_F_bare, F.Cu at (-56.3, 115.8)
- added J25: Conn_01x05, shim:Conn_70AAJ-M_SIB_1x05_P2.54mm_F_bare, F.Cu at (-105.0, 165.8)
- added J27: Conn_01x05, shim:Conn_70AAJ-M_SIB_1x05_P2.54mm_F_bare, F.Cu at (-88.8, 165.8)
- added J32: Conn_01x05, shim:Conn_70AAJ-M_SIB_1x05_P2.54mm_F_bare, F.Cu at (-72.5, 165.8)
- added J35: Conn_01x05, shim:Conn_70AAJ-M_SIB_1x05_P2.54mm_F_bare, B.Cu at (344.0, 110.8)
- added J37: Conn_01x05, shim:Conn_70AAJ-M_SIB_1x05_P2.54mm_F_bare, F.Cu at (-105.0, 127.8)
- added J42: Conn_01x05, shim:Conn_70AAJ-M_SIB_1x05_P2.54mm_F_bare, B.Cu at (158.8, 110.8)
- added J45: Conn_01x05, shim:Conn_70AAJ-M_SIB_1x05_P2.54mm_F_bare, F.Cu at (-72.5, 127.8)
- added J47: Conn_01x05, shim:Conn_70AAJ-M_SIB_1x05_P2.54mm_F_bare, F.Cu at (-56.3, 127.8)
- added J52: Conn_01x05, shim:Conn_70AAJ-M_SIB_1x05_P2.54mm_F_bare, F.Cu at (-105.0, 177.8)
- added J55: Conn_01x05, shim:Conn_70AAJ-M_SIB_1x05_P2.54mm_F_bare, F.Cu at (-88.8, 177.8)
- added J57: Conn_01x05, shim:Conn_70AAJ-M_SIB_1x05_P2.54mm_F_bare, F.Cu at (-72.5, 177.8)
- added J62: Conn_01x05, shim:Conn_70AAJ-M_SIB_1x05_P2.54mm_F_bare, B.Cu at (358.2, 110.8)
- added J65: Conn_01x05, shim:Conn_70AAJ-M_SIB_1x05_P2.54mm_F_bare, F.Cu at (-105.0, 139.8)
- added J67: Conn_01x05, shim:Conn_70AAJ-M_SIB_1x05_P2.54mm_F_bare, F.Cu at (-105.0, 151.8)
- added J72: Conn_01x05, shim:Conn_70AAJ-M_SIB_1x05_P2.54mm_F_bare, B.Cu at (146.2, 96.2)
- added J75: Conn_01x05, shim:Conn_70AAJ-M_SIB_1x05_P2.54mm_F_bare, B.Cu at (158.8, 96.2)
- added J77: Conn_01x05, shim:Conn_70AAJ-M_SIB_1x05_P2.54mm_F_bare, F.Cu at (-72.5, 139.8)
- added J82: Conn_01x05, shim:Conn_70AAJ-M_SIB_1x05_P2.54mm_F_bare, F.Cu at (-72.5, 151.8)
- added J85: Conn_01x05, shim:Conn_70AAJ-M_SIB_1x05_P2.54mm_F_bare, F.Cu at (-56.3, 139.8)
- added J87: Conn_01x05, shim:Conn_70AAJ-M_SIB_1x05_P2.54mm_F_bare, F.Cu at (-56.3, 151.8)
- C186, C84, R161, R77: moved to F.Cu
- moved R161 21.3 mm to (350.5, 125.0)
- moved R77 18.4 mm to (144.2, 126.0)
- moved C186 17.6 mm to (346.2, 125.0)
- moved C84 13.2 mm to (142.5, 123.3)
- moved R190 10.8 mm to (156.7, 78.2), turned to 90 degrees
- moved TP65 10.6 mm to (161.0, 78.2), turned to 0 degrees
- moved J86 10.4 mm to (351.7, 119.5)
- moved R167 7.38 mm to (158.5, 89.2), turned to 180 degrees
- moved Q7 7.11 mm to (146.8, 83.2)
- moved C65 6.93 mm to (146.8, 78.8)
- moved R185 6.93 mm to (146.8, 80.5)
- moved R189 6.09 mm to (153.4, 81.8)
- moved U49 6.09 mm to (156.2, 81.8)
- moved C217 6.03 mm to (139.2, 88.1), turned to 0 degrees
- moved R71 5.85 mm to (152.2, 76.5), turned to 180 degrees
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Routing:
- net /Channel 2/EA_Out_Filt: track 15.7 -> 29.3 mm, vias 0 -> 1
- net /Channel 2/Out+_Unfused: track 45.5 -> 57.9 mm
- net /Out8+: track 56.1 -> 44.1 mm
- net /Channel 2/Vout_cmd: track 62.0 -> 69.8 mm, vias 0 -> 1
- net Net-(D37-A): track 12.5 -> 6.66 mm
- net Net-(U49-REF): track 3.60 -> 8.34 mm
- net /Offset_Cal_Drive: track 320.3 -> 324.3 mm
- net /Vref_Buffered: track 686.1 -> 682.7 mm
- net Net-(Q8-C): track 14.8 -> 16.3 mm
- net GND: track 1000.9 -> 999.4 mm, vias 538 -> 536
- net Net-(Q7-C): track 16.6 -> 17.9 mm
- net Net-(Q8-B): track 6.47 -> 7.72 mm
- net Net-(Q5-B): track 8.82 -> 10.0 mm
- net Net-(JP112-A): track 18.4 -> 19.4 mm
- net /Channel 2/EA_Out: track 25.0 -> 24.3 mm
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