File: pcbs/amp ctrl/amp ctrl.kicad_pcb (KiCad board)
At the start: 4 copper layers, 343.2 x 120 mm, 1296 parts, among them J1 Conn_02x25_Odd_Even, J10 Conn_01x05, J100 Conn_01x05, J101 Conn_01x05, J102 Conn_01x05, J103 Conn_01x05, J104 Conn_01x05, J105 Conn_01x05, J106 Conn_01x05, J107 Conn_01x05, J108 Conn_01x02, J109 Conn_01x02, J11 Conn_01x02, J110 Conn_01x02, J111 Conn_01x02, J112 Conn_01x02, J113 Conn_01x02, J114 Conn_01x02, J115 Conn_01x02, J116 Conn_01x02, J117 Conn_01x02, J118 Conn_01x02, J119 Conn_01x02, J12 Conn_01x05, J120 Conn_01x02, J13 Conn_02x02, J14 RF_Shield_Two_Pieces, J15 RJ45_Shielded, J16 Conn_01x05, J17 RJ45_Shielded, J21 Conn_02x02, J22 Conn_01x05, J23 Conn_02x10_Odd_Even, J24 Conn_02x02, J25 Conn_01x05, J26 Conn_01x02, J27 Conn_01x05, J31 Conn_02x02, J32 Conn_01x05, J33 Conn_02x10_Odd_Even, J34 Conn_02x02, J35 Conn_01x05, J36 Conn_01x02, J37 Conn_01x05, J4 Conn_01x02, J41 Conn_02x02, J42 Conn_01x05, J43 Conn_02x10_Odd_Even, J44 Conn_02x02, J45 Conn_01x05, J46 Conn_01x02, J47 Conn_01x05, J51 Conn_02x02, J52 Conn_01x05, J53 Conn_02x10_Odd_Even, J54 Conn_02x02, J55 Conn_01x05, J56 Conn_01x02, J57 Conn_01x05, J6 Conn_02x02, J61 Conn_02x02, J62 Conn_01x05, J63 Conn_02x10_Odd_Even, J64 Conn_02x02, J65 Conn_01x05, J66 Conn_01x02, J67 Conn_01x05, J7 Conn_02x08_Odd_Even, J71 Conn_02x02, J72 Conn_01x05, J73 Conn_02x10_Odd_Even, J74 Conn_02x02, J75 Conn_01x05, J76 Conn_01x02, J77 Conn_01x05, J8 Conn_02x10_Odd_Even, J81 Conn_02x02, J82 Conn_01x05, J83 Conn_02x10_Odd_Even, J84 Conn_02x02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

Commit message: Amp ctrl layout for spring pins
Copied layout to all channels & cleaned up inter-channel routing
Updated footprints to latest copies from libraries
Added new SOT-563 footprint for wider clearance between pads, as KiCAD library now has boundary-pushing 0.15 mm (vs. 0.2 mm recc. in 2N7002 datasheet)
Fixed DRC errors
Marked former inter-board connectors (now alternates for spring pins) as DNP
Parts:
- C101, C118, C135, C152, C169, C19, R105, R119, R133, R14, R147, R91: moved to F.Cu
- Q37, Q41, Q45, Q49, Q53, Q57, Q61, Q65: footprint Package_TO_SOT_SMD:SOT-563 -> shim:SOT-563
- moved J10 308.9 mm to (116.9, 110.8)
- moved J16 302.6 mm to (182.9, 110.8)
- moved J22 301.2 mm to (212.2, 110.8)
- moved J65 299.8 mm to (116.9, 96.2), turned to 180 degrees
- moved J37 294.3 mm to (129.6, 110.8)
- moved J77 293.3 mm to (182.9, 96.2), turned to 180 degrees
- moved J85 291.8 mm to (212.2, 96.2), turned to 180 degrees
- moved J45 289.3 mm to (195.6, 110.8)
- moved J47 288.3 mm to (224.8, 110.8)
- moved J67 285.2 mm to (129.6, 96.2), turned to 180 degrees
- moved J82 279.9 mm to (195.6, 96.2), turned to 180 degrees
- moved J87 278.9 mm to (224.8, 96.2), turned to 180 degrees
- moved J32 266.3 mm to (314.9, 110.8)
- moved J106 262.4 mm to (344.1, 96.2), turned to 180 degrees
- moved J27 259.9 mm to (278.1, 110.8)
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Routing:
- net (no net): track 297.0 -> 0.00 mm
- net Net-(J118-Pin_2): track 17.4 -> 301.9 mm
- net GND: track 1027.6 -> 1225.2 mm, vias 532 -> 530
- net +VDC: track 486.6 -> 572.7 mm, vias 140 -> 149
- net /Vref_Buffered: track 698.4 -> 746.9 mm
- net /Offset_Cal_Short: track 586.8 -> 631.3 mm
- net /Channel 6/Vout_cmd: track 31.4 -> 70.6 mm, vias 0 -> 1
- net /Channel 8/Out+_Unfused: track 45.5 -> 78.5 mm
- net /Channel 7/Out+_Unfused: track 45.5 -> 78.5 mm
- net /Channel 6/Out+_Unfused: track 45.5 -> 78.5 mm
- net /Channel 1/Out+_Unfused: track 45.5 -> 78.5 mm
- net /Channel 5/Out+_Unfused: track 45.5 -> 78.5 mm
- net /Channel 3/Out+_Unfused: track 45.5 -> 78.5 mm
- net /Channel 4/Out+_Unfused: track 45.5 -> 78.5 mm
- net /Channel 3/Vout_cmd: track 32.5 -> 64.1 mm, vias 0 -> 1
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Other:
- board text removed: "Tap M3x0.5"
