File: pcbs/backplane/fpga.kicad_sch (KiCad schematic)
At the start: 67 parts, among them U28 Snickerdoodle

Commit message: Schematic file fix, misc. PCB
Fixed issue with KiCAD's automatic V5→V6 migration (corrected in 6.0.11) that caused problems with component references in multi-channel schematic sheets
Finished migration in amp ctrl PCB, inc. re-assigning "exclude from BOM" attributes to testpoints, solder jumpers
Added mounting hole to amp ctrl PCB for addl support to Ethernet jacks, power connector through stiffener
Parts:
- C? (x6): renamed from ?; value 1uF 50V X7R -> (none); footprint Capacitor_SMD:C_0805_2012Metric -> (none)
- C? (x9): renamed from ?; value 100nF 50V X7R -> (none); footprint Capacitor_SMD:C_0603_1608Metric -> (none)
- JP13, JP14, JP15, JP17, JP18, JP19, JP20, JP21, JP22, JP23, JP24, JP25, JP26, JP27, JP28, JP29, JP30: renamed from ?; value Jumper_NC_Small -> (none); footprint Jumper:SolderJumper-2_P1.3mm_Bridged_RoundedPad1.0x1.5mm -> (none)
- JP31: renamed from ?; value Jumper_NO_Small -> (none); footprint Jumper:SolderJumper-2_P1.3mm_Open_TrianglePad1.0x1.5mm -> (none)
- TP? (x7): renamed from ?; value TestPoint_Flag -> (none); footprint TestPoint:TestPoint_Keystone_5019_Minature -> (none)
- TP? (x4): renamed from ?; value TestPoint -> (none); footprint TestPoint:TestPoint_Pad_D2.0mm -> (none)
- U7: renamed from ?; symbol Regulator_Linear:MCP1703A-2502_SOT23 -> backplane-rescue:MCP1703A-2502_SOT23-Regulator_Linear
- U? (x3): renamed from ?; value 74LVC2T45 -> (none); footprint Martinos_std:VSSOP-8_2.3x2mm_P0.5mm -> (none)
- gave numbers to parts that had none: 18

Commit message: Amp ctrl: lengthened ADC & DAC reset delay to ~50 ms (#14) Backplane: added clock multiplier for 10 Mhz scanner clock (fixes #21) Backplane: reduced R5 from 10 to 1 ohm, to avoid excessive voltage drop (#20) Backplane: replaced 15V regulator with efficient voltage limiter (#20) Backplane: changed all mounting holes to signal ground Backplane: replaced +2.5V regulator with a higher-current model to support FPGA I/O bank current draw Updated to KiCAD 8
Parts:
- removed U11: 78M15, Package_TO_SOT_SMD:TO-252-2, symbol Regulator_Linear:LM78M05_TO252
- removed U7: AP2120N-2.5, Martinos_std:SOT-23, symbol backplane-rescue:MCP1703A-2502_SOT23-Regulator_Linear
- added C67: 100nF 50V X7R, Capacitor_SMD:C_0603_1608Metric, symbol Device:C
- added D17: 16V, Don_std:D_SOD-323F, symbol amp-ctrl-rescue:D_Zener_ALT-Device
- added JP16: Jumper_NO_Small, Jumper:SolderJumper-2_P1.3mm_Open_TrianglePad1.0x1.5mm, symbol Jumper:Jumper_2_Small_Open
- added JP32: Jumper_NC_Small, Jumper:SolderJumper-2_P1.3mm_Bridged_RoundedPad1.0x1.5mm, symbol backplane-rescue:Jumper_NC_Small-Device
- added Q10, Q11: MMBT3906, Package_TO_SOT_SMD:SOT-23, symbol Transistor_BJT:MMBT3906
- added Q9: D44H11G, Package_TO_SOT_THT:TO-220-3_Horizontal_TabDown, symbol Device:Q_NPN_BCE
- added R73: 0, Resistor_SMD:R_0805_2012Metric, symbol Device:R
- added R74: 20K, Resistor_SMD:R_0805_2012Metric, symbol Device:R
- added R75: 56, Resistor_SMD:R_0805_2012Metric, symbol Device:R
- added R76: 1K, Resistor_SMD:R_0805_2012Metric, symbol Device:R
- added TP12, TP13: TestPoint, TestPoint:TestPoint_Pad_D2.0mm, symbol Connector:TestPoint
- added U34: ICS501, Don_std:SOIC-8_3.9x4.9mm_P1.27mm, symbol Don:ICS501
- added U7: AP7361C-25E, Package_TO_SOT_SMD:SOT-223-3_TabPin2, symbol Regulator_Linear:LT1129-3.3_SOT223
- C21, C25, C27, C31, C34, C35: renamed from C?; value (none) -> 1uF 50V X7R; footprint (none) -> Capacitor_SMD:C_0805_2012Metric
- C22, C23, C24, C26, C28, C29, C30, C32, C33: renamed from C?; value (none) -> 100nF 50V X7R; footprint (none) -> Capacitor_SMD:C_0603_1608Metric
- JP13, JP14, JP15, JP17, JP18, JP19, JP20, JP21, JP22, JP23, JP24, JP25, JP26, JP27, JP28, JP29, JP30: value (none) -> Jumper_NC_Small; footprint (none) -> Jumper:SolderJumper-2_P1.3mm_Bridged_RoundedPad1.0x1.5mm
- JP31: value (none) -> Jumper_NO_Small; footprint (none) -> Jumper:SolderJumper-2_P1.3mm_Open_TrianglePad1.0x1.5mm
- R18: value 1 -> 1 0.25W; footprint Resistor_SMD:R_0805_2012Metric -> Resistor_SMD:R_2010_5025Metric; Notes Can substitute generic resistor with same package, value, 1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 -> (none); Part Number RK73H2ATTD1R00F -> RK73H2HTTE1R00F
- TP4, TP50, TP51, TP6, TP7, TP8, TP9: renamed from TP?; value (none) -> TestPoint_Flag; footprint (none) -> TestPoint:TestPoint_Keystone_5019_Minature
- TP52, TP53, TP62, TP63: renamed from TP?; value (none) -> TestPoint; footprint (none) -> TestPoint:TestPoint_Pad_D2.0mm
- U10, U8, U9: renamed from U?; value (none) -> 74LVC2T45; footprint (none) -> Martinos_std:VSSOP-8_2.3x2mm_P0.5mm
Connections:
- net +2.5V: now also U7.3 (VO)
- net +3V3: now also C67.2, JP32.1, U34.2 (Vdd), U34.7 (OE), U7.1 (VI)
- net 10Mhz: now also TP13.1, U34.1 (X1/IClk); no longer U9.3 (2A)
- net FPGA_Vin: now also Q9.3 (E); no longer C35.2
- net GND: now also C67.1, D17.2 (A), JP16.1 (A), R74.1, U34.3 (Gnd), U7.2 (GND)
- net at C34.2, JP31.1, L1.2: now also Q11.2 (E), Q9.2 (C), R75.2
- net 10Mhz_2.5 renamed Scanner_Clk_2.5
- new net: C35.2, D17.1 (K), Q9.1 (B), R73.1
- new net: TP12.1, U34.5 (Clk), U9.3 (2A)
- new net: JP16.2 (B), U34.6 (S0)
- new net: Q10.2 (E), R75.1, R76.1
- new net: JP32.2, U34.4 (S1)
- new net: Q10.3 (C), R73.2
- new net: Q10.1 (B), Q11.3 (C), R74.2
- new net: Q11.1 (B), R76.2
- no-connect marks 55 -> 56
Other:
- note added: "Requirements: 600 mA Iout-max Dropout voltage < 0.8V @ 600 mA"
- moved on the sheet: C22, C23, C24, C26, C28, C31, C32, C33, C34, C35, JP13, JP14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

Commit message: Comms fix, misc. improvements
Added 33KΩ pull-ups & pull-downs to amp ctrl board's LVDS inputs, to solve issues caused by unconfigured FPGA pins during boot (fixes #23)
Swapped backplane power input polarity for consistency with power connectors (fixes #20)
Added "manual enable" optical input to backplane, for safety: requires positive enable to keep amplifiers enabled
Connections:
- net Eth_Clk renamed ~{Power_Enable_Sense}
- net RGMII_RXD0: no longer names the net of J3.12 (Pin_12)
- net RGMII_RXD1: no longer names the net of J3.17 (Pin_17)
- net RGMII_RXD2: no longer names the net of J3.19 (Pin_19)
- net RGMII_RXD3: no longer names the net of J3.20 (Pin_20)
- net RGMII_RX_CLK: no longer names the net of J3.14 (Pin_14)
- net RGMII_RX_CTL: no longer names the net of J3.18 (Pin_18)
- net RGMII_TXD0: no longer names the net of J3.7 (Pin_7)
- net RGMII_TXD1: no longer names the net of J3.8 (Pin_8)
- net RGMII_TXD2: no longer names the net of J3.6 (Pin_6)
- net RGMII_TXD3: no longer names the net of J3.11 (Pin_11)
- net RGMII_TX_CLK: no longer names the net of J3.5 (Pin_5)
- net RGMII_TX_CTL: no longer names the net of J3.13 (Pin_13)
- no-connect marks 56 -> 68

Commit message: Corrected power-up behavior
Backplane: Inverted polarity of Shutdown_Force (now Power_Enable_FPGA), to keep amps powered off until software starts: fixes #23
Backplane: Routed Shutdown_Force to unused pin 3 on RJ45 jack B to amp boards: fixes #23
Backplane: Added pull-up and pull-down resistors to fanout buffer inputs, to keep SCK & ~LDAC signals in proper state during power-on: fixes #23
Amp control: Added transistor to reset DAC & ADC from pin 3 of RJ45 jack B
Parts:
- removed C31, C34: 1uF 50V X7R, Capacitor_SMD:C_0805_2012Metric, symbol Device:C
- removed L1: 500nH, Martinos:L_Coilcraft_2929SQ-501, symbol Device:L
- removed R18: 1 0.25W, Resistor_SMD:R_2010_5025Metric, symbol Device:R
- J2: footprint Martinos:Conn_Samtec_TFM-115-x1,3-x-D-WT -> Don:Conn_Samtec_TFM-115-x1,3-x-D-WT
- J3, JA1, JA2, JB1, JB2, JC1: footprint Martinos:Conn_Samtec_TFM-120-x1,3-x-D-WT -> Don:Conn_Samtec_TFM-120-x1,3-x-D-WT
- RN1, RN2: footprint Martinos:CTS_745C -> Don:CTS_745C
- U10, U8, U9: footprint Martinos_std:VSSOP-8_2.3x2mm_P0.5mm -> Don_std:VSSOP-8_2.3x2mm_P0.5mm
- U28: footprint Martinos:Snickerdoodle -> Don:Snickerdoodle
- U4, U5: footprint Martinos_std:TSSOP-20_4.4x6.5mm_P0.65mm -> Don_std:TSSOP-20_4.4x6.5mm_P0.65mm
- U6: footprint Martinos_std:TSSOP-16_4.4x5mm_P0.65mm -> Don_std:TSSOP-16_4.4x5mm_P0.65mm
Connections:
- net VD: now also JP31.1, Q11.2 (E), Q9.2 (C), R75.2
- net Shutdown_Force renamed Power_Enable_FPGA
- net ~{Power_Enable_Sense} renamed Power_Enable_Ext_Sense
Other:
- note added: "Optional bypass"
- note removed: "22 mW @ 150 mA"
- note removed: "Noise filter, 225 kHz LPF"
- moved on the sheet: C25, C27, C35, D17, JP31, Q10, Q11, Q9, R73, R74, R75, R76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

Commit message: Misc. cleanup for mfg & improvements
Minor backplane pinout doc corrections (SCKO5 polarity, clarified some descriptions)
Backplane: Added differential- and common-mode (to standoffs) power filtering, for EMI escaping over power wiring
Amp ctrl: Changed DAC testpoints from individual pads to Keystone 5019 for easier probing
Corrected part numbers, DNP vs. non-BOM-item indications, other misc. BOM issues
Parts:
- JP13, JP14, JP15, JP16, JP17, JP18, JP19, JP20, JP21, JP22, JP23, JP25, JP26, JP27, JP28, JP30, JP31, JP32, TP12, TP13, TP52, TP53, TP62, TP63: now left out of the parts list
- Q10, Q11: Manufacturer (none) -> Diodes Inc.; Manufacturer Alt. (none) -> Nexperia; Part Number (none) -> MMBT3906-7-F; Part Number Alt. (none) -> MMBT3906,215
- R73: Part Number (none) -> RK73Z2ATTD
- R75: Part Number RK73H2ATTD4701F -> RK73H2ATTD56R0F
Changed lines of the file:
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@@
 		(unit 1)
 		(exclude_from_sim no)
-		(in_bom yes)
+		(in_bom no)
 		(on_board yes)
 		(dnp no)
@@
 		(unit 1)
 		(exclude_from_sim no)
-		(in_bom yes)
+		(in_bom no)
 		(on_board yes)
 		(dnp no)
@@
 		(unit 1)
 		(exclude_from_sim no)
-		(in_bom yes)
+		(in_bom no)
 		(on_board yes)
 		(dnp no)
@@
 		(unit 1)
 		(exclude_from_sim no)
-		(in_bom yes)
+		(in_bom no)
 		(on_board yes)
 		(dnp no)
@@
 		(unit 1)
 		(exclude_from_sim no)
-		(in_bom yes)
+		(in_bom no)
 		(on_board yes)
 		(dnp no)
@@
 		(unit 1)
 		(exclude_from_sim no)
-		(in_bom yes)
+		(in_bom no)
 		(on_board yes)
 		(dnp no)
@@
 		(unit 1)
 		(exclude_from_sim no)
-		(in_bom yes)
+		(in_bom no)
 		(on_board yes)
 		(dnp no)
@@
 		(unit 1)
 		(exclude_from_sim no)
-		(in_bom yes)
+		(in_bom no)
 		(on_board yes)
 		(dnp no)
@@
 		(unit 1)
 		(exclude_from_sim no)
-		(in_bom yes)
+		(in_bom no)
 		(on_board yes)
 		(dnp no)
@@
 		(unit 1)
 		(exclude_from_sim no)
-		(in_bom yes)
+		(in_bom no)
 		(on_board yes)
 		(dnp no)
@@
 		(unit 1)
 		(exclude_from_sim no)
-		(in_bom yes)
+		(in_bom no)
 		(on_board yes)
 		(dnp no)
@@
 		(unit 1)
 		(exclude_from_sim no)
-		(in_bom yes)
+		(in_bom no)
 		(on_board yes)
 		(dnp no)
@@
 		(unit 1)
 		(exclude_from_sim no)
-		(in_bom yes)
+		(in_bom no)
 		(on_board yes)
 		(dnp no)
@@
 		(unit 1)
 		(exclude_from_sim no)
-		(in_bom yes)
+		(in_bom no)
 		(on_board yes)
 		(dnp no)
@@
 		(unit 1)
 		(exclude_from_sim no)
-		(in_bom yes)
+		(in_bom no)
 		(on_board yes)
 		(dnp no)
@@
 		(unit 1)
 		(exclude_from_sim no)
-		(in_bom yes)
+		(in_bom no)
 		(on_board yes)
 		(dnp no)
@@
 		(unit 1)
 		(exclude_from_sim no)
-		(in_bom yes)
+		(in_bom no)
 		(on_board yes)
 		(dnp no)
@@
 		(unit 1)
 		(exclude_from_sim no)
-		(in_bom yes)
+		(in_bom no)
 		(on_board yes)
 		(dnp no)
@@
 		(unit 1)
 		(exclude_from_sim no)
-		(in_bom yes)
+		(in_bom no)
 		(on_board yes)
 		(dnp no)
@@
 		(unit 1)
 		(exclude_from_sim no)
-		(in_bom yes)
+		(in_bom no)
 		(on_board yes)
 		(dnp no)
@@
 		(unit 1)
 		(exclude_from_sim yes)
-		(in_bom yes)
+		(in_bom no)
 		(on_board yes)
 		(dnp no)
@@
 			)
 		)
-		(property "Part Number" "RK73H2ATTD4701F"
+		(property "Part Number" "RK73H2ATTD56R0F"
 			(at 364.49 115.57 0)
 			(effects
@@
 		(unit 1)
 		(exclude_from_sim no)
-		(in_bom yes)
+		(in_bom no)
 		(on_board yes)
 		(dnp no)
@@
 		(unit 1)
 		(exclude_from_sim no)
-		(in_bom yes)
+		(in_bom no)
 		(on_board yes)
 		(dnp no)
@@
 			)
 		)
-		(property "Part Number" ""
+		(property "Part Number" "RK73Z2ATTD"
 			(at 378.46 129.54 0)
 			(effects
@@
 			)
 		)
+		(property "Manufacturer" "Diodes Inc."
+			(at 369.57 132.08 0)
+			(effects
+				(font
+					(size 1.27 1.27)
+				)
+				(hide yes)
+			)
+		)
+		(property "Manufacturer Alt." "Nexperia"
+			(at 369.57 132.08 0)
+			(effects
+				(font
+					(size 1.27 1.27)
+				)
+				(hide yes)
+			)
+		)
+		(property "Part Number" "MMBT3906-7-F"
+			(at 369.57 132.08 0)
+			(effects
+				(font
+					(size 1.27 1.27)
+				)
+				(hide yes)
+			)
+		)
+		(property "Part Number Alt." "MMBT3906,215"
+			(at 369.57 132.08 0)
+			(effects
+				(font
+					(size 1.27 1.27)
+				)
+				(hide yes)
+			)
+		)
 		(pin "3"
 		)
@@
 			)
 		)
+		(property "Manufacturer" "Diodes Inc."
+			(at 351.79 119.38 0)
+			(effects
+				(font
+					(size 1.27 1.27)
+				)
+				(hide yes)
+			)
+		)
+		(property "Manufacturer Alt." "Nexperia"
+			(at 351.79 119.38 0)
+			(effects
+				(font
+					(size 1.27 1.27)
+				)
+				(hide yes)
+			)
+		)
+		(property "Part Number" "MMBT3906-7-F"
+			(at 351.79 119.38 0)
+			(effects
+				(font
+					(size 1.27 1.27)
+				)
+				(hide yes)
+			)
+		)
+		(property "Part Number Alt." "MMBT3906,215"
+			(at 351.79 119.38 0)
+			(effects
+				(font
+					(size 1.27 1.27)
+				)
+				(hide yes)
+			)
+		)
 		(pin "3"
 		)
@@
 		(unit 1)
 		(exclude_from_sim no)
-		(in_bom yes)
+		(in_bom no)
 		(on_board yes)
 		(dnp no)

Commit message: Backplane cleanup for mfg, schematic clarifications, added alt. power connectors
Parts:
- JP24, JP29: now left out of the parts list
- Q10, Q11, U34, U7: Type (none) -> SMT
- Q9: Type (none) -> Through-hole
Changed lines of the file:
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@@
 	(title_block
 		(title "FPGA Board, Signal Distribution")
-		(rev "D1")
+		(rev "D2")
 		(company "Martinos Center @ MGH")
 		(comment 1 "Don Straney")
@@
 		(unit 1)
 		(exclude_from_sim no)
-		(in_bom yes)
+		(in_bom no)
 		(on_board yes)
 		(dnp no)
@@
 		(unit 1)
 		(exclude_from_sim no)
-		(in_bom yes)
+		(in_bom no)
 		(on_board yes)
 		(dnp no)
@@
 			)
 		)
+		(property "Type" "SMT"
+			(at 240.03 113.03 0)
+			(effects
+				(font
+					(size 1.27 1.27)
+				)
+				(hide yes)
+			)
+		)
 		(pin "3"
 		)
@@
 			)
 		)
+		(property "Type" "Through-hole"
+			(at 382.27 114.3 0)
+			(effects
+				(font
+					(size 1.27 1.27)
+				)
+				(hide yes)
+			)
+		)
 		(pin "2"
 		)
@@
 			)
 		)
+		(property "Type" "SMT"
+			(at 369.57 132.08 0)
+			(effects
+				(font
+					(size 1.27 1.27)
+				)
+				(hide yes)
+			)
+		)
 		(pin "3"
 		)
@@
 			)
 		)
+		(property "Type" "SMT"
+			(at 351.79 119.38 0)
+			(effects
+				(font
+					(size 1.27 1.27)
+				)
+				(hide yes)
+			)
+		)
 		(pin "3"
 		)
@@
 			(at 285.75 220.98 0)
 			(effects
+				(font
+					(size 1.27 1.27)
+				)
+				(hide yes)
+			)
+		)
+		(property "Type" "SMT"
+			(at 285.75 220.98 0)
+			(effects

Commit message: Moved all project-specific symbols & footprints into new "shim" libraries Updated projects to reference the new "shim" library
Parts:
- D17: footprint Don_std:D_SOD-323F -> shim:D_SOD-323F
- J2: footprint Don:Conn_Samtec_TFM-115-x1,3-x-D-WT -> shim:Conn_Samtec_TFM-115-x1,3-x-D-WT
- J3, JA1, JA2, JB1, JB2, JC1: footprint Don:Conn_Samtec_TFM-120-x1,3-x-D-WT -> shim:Conn_Samtec_TFM-120-x1,3-x-D-WT
- RN1, RN2: footprint Don:CTS_745C -> shim:CTS_745C
- U10, U8, U9: footprint Don_std:VSSOP-8_2.3x2mm_P0.5mm -> Package_SO:VSSOP-8_2.3x2mm_P0.5mm
- U28: footprint Don:Snickerdoodle -> shim:Snickerdoodle
- U34: footprint Don_std:SOIC-8_3.9x4.9mm_P1.27mm -> Package_SO:SOIC-8_3.9x4.9mm_P1.27mm; symbol Don:ICS501 -> shim:ICS501
- U4, U5: footprint Don_std:TSSOP-20_4.4x6.5mm_P0.65mm -> Package_SO:TSSOP-20_4.4x6.5mm_P0.65mm
- U6: footprint Don_std:TSSOP-16_4.4x5mm_P0.65mm -> Package_SO:TSSOP-16_4.4x5mm_P0.65mm
Changed lines of the file:
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@@
 			)
 		)
-		(property "Footprint" "Don:Conn_Samtec_TFM-115-x1,3-x-D-WT"
+		(property "Footprint" "shim:Conn_Samtec_TFM-115-x1,3-x-D-WT"
 			(at 384.81 50.8 0)
 			(effects
@@
 			)
 		)
-		(property "Footprint" "Don:Conn_Samtec_TFM-120-x1,3-x-D-WT"
+		(property "Footprint" "shim:Conn_Samtec_TFM-120-x1,3-x-D-WT"
 			(at 53.34 55.88 0)
 			(effects
@@
 			)
 		)
-		(property "Footprint" "Don:Conn_Samtec_TFM-120-x1,3-x-D-WT"
+		(property "Footprint" "shim:Conn_Samtec_TFM-120-x1,3-x-D-WT"
 			(at 109.22 55.88 0)
 			(effects
@@
 			)
 		)
-		(property "Footprint" "Don:Conn_Samtec_TFM-120-x1,3-x-D-WT"
+		(property "Footprint" "shim:Conn_Samtec_TFM-120-x1,3-x-D-WT"
 			(at 165.1 55.88 0)
 			(effects
@@
 			)
 		)
-		(property "Footprint" "Don:Conn_Samtec_TFM-120-x1,3-x-D-WT"
+		(property "Footprint" "shim:Conn_Samtec_TFM-120-x1,3-x-D-WT"
 			(at 220.98 55.88 0)
 			(effects
@@
 			)
 		)
-		(property "Footprint" "Don:Conn_Samtec_TFM-120-x1,3-x-D-WT"
+		(property "Footprint" "shim:Conn_Samtec_TFM-120-x1,3-x-D-WT"
 			(at 276.86 55.88 0)
 			(effects
@@
 			)
 		)
-		(property "Footprint" "Don:Conn_Samtec_TFM-120-x1,3-x-D-WT"
+		(property "Footprint" "shim:Conn_Samtec_TFM-120-x1,3-x-D-WT"
 			(at 332.74 55.88 0)
 			(effects
@@
 			)
 		)
-		(property "Footprint" "Don:CTS_745C"
+		(property "Footprint" "shim:CTS_745C"
 			(at 177.8 136.525 90)
 			(effects
@@
 			)
 		)
-		(property "Footprint" "Don_std:VSSOP-8_2.3x2mm_P0.5mm"
+		(property "Footprint" "Package_SO:VSSOP-8_2.3x2mm_P0.5mm"
 			(at 265.43 187.96 0)
 			(effects
@@
 			)
 		)
-		(property "Footprint" "Don_std:TSSOP-16_4.4x5mm_P0.65mm"
+		(property "Footprint" "Package_SO:TSSOP-16_4.4x5mm_P0.65mm"
 			(at 170.18 232.41 0)
 			(effects
@@
 			)
 		)
-		(property "Footprint" "Don_std:TSSOP-20_4.4x6.5mm_P0.65mm"
+		(property "Footprint" "Package_SO:TSSOP-20_4.4x6.5mm_P0.65mm"
 			(at 86.36 168.91 0)
 			(effects
@@
 			)
 		)
-		(property "Footprint" "Don_std:TSSOP-20_4.4x6.5mm_P0.65mm"
+		(property "Footprint" "Package_SO:TSSOP-20_4.4x6.5mm_P0.65mm"
 			(at 149.86 168.91 0)
 			(effects
@@
 			)
 		)
-		(property "Footprint" "Don:CTS_745C"
+		(property "Footprint" "shim:CTS_745C"
 			(at 177.8 167.005 90)
 			(effects
@@
 			)
 		)
-		(property "Footprint" "Don_std:VSSOP-8_2.3x2mm_P0.5mm"
+		(property "Footprint" "Package_SO:VSSOP-8_2.3x2mm_P0.5mm"
 			(at 325.12 187.96 0)
 			(effects
@@
 			)
 		)
-		(property "Footprint" "Don_std:VSSOP-8_2.3x2mm_P0.5mm"
+		(property "Footprint" "Package_SO:VSSOP-8_2.3x2mm_P0.5mm"
 			(at 325.12 237.49 0)
 			(effects
@@
 			)
 		)
-		(property "Footprint" "Don:Snickerdoodle"
+		(property "Footprint" "shim:Snickerdoodle"
 			(at 222.25 12.7 0)
 			(effects
@@
 			)
 		)
-		(property "Footprint" "Don_std:D_SOD-323F"
+		(property "Footprint" "shim:D_SOD-323F"
 			(at 382.27 133.35 0)
 			(effects
@@
 	)
 	(symbol
-		(lib_id "Don:ICS501")
+		(lib_id "shim:ICS501")
 		(at 285.75 220.98 0)
 		(unit 1)
@@
 			)
 		)
-		(property "Footprint" "Don_std:SOIC-8_3.9x4.9mm_P1.27mm"
+		(property "Footprint" "Package_SO:SOIC-8_3.9x4.9mm_P1.27mm"
 			(at 287.02 220.98 0)
 			(effects
