File: pcbs/backplane/backplane.kicad_pcb (KiCad board)
At the start: 6 copper layers, 145 x 355 mm, 392 parts, among them J1 Conn_01x02, J10 AFBR-2624Z, J11 AFBR-2624Z, J12 AFBR-1624Z, J13 RJ45_Shielded, J14 Conn_01x02, J15 RJ45_Shielded, J16 RJ45_Shielded, J17 Conn_01x02, J18 RJ45_Shielded, J19 Conn_01x02, J2 Conn_02x15_Odd_Even, J20 RJ45_Shielded, J21 RJ45_Shielded, J22 Conn_01x02, J23 RJ45_Shielded, J24 Conn_01x02, J25 RJ45_Shielded, J26 RJ45_Shielded, J27 Conn_01x02, J28 RJ45_Shielded, J29 Conn_01x02, J3 Conn_02x20_Odd_Even, J30 RJ45_Shielded, J31 RJ45_Shielded, J32 Conn_01x02, J33 RJ45_Shielded, J34 Conn_01x02, J35 RJ45_Shielded, J36 RJ45_Shielded, J37 Conn_01x02, J38 RJ45_Shielded, J39 Conn_01x02, J4 RJ45_Shielded, J40 RJ45_Shielded, J41 RJ45_Shielded, J42 Conn_01x02, J43 RJ45_Shielded, J44 Conn_01x02, J45 RJ45_Shielded, J46 RJ45_Shielded, J47 Conn_01x02, J48 Conn_01x02, J5 AFBR-2624Z, J6 RJ45_Shielded, J7 RJ45_Shielded, J8 Conn_01x02, J9 AFBR-2624Z, Q1 MMBT3904, Q10 MMBT3906, Q11 MMBT3906, Q12 MMBT3904, Q13 MMBT3904, Q2 MMBT3904, Q3 MMBT3904, Q4 MMBT3904, Q5 MMBT3904, Q6 MMBT3904, Q7 MMBT3904, Q8 MMBT3904, Q9 D44H11G, U1 74LVC1G14, U10 74LVC2T45, U12 74LVC1G14, U13 74LVC2G02, U14 74LVC1G14, U15 74LVC2G02, U16 74LVC2G02, U17 74LVC1G14, U18 74LVC2G02, U19 74LVC1G14, U2 CDCUN1208LP, U20 74LVC2G02, U21 74LVC1G14, U22 74LVC2G02, U23 74LVC1G14, U24 74LVC2G02, U25 74LVC1G14, U26 74LVC2G02, U27 74LVC1G14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

Commit message: Backplane comms updates, manufacturing renaming
Removed misspelled "maunfacturing" folder, fixed gitignore rule to remove manufacturing folders within individual PCB folders too
Changed SCKI/SCKO terminology to SCK, SCK_LB (loopback) for clarity
Added ADC_CS loopback signal between amp ctrl board & backplane for better fast-clock timing (#38)
Backplane: changed LVDS FPGA outputs to single-ended FPGA outputs to gain more I/O pins, added external LVDS transceivers (#38)
Backplane: replaced global clock & ~LDAC buffers with a separate FPGA pin for each amp ctrl board (#38)
Backplane: removed +2.5V power supply and level translations, no longer needed without FPGA I/O pins using LVDS_25 I/O configuration
Backplane: replaced +VDC-input resistor with solder jumper (on by default)
Backplane: changed field names (Part Number to MPN) to match Aisler's naming convention for automatic recognition
Amp ctrl: fixed optional level-shifter circuit on each channel for voltage inputs (#9) schematic & channel-1 layout
Parts:
- removed C14, C15, C29, C30: 100nF 50V X7R, Capacitor_SMD:C_0603_1608Metric
- removed C25, C27, C36, C37: 1uF 50V X7R, Capacitor_SMD:C_0805_2012Metric
- removed D5: Green, LED_SMD:LED_0805_2012Metric
- removed JP34: Jumper_NC_Small, Jumper:SolderJumper-2_P1.3mm_Bridged_RoundedPad1.0x1.5mm
- removed R1, R2: 100, Resistor_SMD:R_0402_1005Metric
- removed R12: 560, Resistor_SMD:R_0805_2012Metric
- removed R5: 1 0.25W, Resistor_SMD:R_2010_5025Metric
- removed R84, R85, R86, R87: 10K, Resistor_SMD:R_0402_1005Metric
- removed R88: 20K, Resistor_SMD:R_0805_2012Metric
- removed R89: 10K, Resistor_SMD:R_0805_2012Metric
- removed TP11, TP16, TP31, TP36, TP41, TP46, TP53, TP62: TestPoint, TestPoint:TestPoint_Pad_D2.0mm
- removed TP7: TestPoint_Flag, TestPoint:TestPoint_Keystone_5019_Miniature
- removed U7: AP7361C-25E, Package_TO_SOT_SMD:SOT-223-3_TabPin2
- removed U9: 74LVC2T45, Package_SO:VSSOP-8_2.3x2mm_P0.5mm
- added C100: 1uF 16V X7R, Capacitor_SMD:C_0603_1608Metric, F.Cu at (107.0, 87.2)
- added C101: 1uF 16V X7R, Capacitor_SMD:C_0603_1608Metric, F.Cu at (156.7, 139.0)
- added C102: 1uF 16V X7R, Capacitor_SMD:C_0603_1608Metric, F.Cu at (113.5, 28.2)
- added C103: 1uF 16V X7R, Capacitor_SMD:C_0603_1608Metric, F.Cu at (156.7, 80.0)
- added C104: 22pF 50V NP0, shim:C_Array_0612_1632Metric, F.Cu at (102.1, 339.6)
- added C105: 22pF 50V NP0, shim:C_Array_0612_1632Metric, F.Cu at (156.7, 352.4)
- added C106: 22pF 50V NP0, shim:C_Array_0612_1632Metric, F.Cu at (100.1, 165.9)
- added C107: 22pF 50V NP0, shim:C_Array_0612_1632Metric, F.Cu at (156.7, 178.3)
- added C108: 22pF 50V NP0, shim:C_Array_0612_1632Metric, F.Cu at (107.1, 106.9)
- added C109: 22pF 50V NP0, shim:C_Array_0612_1632Metric, F.Cu at (156.7, 119.3)
- added C110: 22pF 50V NP0, shim:C_Array_0612_1632Metric, F.Cu at (113.6, 47.9)
- added C111: 22pF 50V NP0, shim:C_Array_0612_1632Metric, F.Cu at (156.7, 60.4)
- added C112: 22pF 50V NP0, shim:C_Array_0612_1632Metric, F.Cu at (102.3, 325.6)
- added C113: 22pF 50V NP0, shim:C_Array_0612_1632Metric, F.Cu at (156.4, 366.4)
- added C114: 22pF 50V NP0, shim:C_Array_0612_1632Metric, F.Cu at (100.3, 151.9)
- added C115: 22pF 50V NP0, shim:C_Array_0612_1632Metric, F.Cu at (156.4, 192.3)
- added C116: 22pF 50V NP0, shim:C_Array_0612_1632Metric, F.Cu at (107.3, 92.9)
- added C117: 22pF 50V NP0, shim:C_Array_0612_1632Metric, F.Cu at (156.4, 133.3)
- added C118: 22pF 50V NP0, shim:C_Array_0612_1632Metric, F.Cu at (113.8, 33.9)
- added C119: 22pF 50V NP0, shim:C_Array_0612_1632Metric, F.Cu at (156.4, 74.3)
- added C80: 1uF 16V X7R, Capacitor_SMD:C_0603_1608Metric, F.Cu at (101.0, 333.2)
- added C81: 1uF 16V X7R, Capacitor_SMD:C_0603_1608Metric, F.Cu at (157.8, 358.8)
- added C82: 1uF 16V X7R, Capacitor_SMD:C_0603_1608Metric, F.Cu at (99.0, 159.5)
- added C83: 1uF 16V X7R, Capacitor_SMD:C_0603_1608Metric, F.Cu at (157.8, 184.8)
- added C84: 1uF 16V X7R, Capacitor_SMD:C_0603_1608Metric, F.Cu at (106.0, 100.5)
- added C85: 1uF 16V X7R, Capacitor_SMD:C_0603_1608Metric, F.Cu at (157.8, 125.8)
- added C86: 1uF 16V X7R, Capacitor_SMD:C_0603_1608Metric, F.Cu at (112.5, 41.5)
- added C87: 1uF 16V X7R, Capacitor_SMD:C_0603_1608Metric, F.Cu at (157.8, 66.8)
- added C88: 1uF 16V X7R, Capacitor_SMD:C_0603_1608Metric, F.Cu at (101.8, 328.8)
- added C89: 1uF 16V X7R, Capacitor_SMD:C_0603_1608Metric, F.Cu at (157.0, 363.2)
- added C90: 1uF 16V X7R, Capacitor_SMD:C_0603_1608Metric, F.Cu at (99.8, 155.0)
- added C91: 1uF 16V X7R, Capacitor_SMD:C_0603_1608Metric, F.Cu at (157.0, 189.2)
- added C92: 1uF 16V X7R, Capacitor_SMD:C_0603_1608Metric, F.Cu at (106.8, 96.0)
- added C93: 1uF 16V X7R, Capacitor_SMD:C_0603_1608Metric, F.Cu at (157.0, 130.2)
- added C94: 1uF 16V X7R, Capacitor_SMD:C_0603_1608Metric, F.Cu at (113.2, 37.0)
- added C95: 1uF 16V X7R, Capacitor_SMD:C_0603_1608Metric, F.Cu at (157.0, 71.2)
- added C96: 1uF 16V X7R, Capacitor_SMD:C_0603_1608Metric, F.Cu at (102.0, 320.0)
- added C97: 1uF 16V X7R, Capacitor_SMD:C_0603_1608Metric, F.Cu at (156.7, 372.0)
- added C98: 1uF 16V X7R, Capacitor_SMD:C_0603_1608Metric, F.Cu at (100.0, 146.2)
- added C99: 1uF 16V X7R, Capacitor_SMD:C_0603_1608Metric, F.Cu at (156.7, 198.0)
- added JP35: Jumper_2_Open, Jumper:SolderJumper-2_P1.3mm_Open_RoundedPad1.0x1.5mm, B.Cu at (104.0, 119.8)
- added JP36: Jumper_2_Open, Jumper:SolderJumper-2_P1.3mm_Open_RoundedPad1.0x1.5mm, B.Cu at (159.8, 106.4)
- added JP37: Jumper_2_Open, Jumper:SolderJumper-2_P1.3mm_Open_RoundedPad1.0x1.5mm, B.Cu at (110.5, 60.9)
- added JP38: Jumper_2_Open, Jumper:SolderJumper-2_P1.3mm_Open_RoundedPad1.0x1.5mm, B.Cu at (159.8, 47.4)
- added JP39: Jumper_2_Bridged, Jumper:SolderJumper-2_P1.3mm_Bridged_RoundedPad1.0x1.5mm, B.Cu at (95.2, 349.5)
- added JP40: Jumper_2_Bridged, Jumper:SolderJumper-2_P1.3mm_Bridged_RoundedPad1.0x1.5mm, B.Cu at (163.5, 342.5)
- added JP41: Jumper_2_Bridged, Jumper:SolderJumper-2_P1.3mm_Bridged_RoundedPad1.0x1.5mm, B.Cu at (93.2, 175.8)
- added JP42: Jumper_2_Bridged, Jumper:SolderJumper-2_P1.3mm_Bridged_RoundedPad1.0x1.5mm, B.Cu at (163.5, 168.5)
- added JP43: Jumper_2_Bridged, Jumper:SolderJumper-2_P1.3mm_Bridged_RoundedPad1.0x1.5mm, B.Cu at (100.2, 116.8)
- added JP44: Jumper_2_Bridged, Jumper:SolderJumper-2_P1.3mm_Bridged_RoundedPad1.0x1.5mm, B.Cu at (163.5, 109.5)
- added JP45: Jumper_2_Bridged, Jumper:SolderJumper-2_P1.3mm_Bridged_RoundedPad1.0x1.5mm, B.Cu at (106.8, 57.8)
- added JP46: Jumper_2_Bridged, Jumper:SolderJumper-2_P1.3mm_Bridged_RoundedPad1.0x1.5mm, B.Cu at (163.5, 50.5)
- added JP47: Jumper_2_Bridged, Jumper:SolderJumper-2_P1.3mm_Bridged_RoundedPad1.0x1.5mm, B.Cu at (97.8, 349.6)
- added JP48: Jumper_2_Bridged, Jumper:SolderJumper-2_P1.3mm_Bridged_RoundedPad1.0x1.5mm, B.Cu at (161.0, 342.4)
- added JP49: Jumper_2_Bridged, Jumper:SolderJumper-2_P1.3mm_Bridged_RoundedPad1.0x1.5mm, B.Cu at (95.8, 175.8)
- added JP50: Jumper_2_Bridged, Jumper:SolderJumper-2_P1.3mm_Bridged_RoundedPad1.0x1.5mm, B.Cu at (161.0, 168.4)
- added JP51: Jumper_2_Bridged, Jumper:SolderJumper-2_P1.3mm_Bridged_RoundedPad1.0x1.5mm, B.Cu at (102.8, 116.8)
- added JP52: Jumper_2_Bridged, Jumper:SolderJumper-2_P1.3mm_Bridged_RoundedPad1.0x1.5mm, B.Cu at (161.0, 109.4)
- added JP53: Jumper_2_Bridged, Jumper:SolderJumper-2_P1.3mm_Bridged_RoundedPad1.0x1.5mm, B.Cu at (109.2, 57.9)
- added JP54: Jumper_2_Bridged, Jumper:SolderJumper-2_P1.3mm_Bridged_RoundedPad1.0x1.5mm, B.Cu at (161.0, 50.4)
- added JP55: Jumper_2_Bridged, Jumper:SolderJumper-2_P1.3mm_Bridged_RoundedPad1.0x1.5mm, F.Cu at (52.2, 32.0)
- added RN10: 100 5%, Resistor_SMD:R_Array_Concave_4x0603, F.Cu at (114.2, 58.2)
- added RN11: 100 5%, Resistor_SMD:R_Array_Concave_4x0603, F.Cu at (156.0, 50.0)
- added RN12: 100 5%, Resistor_SMD:R_Array_Concave_4x0603, F.Cu at (100.8, 343.6)
- added RN13: 100 5%, Resistor_SMD:R_Array_Concave_4x0603, F.Cu at (158.0, 348.4)
- added RN14: 100 5%, Resistor_SMD:R_Array_Concave_4x0603, F.Cu at (98.8, 169.9)
- added RN15: 100 5%, Resistor_SMD:R_Array_Concave_4x0603, F.Cu at (158.0, 174.3)
- added RN16: 100 5%, Resistor_SMD:R_Array_Concave_4x0603, F.Cu at (105.8, 110.9)
- added RN17: 100 5%, Resistor_SMD:R_Array_Concave_4x0603, F.Cu at (158.0, 115.3)
- added RN18: 100 5%, Resistor_SMD:R_Array_Concave_4x0603, F.Cu at (112.2, 51.9)
- added RN19: 100 5%, Resistor_SMD:R_Array_Concave_4x0603, F.Cu at (158.0, 56.4)
- added RN20: 100 5%, Resistor_SMD:R_Array_Concave_4x0603, F.Cu at (102.1, 336.4)
- added RN21: 100 5%, Resistor_SMD:R_Array_Concave_4x0603, F.Cu at (156.7, 355.6)
- added RN22: 100 5%, Resistor_SMD:R_Array_Concave_4x0603, F.Cu at (100.1, 162.7)
- added RN23: 100 5%, Resistor_SMD:R_Array_Concave_4x0603, F.Cu at (156.7, 181.6)
- added RN24: 100 5%, Resistor_SMD:R_Array_Concave_4x0603, F.Cu at (107.1, 103.7)
- added RN25: 100 5%, Resistor_SMD:R_Array_Concave_4x0603, F.Cu at (156.7, 122.6)
- added RN26: 100 5%, Resistor_SMD:R_Array_Concave_4x0603, F.Cu at (113.6, 44.6)
- added RN27: 100 5%, Resistor_SMD:R_Array_Concave_4x0603, F.Cu at (156.7, 63.6)
- added RN28: 100 5%, Resistor_SMD:R_Array_Concave_4x0603, F.Cu at (102.3, 322.4)
- added RN29: 100 5%, Resistor_SMD:R_Array_Concave_4x0603, F.Cu at (156.4, 369.6)
- added RN30: 100 5%, Resistor_SMD:R_Array_Concave_4x0603, F.Cu at (100.3, 148.7)
- added RN31: 100 5%, Resistor_SMD:R_Array_Concave_4x0603, F.Cu at (156.4, 195.6)
- added RN32: 100 5%, Resistor_SMD:R_Array_Concave_4x0603, F.Cu at (107.3, 89.7)
- added RN33: 100 5%, Resistor_SMD:R_Array_Concave_4x0603, F.Cu at (156.4, 136.6)
- added RN34: 100 5%, Resistor_SMD:R_Array_Concave_4x0603, F.Cu at (113.8, 30.6)
- added RN35: 100 5%, Resistor_SMD:R_Array_Concave_4x0603, F.Cu at (156.4, 77.6)
- added RN4: 100 5%, Resistor_SMD:R_Array_Concave_4x0603, F.Cu at (102.8, 350.0)
- added RN5: 100 5%, Resistor_SMD:R_Array_Concave_4x0603, F.Cu at (156.0, 342.0)
- added RN6: 100 5%, Resistor_SMD:R_Array_Concave_4x0603, F.Cu at (100.8, 176.2)
- added RN7: 100 5%, Resistor_SMD:R_Array_Concave_4x0603, F.Cu at (156.0, 168.0)
- added RN8: 100 5%, Resistor_SMD:R_Array_Concave_4x0603, F.Cu at (107.8, 117.2)
- added RN9: 100 5%, Resistor_SMD:R_Array_Concave_4x0603, F.Cu at (156.0, 109.0)
- added TP24: TestPoint, TestPoint:TestPoint_Pad_D2.0mm, F.Cu at (170.8, 224.8)
- added TP25: TestPoint, TestPoint:TestPoint_Pad_D2.0mm, F.Cu at (171.0, 231.2)
- added TP27: TestPoint, TestPoint:TestPoint_Pad_D2.0mm, F.Cu at (82.3, 281.5)
- added U50: FIN1027, Package_SO:SOIC-8_3.9x4.9mm_P1.27mm, F.Cu at (95.5, 164.0)
- added U51: FIN1027, Package_SO:SOIC-8_3.9x4.9mm_P1.27mm, F.Cu at (161.2, 180.2)
- added U52: FIN1027, Package_SO:SOIC-8_3.9x4.9mm_P1.27mm, F.Cu at (102.5, 105.0)
- added U53: FIN1027, Package_SO:SOIC-8_3.9x4.9mm_P1.27mm, F.Cu at (161.2, 121.2)
- added U54: FIN1027, Package_SO:SOIC-8_3.9x4.9mm_P1.27mm, F.Cu at (109.0, 46.0)
- added U55: FIN1027, Package_SO:SOIC-8_3.9x4.9mm_P1.27mm, F.Cu at (161.2, 62.2)
- added U56: FIN1027, Package_SO:SOIC-8_3.9x4.9mm_P1.27mm, F.Cu at (97.5, 330.3)
- added U57: FIN1027, Package_SO:SOIC-8_3.9x4.9mm_P1.27mm, F.Cu at (161.2, 361.7)
- added U58: FIN1027, Package_SO:SOIC-8_3.9x4.9mm_P1.27mm, F.Cu at (95.5, 156.5)
- added U59: FIN1027, Package_SO:SOIC-8_3.9x4.9mm_P1.27mm, F.Cu at (161.2, 187.7)
- added U60: FIN1027, Package_SO:SOIC-8_3.9x4.9mm_P1.27mm, F.Cu at (102.5, 97.5)
- added U61: FIN1027, Package_SO:SOIC-8_3.9x4.9mm_P1.27mm, F.Cu at (161.2, 128.7)
- added U62: FIN1027, Package_SO:SOIC-8_3.9x4.9mm_P1.27mm, F.Cu at (109.0, 38.5)
- added U63: FIN1027, Package_SO:SOIC-8_3.9x4.9mm_P1.27mm, F.Cu at (161.2, 69.7)
- added U64: FIN1027, Package_SO:SOIC-8_3.9x4.9mm_P1.27mm, F.Cu at (97.6, 322.7)
- added U65: FIN1027, Package_SO:SOIC-8_3.9x4.9mm_P1.27mm, F.Cu at (161.2, 369.3)
- added U66: FIN1027, Package_SO:SOIC-8_3.9x4.9mm_P1.27mm, F.Cu at (95.6, 148.9)
- added U67: FIN1027, Package_SO:SOIC-8_3.9x4.9mm_P1.27mm, F.Cu at (161.2, 195.3)
- added U68: FIN1027, Package_SO:SOIC-8_3.9x4.9mm_P1.27mm, F.Cu at (102.6, 89.9)
- added U69: FIN1027, Package_SO:SOIC-8_3.9x4.9mm_P1.27mm, F.Cu at (161.2, 136.3)
- added U70: FIN1027, Package_SO:SOIC-8_3.9x4.9mm_P1.27mm, F.Cu at (109.1, 30.9)
- added U71: FIN1027, Package_SO:SOIC-8_3.9x4.9mm_P1.27mm, F.Cu at (161.2, 77.3)
- added U72: FIN1048, Package_SO:TSSOP-16_4.4x5mm_P0.65mm, F.Cu at (98.0, 349.9)
- added U73: FIN1048, Package_SO:TSSOP-16_4.4x5mm_P0.65mm, F.Cu at (160.7, 342.1)
- added U74: FIN1048, Package_SO:TSSOP-16_4.4x5mm_P0.65mm, F.Cu at (96.0, 176.1)
- added U75: FIN1048, Package_SO:TSSOP-16_4.4x5mm_P0.65mm, F.Cu at (160.7, 168.1)
- added U76: FIN1048, Package_SO:TSSOP-16_4.4x5mm_P0.65mm, F.Cu at (103.0, 117.1)
- added U77: FIN1048, Package_SO:TSSOP-16_4.4x5mm_P0.65mm, F.Cu at (160.7, 109.1)
- added U78: FIN1048, Package_SO:TSSOP-16_4.4x5mm_P0.65mm, F.Cu at (109.5, 58.1)
- added U79: FIN1048, Package_SO:TSSOP-16_4.4x5mm_P0.65mm, F.Cu at (160.7, 50.1)
- C11, C12, C13, C5, C6, C7, C8, C9: value 100nF 50V X7R -> 1uF 16V X7R
- JP1, JP7: value Jumper_NO_Small -> Jumper_2_Open; footprint Jumper:SolderJumper-2_P1.3mm_Open_TrianglePad1.0x1.5mm -> Jumper:SolderJumper-2_P1.3mm_Open_RoundedPad1.0x1.5mm
- JP10, JP3, JP4, JP9: value Jumper_NC_Small -> Jumper_2_Open; footprint Jumper:SolderJumper-2_P1.3mm_Bridged_RoundedPad1.0x1.5mm -> Jumper:SolderJumper-2_P1.3mm_Open_RoundedPad1.0x1.5mm; moved to B.Cu
- JP11, JP12, JP2, JP5, JP6, JP8: value Jumper_NC_Small -> Jumper_2_Open; footprint Jumper:SolderJumper-2_P1.3mm_Bridged_RoundedPad1.0x1.5mm -> Jumper:SolderJumper-2_P1.3mm_Open_RoundedPad1.0x1.5mm
- U2, U3: value CDCUN1208LP -> FIN1027; footprint shim:VQFN-32-1EP_5x5mm_P0.5mm_EP3.45x3.45mm -> Package_SO:SOIC-8_3.9x4.9mm_P1.27mm
- moved TP23 259.3 mm to (127.2, 372.8), turned to 0 degrees
- moved JP8 240.3 mm to (162.2, 47.4), turned to 90 degrees
- moved C13 222.9 mm to (161.5, 54.8), turned to 0 degrees
- moved JP7 222.6 mm to (108.0, 60.9), turned to -90 degrees
- moved C12 220.3 mm to (108.8, 53.5), turned to 180 degrees
- moved C11 167.1 mm to (161.5, 113.8)
- moved JP6 163.2 mm to (162.2, 106.4), turned to 90 degrees
- moved C9 156.2 mm to (102.2, 112.5), turned to 180 degrees
- moved JP5 150.3 mm to (101.5, 119.8), turned to -90 degrees
- moved JP12 120.7 mm to (159.8, 165.4), turned to 90 degrees
- moved JP11 107.7 mm to (97.0, 178.8), turned to -90 degrees
- moved C8 102.5 mm to (161.5, 172.8), turned to 0 degrees
- moved JP4 101.7 mm to (162.2, 165.4), turned to 90 degrees
- moved C6 97.0 mm to (161.5, 346.8), turned to 0 degrees
- moved JP3 92.4 mm to (94.5, 178.8), turned to -90 degrees
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Connections:
- C1 pad 1: +2.5V -> +3V3
- C11 pad 1: +3V3 -> GND
- C11 pad 2: GND -> +3V3
- C12 pad 1: +3V3 -> GND
- C12 pad 2: GND -> +3V3
- C13 pad 1: +3V3 -> GND
- C13 pad 2: GND -> +3V3
- C24 pad 1: +2.5V -> +3V3
- C38 pad 1: +2.5V -> +3V3
- C39 pad 2: +2.5V -> +3V3
- C40 pad 1: +2.5V -> +3V3
- C41 pad 1: +2.5V -> +3V3
- C42 pad 2: +2.5V -> +3V3
- C43 pad 1: +2.5V -> +3V3
- C44 pad 1: +2.5V -> +3V3
- C45 pad 2: +2.5V -> +3V3
- C46 pad 1: +2.5V -> +3V3
- C47 pad 1: +2.5V -> +3V3
- C48 pad 2: +2.5V -> +3V3
- C49 pad 1: +2.5V -> +3V3
- C5 pad 1: +3V3 -> GND
- C5 pad 2: GND -> +3V3
- C50 pad 1: +2.5V -> +3V3
- C51 pad 2: +2.5V -> +3V3
- C52 pad 1: +2.5V -> +3V3
- C53 pad 1: +2.5V -> +3V3
- C54 pad 2: +2.5V -> +3V3
- C55 pad 1: +2.5V -> +3V3
- C56 pad 1: +2.5V -> +3V3
- C57 pad 2: +2.5V -> +3V3
- C58 pad 1: +2.5V -> +3V3
- C59 pad 1: +2.5V -> +3V3
- C6 pad 1: +3V3 -> GND
- C6 pad 2: GND -> +3V3
- C60 pad 2: +2.5V -> +3V3
- C7 pad 1: +3V3 -> GND
- C7 pad 2: GND -> +3V3
- C8 pad 1: +3V3 -> GND
- C8 pad 2: GND -> +3V3
- C9 pad 1: +3V3 -> GND
- C9 pad 2: GND -> +3V3
- J13 pad 1: /Amp board 1 interface/~{Shutdown} -> /Amp board 1 interface/~{ADC_CS_LB-}
- J13 pad 2: GND -> /Amp board 1 interface/~{ADC_CS_LB+}
- J13 pad 4: /ADC_MOSI+1 -> /Amp board 1 interface/ADC_MOSI+
- J13 pad 5: /ADC_MOSI-1 -> /Amp board 1 interface/ADC_MOSI-
- J13 pad 7: /~{ADC_CS+1} -> /Amp board 1 interface/~{ADC_CS+}
- J13 pad 8: /~{ADC_CS-1} -> /Amp board 1 interface/~{ADC_CS-}
- J15 pad 1: /DAC_MISO-1 -> /Amp board 1 interface/DAC_MISO-
- J15 pad 2: /DAC_MISO+1 -> /Amp board 1 interface/DAC_MISO+
- J15 pad 4: /SCKO-1 -> /Amp board 1 interface/SCK_LB-
- J15 pad 5: /SCKO+1 -> /Amp board 1 interface/SCK_LB+
- J15 pad 6: unconnected-(J15-Pad6) -> /Amp board 1 interface/~{Shutdown}
- J15 pad 7: /ADC_MISO-1 -> /Amp board 1 interface/ADC_MISO-
- J15 pad 8: /ADC_MISO+1 -> /Amp board 1 interface/ADC_MISO+
- J16 pad 1: /SCKI-1 -> /Amp board 1 interface/SCK-
- J16 pad 2: /SCKI+1 -> /Amp board 1 interface/SCK+
- J16 pad 3: /~{DAC_CS-1} -> /Amp board 1 interface/~{DAC_CS-}
- J16 pad 4: /DAC_MOSI-1 -> /Amp board 1 interface/DAC_MOSI-
- J16 pad 5: /DAC_MOSI+1 -> /Amp board 1 interface/DAC_MOSI+
- J16 pad 6: /~{DAC_CS+1} -> /Amp board 1 interface/~{DAC_CS+}
- J16 pad 7: /~{LDAC-1} -> /Amp board 1 interface/~{LDAC-}
- J16 pad 8: /~{LDAC+1} -> /Amp board 1 interface/~{LDAC+}
- J18 pad 1: /Amp board 2 interface/~{Shutdown} -> /Amp board 2 interface/~{ADC_CS_LB-}
- J18 pad 2: GND -> /Amp board 2 interface/~{ADC_CS_LB+}
- J18 pad 4: /ADC_MOSI+2 -> /Amp board 2 interface/ADC_MOSI+
- J18 pad 5: /ADC_MOSI-2 -> /Amp board 2 interface/ADC_MOSI-
- J18 pad 7: /~{ADC_CS+2} -> /Amp board 2 interface/~{ADC_CS+}
- J18 pad 8: /~{ADC_CS-2} -> /Amp board 2 interface/~{ADC_CS-}
- J20 pad 1: /DAC_MISO-2 -> /Amp board 2 interface/DAC_MISO-
- J20 pad 2: /DAC_MISO+2 -> /Amp board 2 interface/DAC_MISO+
- J20 pad 4: /SCKO-2 -> /Amp board 2 interface/SCK_LB-
- J20 pad 5: /SCKO+2 -> /Amp board 2 interface/SCK_LB+
- J20 pad 6: unconnected-(J20-Pad6) -> /Amp board 2 interface/~{Shutdown}
- J20 pad 7: /ADC_MISO-2 -> /Amp board 2 interface/ADC_MISO-
- J20 pad 8: /ADC_MISO+2 -> /Amp board 2 interface/ADC_MISO+
- J21 pad 1: /SCKI-2 -> /Amp board 2 interface/SCK-
- J21 pad 2: /SCKI+2 -> /Amp board 2 interface/SCK+
- J21 pad 3: /~{DAC_CS-2} -> /Amp board 2 interface/~{DAC_CS-}
- J21 pad 4: /DAC_MOSI-2 -> /Amp board 2 interface/DAC_MOSI-
- J21 pad 5: /DAC_MOSI+2 -> /Amp board 2 interface/DAC_MOSI+
- J21 pad 6: /~{DAC_CS+2} -> /Amp board 2 interface/~{DAC_CS+}
- J21 pad 7: /~{LDAC-2} -> /Amp board 2 interface/~{LDAC-}
- J21 pad 8: /~{LDAC+2} -> /Amp board 2 interface/~{LDAC+}
- J23 pad 1: /Amp board 5 interface/~{Shutdown} -> /Amp board 5 interface/~{ADC_CS_LB-}
- J23 pad 2: GND -> /Amp board 5 interface/~{ADC_CS_LB+}
- J23 pad 4: /ADC_MOSI+5 -> /Amp board 5 interface/ADC_MOSI+
- J23 pad 5: /ADC_MOSI-5 -> /Amp board 5 interface/ADC_MOSI-
- J23 pad 7: /~{ADC_CS+5} -> /Amp board 5 interface/~{ADC_CS+}
- J23 pad 8: /~{ADC_CS-5} -> /Amp board 5 interface/~{ADC_CS-}
- J25 pad 1: /DAC_MISO-5 -> /Amp board 5 interface/DAC_MISO-
- J25 pad 2: /DAC_MISO+5 -> /Amp board 5 interface/DAC_MISO+
- J25 pad 4: /SCKO-5 -> /Amp board 5 interface/SCK_LB-
- J25 pad 5: /SCKO+5 -> /Amp board 5 interface/SCK_LB+
- J25 pad 6: unconnected-(J25-Pad6) -> /Amp board 5 interface/~{Shutdown}
- J25 pad 7: /ADC_MISO-5 -> /Amp board 5 interface/ADC_MISO-
- J25 pad 8: /ADC_MISO+5 -> /Amp board 5 interface/ADC_MISO+
- J26 pad 1: /SCKI-5 -> /Amp board 5 interface/SCK-
- J26 pad 2: /SCKI+5 -> /Amp board 5 interface/SCK+
- J26 pad 3: /~{DAC_CS-5} -> /Amp board 5 interface/~{DAC_CS-}
- J26 pad 4: /DAC_MOSI-5 -> /Amp board 5 interface/DAC_MOSI-
- J26 pad 5: /DAC_MOSI+5 -> /Amp board 5 interface/DAC_MOSI+
- J26 pad 6: /~{DAC_CS+5} -> /Amp board 5 interface/~{DAC_CS+}
- J26 pad 7: /~{LDAC-5} -> /Amp board 5 interface/~{LDAC-}
- J26 pad 8: /~{LDAC+5} -> /Amp board 5 interface/~{LDAC+}
- J28 pad 1: /Amp board 4 interface/~{Shutdown} -> /Amp board 4 interface/~{ADC_CS_LB-}
- J28 pad 2: GND -> /Amp board 4 interface/~{ADC_CS_LB+}
- J28 pad 4: /ADC_MOSI+4 -> /Amp board 4 interface/ADC_MOSI+
- J28 pad 5: /ADC_MOSI-4 -> /Amp board 4 interface/ADC_MOSI-
- J28 pad 7: /~{ADC_CS+4} -> /Amp board 4 interface/~{ADC_CS+}
- J28 pad 8: /~{ADC_CS-4} -> /Amp board 4 interface/~{ADC_CS-}
- J30 pad 1: /DAC_MISO-4 -> /Amp board 4 interface/DAC_MISO-
- J30 pad 2: /DAC_MISO+4 -> /Amp board 4 interface/DAC_MISO+
- J30 pad 4: /SCKO-4 -> /Amp board 4 interface/SCK_LB-
- J30 pad 5: /SCKO+4 -> /Amp board 4 interface/SCK_LB+
- J30 pad 6: unconnected-(J30-Pad6) -> /Amp board 4 interface/~{Shutdown}
- J30 pad 7: /ADC_MISO-4 -> /Amp board 4 interface/ADC_MISO-
- J30 pad 8: /ADC_MISO+4 -> /Amp board 4 interface/ADC_MISO+
- J31 pad 1: /SCKI-4 -> /Amp board 4 interface/SCK-
- J31 pad 2: /SCKI+4 -> /Amp board 4 interface/SCK+
- J31 pad 3: /~{DAC_CS-4} -> /Amp board 4 interface/~{DAC_CS-}
- J31 pad 4: /DAC_MOSI-4 -> /Amp board 4 interface/DAC_MOSI-
- J31 pad 5: /DAC_MOSI+4 -> /Amp board 4 interface/DAC_MOSI+
- J31 pad 6: /~{DAC_CS+4} -> /Amp board 4 interface/~{DAC_CS+}
- J31 pad 7: /~{LDAC-4} -> /Amp board 4 interface/~{LDAC-}
- J31 pad 8: /~{LDAC+4} -> /Amp board 4 interface/~{LDAC+}
- J33 pad 1: /Amp board 3 interface/~{Shutdown} -> /Amp board 3 interface/~{ADC_CS_LB-}
- J33 pad 2: GND -> /Amp board 3 interface/~{ADC_CS_LB+}
- J33 pad 4: /ADC_MOSI+3 -> /Amp board 3 interface/ADC_MOSI+
- J33 pad 5: /ADC_MOSI-3 -> /Amp board 3 interface/ADC_MOSI-
- J33 pad 7: /~{ADC_CS+3} -> /Amp board 3 interface/~{ADC_CS+}
- J33 pad 8: /~{ADC_CS-3} -> /Amp board 3 interface/~{ADC_CS-}
- J35 pad 1: /DAC_MISO-3 -> /Amp board 3 interface/DAC_MISO-
- J35 pad 2: /DAC_MISO+3 -> /Amp board 3 interface/DAC_MISO+
- J35 pad 4: /SCKO-3 -> /Amp board 3 interface/SCK_LB-
- J35 pad 5: /SCKO+3 -> /Amp board 3 interface/SCK_LB+
- J35 pad 6: unconnected-(J35-Pad6) -> /Amp board 3 interface/~{Shutdown}
- J35 pad 7: /ADC_MISO-3 -> /Amp board 3 interface/ADC_MISO-
- J35 pad 8: /ADC_MISO+3 -> /Amp board 3 interface/ADC_MISO+
- J36 pad 1: /SCKI-3 -> /Amp board 3 interface/SCK-
- J36 pad 2: /SCKI+3 -> /Amp board 3 interface/SCK+
- J36 pad 3: /~{DAC_CS-3} -> /Amp board 3 interface/~{DAC_CS-}
- J36 pad 4: /DAC_MOSI-3 -> /Amp board 3 interface/DAC_MOSI-
- J36 pad 5: /DAC_MOSI+3 -> /Amp board 3 interface/DAC_MOSI+
- J36 pad 6: /~{DAC_CS+3} -> /Amp board 3 interface/~{DAC_CS+}
- J36 pad 7: /~{LDAC-3} -> /Amp board 3 interface/~{LDAC-}
- J36 pad 8: /~{LDAC+3} -> /Amp board 3 interface/~{LDAC+}
- J38 pad 1: /Amp board 6 interface/~{Shutdown} -> /Amp board 6 interface/~{ADC_CS_LB-}
- J38 pad 2: GND -> /Amp board 6 interface/~{ADC_CS_LB+}
- J38 pad 4: /ADC_MOSI+6 -> /Amp board 6 interface/ADC_MOSI+
- J38 pad 5: /ADC_MOSI-6 -> /Amp board 6 interface/ADC_MOSI-
- J38 pad 7: /~{ADC_CS+6} -> /Amp board 6 interface/~{ADC_CS+}
- J38 pad 8: /~{ADC_CS-6} -> /Amp board 6 interface/~{ADC_CS-}
- J4 pad 1: /Amp board 0 interface/~{Shutdown} -> /Amp board 0 interface/~{ADC_CS_LB-}
- J4 pad 2: GND -> /Amp board 0 interface/~{ADC_CS_LB+}
- J4 pad 4: /ADC_MOSI+0 -> /Amp board 0 interface/ADC_MOSI+
- J4 pad 5: /ADC_MOSI-0 -> /Amp board 0 interface/ADC_MOSI-
- J4 pad 7: /~{ADC_CS+0} -> /Amp board 0 interface/~{ADC_CS+}
- J4 pad 8: /~{ADC_CS-0} -> /Amp board 0 interface/~{ADC_CS-}
- J40 pad 1: /DAC_MISO-6 -> /Amp board 6 interface/DAC_MISO-
- J40 pad 2: /DAC_MISO+6 -> /Amp board 6 interface/DAC_MISO+
- J40 pad 4: /SCKO-6 -> /Amp board 6 interface/SCK_LB-
- J40 pad 5: /SCKO+6 -> /Amp board 6 interface/SCK_LB+
- J40 pad 6: unconnected-(J40-Pad6) -> /Amp board 6 interface/~{Shutdown}
- J40 pad 7: /ADC_MISO-6 -> /Amp board 6 interface/ADC_MISO-
- J40 pad 8: /ADC_MISO+6 -> /Amp board 6 interface/ADC_MISO+
- J41 pad 1: /SCKI-6 -> /Amp board 6 interface/SCK-
- J41 pad 2: /SCKI+6 -> /Amp board 6 interface/SCK+
- J41 pad 3: /~{DAC_CS-6} -> /Amp board 6 interface/~{DAC_CS-}
- J41 pad 4: /DAC_MOSI-6 -> /Amp board 6 interface/DAC_MOSI-
- J41 pad 5: /DAC_MOSI+6 -> /Amp board 6 interface/DAC_MOSI+
- J41 pad 6: /~{DAC_CS+6} -> /Amp board 6 interface/~{DAC_CS+}
- J41 pad 7: /~{LDAC-6} -> /Amp board 6 interface/~{LDAC-}
- J41 pad 8: /~{LDAC+6} -> /Amp board 6 interface/~{LDAC+}
- J43 pad 1: /Amp board 7 interface/~{Shutdown} -> /Amp board 7 interface/~{ADC_CS_LB-}
- J43 pad 2: GND -> /Amp board 7 interface/~{ADC_CS_LB+}
- J43 pad 4: /ADC_MOSI+7 -> /Amp board 7 interface/ADC_MOSI+
- J43 pad 5: /ADC_MOSI-7 -> /Amp board 7 interface/ADC_MOSI-
- J43 pad 7: /~{ADC_CS+7} -> /Amp board 7 interface/~{ADC_CS+}
- J43 pad 8: /~{ADC_CS-7} -> /Amp board 7 interface/~{ADC_CS-}
- J45 pad 1: /DAC_MISO-7 -> /Amp board 7 interface/DAC_MISO-
- J45 pad 2: /DAC_MISO+7 -> /Amp board 7 interface/DAC_MISO+
- J45 pad 4: /SCKO-7 -> /Amp board 7 interface/SCK_LB-
- J45 pad 5: /SCKO+7 -> /Amp board 7 interface/SCK_LB+
- J45 pad 6: unconnected-(J45-Pad6) -> /Amp board 7 interface/~{Shutdown}
- J45 pad 7: /ADC_MISO-7 -> /Amp board 7 interface/ADC_MISO-
- J45 pad 8: /ADC_MISO+7 -> /Amp board 7 interface/ADC_MISO+
- J46 pad 1: /SCKI-7 -> /Amp board 7 interface/SCK-
- J46 pad 2: /SCKI+7 -> /Amp board 7 interface/SCK+
- J46 pad 3: /~{DAC_CS-7} -> /Amp board 7 interface/~{DAC_CS-}
- J46 pad 4: /DAC_MOSI-7 -> /Amp board 7 interface/DAC_MOSI-
- J46 pad 5: /DAC_MOSI+7 -> /Amp board 7 interface/DAC_MOSI+
- J46 pad 6: /~{DAC_CS+7} -> /Amp board 7 interface/~{DAC_CS+}
- J46 pad 7: /~{LDAC-7} -> /Amp board 7 interface/~{LDAC-}
- J46 pad 8: /~{LDAC+7} -> /Amp board 7 interface/~{LDAC+}
- J6 pad 1: /DAC_MISO-0 -> /Amp board 0 interface/DAC_MISO-
- J6 pad 2: /DAC_MISO+0 -> /Amp board 0 interface/DAC_MISO+
- J6 pad 4: /SCKO-0 -> /Amp board 0 interface/SCK_LB-
- J6 pad 5: /SCKO+0 -> /Amp board 0 interface/SCK_LB+
- J6 pad 6: unconnected-(J6-Pad6) -> /Amp board 0 interface/~{Shutdown}
- J6 pad 7: /ADC_MISO-0 -> /Amp board 0 interface/ADC_MISO-
- J6 pad 8: /ADC_MISO+0 -> /Amp board 0 interface/ADC_MISO+
- J7 pad 1: /SCKI-0 -> /Amp board 0 interface/SCK-
- J7 pad 2: /SCKI+0 -> /Amp board 0 interface/SCK+
- J7 pad 3: /~{DAC_CS-0} -> /Amp board 0 interface/~{DAC_CS-}
- J7 pad 4: /DAC_MOSI-0 -> /Amp board 0 interface/DAC_MOSI-
- J7 pad 5: /DAC_MOSI+0 -> /Amp board 0 interface/DAC_MOSI+
- J7 pad 6: /~{DAC_CS+0} -> /Amp board 0 interface/~{DAC_CS+}
- J7 pad 7: /~{LDAC-0} -> /Amp board 0 interface/~{LDAC-}
- J7 pad 8: /~{LDAC+0} -> /Amp board 0 interface/~{LDAC+}
- JA1 pad 11: /DAC_MISO+5 -> /DAC_MOSI5
- JA1 pad 12: /ADC_MISO-5 -> /~{ADC_CS_LB5}
- JA1 pad 13: /DAC_MISO-5 -> /~{LDAC5}
- JA1 pad 14: /ADC_MISO+5 -> /ADC_MISO5
- JA1 pad 17: /ADC_MOSI+5 -> /~{DAC_CS5}
- JA1 pad 18: /~{DAC_CS-5} -> /DAC_MISO5
- JA1 pad 19: /ADC_MOSI-5 -> /Power_Enable_Ext
- JA1 pad 20: /~{DAC_CS+5} -> unconnected-(JA1-Pin_20-Pad20)
- JA1 pad 24: /DAC_MISO-7 -> /~{LDAC7}
- JA1 pad 25: /FPGA Board, Signal Distribution/Power_Enable_Ext_Sense -> unconnected-(JA1-Pin_25-Pad25)
- JA1 pad 26: /DAC_MISO+7 -> /DAC_MOSI7
- JA1 pad 29: /~{DAC_CS+7} -> /SCK5
- JA1 pad 3: +2.5V -> +3V3
- JA1 pad 30: /DAC_MOSI-7 -> /ADC_MISO7
- JA1 pad 31: /~{DAC_CS-7} -> unconnected-(JA1-Pin_31-Pad31)
- JA1 pad 32: /DAC_MOSI+7 -> /~{ADC_CS7}
- JA1 pad 35: /ADC_MISO+7 -> unconnected-(JA1-Pin_35-Pad35)
- JA1 pad 36: /SCKO-5 -> /DAC_MISO7
- JA1 pad 37: /ADC_MISO-7 -> /SCK_LB5
- JA1 pad 38: /SCKO+5 -> unconnected-(JA1-Pin_38-Pad38)
- JA1 pad 5: /DAC_MOSI+5 -> /~{ADC_CS5}
- JA1 pad 6: /~{ADC_CS-5} -> /SCK7
- JA1 pad 7: /DAC_MOSI-5 -> /ADC_MOSI5
- JA1 pad 8: /~{ADC_CS+5} -> /~{DAC_CS7}
- JA2 pad 11: /~{DAC_CS+4} -> unconnected-(JA2-Pin_11-Pad11)
- JA2 pad 12: /ADC_MOSI-6 -> /ADC_MISO6
- JA2 pad 13: /~{DAC_CS-4} -> unconnected-(JA2-Pin_13-Pad13)
- JA2 pad 14: /ADC_MOSI+6 -> /~{ADC_CS6}
- JA2 pad 17: /~{ADC_CS+7} -> unconnected-(JA2-Pin_17-Pad17)
- JA2 pad 18: /DAC_MISO-6 -> /ADC_MOSI6
- JA2 pad 19: /~{ADC_CS-7} -> unconnected-(JA2-Pin_19-Pad19)
- JA2 pad 20: /DAC_MISO+6 -> /DAC_MOSI6
- JA2 pad 23: /~{DAC_CS+6} -> unconnected-(JA2-Pin_23-Pad23)
- JA2 pad 24: /DAC_MOSI-6 -> /~{LDAC6}
- JA2 pad 25: /~{DAC_CS-6} -> unconnected-(JA2-Pin_25-Pad25)
- JA2 pad 26: /DAC_MOSI+6 -> /SCK6
- JA2 pad 29: /ADC_MISO+6 -> /ADC_MOSI7
- JA2 pad 3: +2.5V -> +3V3
- JA2 pad 30: /ADC_MOSI-7 -> /~{DAC_CS6}
- JA2 pad 31: /ADC_MISO-6 -> /~{ADC_CS_LB7}
- JA2 pad 32: /ADC_MOSI+7 -> unconnected-(JA2-Pin_32-Pad32)
- JA2 pad 35: /SCKO+7 -> /SCK_LB7
- JA2 pad 36: /SCKO-6 -> /SCK_LB6
- JA2 pad 37: /SCKO-7 -> unconnected-(JA2-Pin_37-Pad37)
- JA2 pad 38: /SCKO+6 -> unconnected-(JA2-Pin_38-Pad38)
- JA2 pad 5: /~{ADC_CS+6} -> unconnected-(JA2-Pin_5-Pad5)
- JA2 pad 6: /DAC_MOSI-4 -> /DAC_MISO6
- JA2 pad 7: /~{ADC_CS-6} -> unconnected-(JA2-Pin_7-Pad7)
- JA2 pad 8: /DAC_MOSI+4 -> /~{ADC_CS_LB6}
- JB1 pad 11: /DAC_MISO+1 -> /SCK1
- JB1 pad 12: /ADC_MISO-1 -> /ADC_MISO1
- JB1 pad 13: /DAC_MISO-1 -> /SCK3
- JB1 pad 14: /ADC_MISO+1 -> /~{ADC_CS_LB1}
- JB1 pad 17: /ADC_MOSI+1 -> /~{DAC_CS3}
- JB1 pad 18: /~{DAC_CS-1} -> /DAC_MOSI1
- JB1 pad 19: /ADC_MOSI-1 -> /~{LDAC3}
- JB1 pad 20: /~{DAC_CS+1} -> /~{LDAC1}
- JB1 pad 23: /DAC_MOSI+3 -> /DAC_MOSI3
- JB1 pad 24: /ADC_MISO-3 -> unconnected-(JB1-Pin_24-Pad24)
- JB1 pad 25: /DAC_MOSI-3 -> /ADC_MOSI3
- JB1 pad 26: /ADC_MISO+3 -> unconnected-(JB1-Pin_26-Pad26)
- JB1 pad 29: /DAC_MISO+3 -> /~{ADC_CS3}
- JB1 pad 3: +2.5V -> +3V3
- JB1 pad 30: /~{DAC_CS-3} -> unconnected-(JB1-Pin_30-Pad30)
- JB1 pad 31: /DAC_MISO-3 -> /DAC_MISO3
- JB1 pad 32: /~{DAC_CS+3} -> /~{ADC_CS_LB3}
- JB1 pad 35: /SCKO+3 -> /SCK_LB3
- JB1 pad 36: /SCKO-1 -> /ADC_MISO3
- JB1 pad 37: /SCKO-3 -> unconnected-(JB1-Pin_37-Pad37)
- JB1 pad 38: /SCKO+1 -> /SCK_LB1
- JB1 pad 5: /DAC_MOSI+1 -> /ADC_MOSI1
- JB1 pad 6: /~{ADC_CS-1} -> /~{ADC_CS1}
- JB1 pad 7: /DAC_MOSI-1 -> /~{DAC_CS1}
- JB1 pad 8: /~{ADC_CS+1} -> /DAC_MISO1
- JB2 pad 11: /ADC_MISO+0 -> /~{ADC_CS_LB0}
- JB2 pad 12: /DAC_MISO-0 -> /ADC_MOSI0
- JB2 pad 13: /ADC_MISO-0 -> unconnected-(JB2-Pin_13-Pad13)
- JB2 pad 14: /DAC_MISO+0 -> /~{ADC_CS0}
- JB2 pad 17: /~{ADC_CS+0} -> unconnected-(JB2-Pin_17-Pad17)
- JB2 pad 18: /DAC_MOSI-0 -> /~{DAC_CS0}
- JB2 pad 19: /~{ADC_CS-0} -> unconnected-(JB2-Pin_19-Pad19)
- JB2 pad 20: /DAC_MOSI+0 -> /SCK0
- JB2 pad 23: /FPGA Board, Signal Distribution/~{SCKI+} -> unconnected-(JB2-Pin_23-Pad23)
- JB2 pad 24: /FPGA Board, Signal Distribution/LDAC- -> unconnected-(JB2-Pin_24-Pad24)
- JB2 pad 25: /FPGA Board, Signal Distribution/~{SCKI-} -> unconnected-(JB2-Pin_25-Pad25)
- JB2 pad 26: /FPGA Board, Signal Distribution/LDAC+ -> unconnected-(JB2-Pin_26-Pad26)
- JB2 pad 29: /ADC_MOSI+3 -> unconnected-(JB2-Pin_29-Pad29)
- JB2 pad 3: +2.5V -> +3V3
- JB2 pad 30: /~{ADC_CS-3} -> unconnected-(JB2-Pin_30-Pad30)
- JB2 pad 31: /ADC_MOSI-3 -> unconnected-(JB2-Pin_31-Pad31)
- JB2 pad 32: /~{ADC_CS+3} -> unconnected-(JB2-Pin_32-Pad32)
- JB2 pad 35: /SCKO+0 -> /SCK_LB0
- JB2 pad 36: /FPGA Board, Signal Distribution/Trigger_2.5 -> /Activity Indicator (Trigger)/In
- JB2 pad 37: /SCKO-0 -> unconnected-(JB2-Pin_37-Pad37)
- JB2 pad 38: /FPGA Board, Signal Distribution/Scanner_Clk_2.5 -> /FPGA Board, Signal Distribution/Scanner_Clk
- JB2 pad 5: /~{DAC_CS+0} -> /DAC_MISO0
- JB2 pad 6: /ADC_MOSI-0 -> /~{LDAC0}
- JB2 pad 7: /~{DAC_CS-0} -> /ADC_MISO0
- JB2 pad 8: /ADC_MOSI+0 -> /DAC_MOSI0
- JC1 pad 11: /DAC_MOSI+2 -> /~{ADC_CS2}
- JC1 pad 12: /ADC_MISO-2 -> /~{LDAC2}
- JC1 pad 13: /DAC_MOSI-2 -> /~{ADC_CS_LB2}
- JC1 pad 14: /ADC_MISO+2 -> /DAC_MISO4
- JC1 pad 17: /DAC_MISO+2 -> /ADC_MISO2
- JC1 pad 18: /~{DAC_CS-2} -> /~{ADC_CS_LB4}
- JC1 pad 19: /DAC_MISO-2 -> /DAC_MISO2
- JC1 pad 20: /~{DAC_CS+2} -> /ADC_MISO4
- JC1 pad 23: /ADC_MOSI+2 -> /SCK2
- JC1 pad 24: /~{ADC_CS-4} -> /~{ADC_CS4}
- JC1 pad 25: /ADC_MOSI-2 -> /~{DAC_CS2}
- JC1 pad 26: /~{ADC_CS+4} -> /ADC_MOSI4
- JC1 pad 29: /~{ADC_CS+2} -> unconnected-(JC1-Pin_29-Pad29)
- JC1 pad 3: +2.5V -> +3V3
- JC1 pad 30: /ADC_MISO-4 -> /DAC_MOSI4
- JC1 pad 31: /~{ADC_CS-2} -> unconnected-(JC1-Pin_31-Pad31)
- JC1 pad 32: /ADC_MISO+4 -> /~{LDAC4}
- JC1 pad 35: /SCKO+4 -> unconnected-(JC1-Pin_35-Pad35)
- JC1 pad 36: /DAC_MISO-4 -> /SCK4
- JC1 pad 37: /SCKO-4 -> unconnected-(JC1-Pin_37-Pad37)
- JC1 pad 38: /DAC_MISO+4 -> /~{DAC_CS4}
- JC1 pad 5: /ADC_MOSI+4 -> /SCK_LB2
- JC1 pad 6: /SCKO-2 -> /SCK_LB4
- JC1 pad 7: /ADC_MOSI-4 -> /ADC_MOSI2
- JC1 pad 8: /SCKO+2 -> /DAC_MOSI2
- JP1 pad 1: +3V3 -> /Amp board 0 interface/SCK_LB+
- JP1 pad 2: Net-(U2-ERC) -> Net-(JP1-B)
- JP10 pad 1: GND -> /Amp board 1 interface/SCK_LB-
- JP10 pad 2: Net-(U3-ITTP) -> Net-(JP10-B)
- JP11 pad 1: +3V3 -> /Amp board 2 interface/SCK_LB-
- JP11 pad 2: Net-(U3-OE) -> Net-(JP11-B)
- JP12 pad 1: GND -> /Amp board 3 interface/SCK_LB-
- JP12 pad 2: Net-(U3-OTTP) -> Net-(JP12-B)
- JP2 pad 1: Net-(U2-ERC) -> /Amp board 1 interface/SCK_LB+
- JP2 pad 2: GND -> Net-(JP2-B)
- JP3 pad 1: GND -> /Amp board 2 interface/SCK_LB+
- JP3 pad 2: Net-(U2-Insel) -> Net-(JP3-B)
- JP4 pad 1: GND -> /Amp board 3 interface/SCK_LB+
- JP4 pad 2: Net-(U2-ITTP) -> Net-(JP4-B)
- JP5 pad 1: +3V3 -> /Amp board 4 interface/SCK_LB+
- JP5 pad 2: Net-(U2-OE) -> Net-(JP5-B)
- JP6 pad 1: GND -> /Amp board 5 interface/SCK_LB+
- JP6 pad 2: Net-(U2-OTTP) -> Net-(JP52-B)
- JP7 pad 1: +3V3 -> /Amp board 6 interface/SCK_LB+
- JP7 pad 2: Net-(U3-ERC) -> Net-(JP53-B)
- JP8 pad 1: Net-(U3-ERC) -> /Amp board 7 interface/SCK_LB+
- JP8 pad 2: GND -> Net-(JP54-B)
- JP9 pad 1: GND -> /Amp board 0 interface/SCK_LB-
- JP9 pad 2: Net-(U3-Insel) -> Net-(JP39-B)
- TP12 pad 1: Net-(U34-Clk) -> /FPGA Board, Signal Distribution/Scanner_Clk
- TP23 pad 1: /Shutdown_Reset -> /Shutdown_Force
- U1 pad 5: +2.5V -> +3V3
- U12 pad 5: +2.5V -> +3V3
- U13 pad 8: +2.5V -> +3V3
- U14 pad 5: +2.5V -> +3V3
- U15 pad 8: +2.5V -> +3V3
- U16 pad 8: +2.5V -> +3V3
- U17 pad 5: +2.5V -> +3V3
- U18 pad 8: +2.5V -> +3V3
- U19 pad 5: +2.5V -> +3V3
- U2 pad 1: unconnected-(U2-Divide-Pad1) -> +3V3
- U2 pad 2: Net-(U2-Insel) -> /ADC_MOSI0
- U2 pad 3: /FPGA Board, Signal Distribution/~{SCKI-} -> /~{ADC_CS0}
- U2 pad 4: /FPGA Board, Signal Distribution/~{SCKI+} -> GND
- U2 pad 5: +3V3 -> /Amp board 0 interface/~{ADC_CS-}
- U2 pad 6: GND -> /Amp board 0 interface/~{ADC_CS+}
- U2 pad 7: GND -> /Amp board 0 interface/ADC_MOSI-
- U2 pad 8: Net-(U2-ITTP) -> /Amp board 0 interface/ADC_MOSI+
- U20 pad 8: +2.5V -> +3V3
- U21 pad 5: +2.5V -> +3V3
- U22 pad 8: +2.5V -> +3V3
- U23 pad 5: +2.5V -> +3V3
- U24 pad 8: +2.5V -> +3V3
- U25 pad 5: +2.5V -> +3V3
- U26 pad 8: +2.5V -> +3V3
- U3 pad 1: unconnected-(U3-Divide-Pad1) -> +3V3
- U3 pad 2: Net-(U3-Insel) -> /ADC_MOSI1
- U3 pad 3: /FPGA Board, Signal Distribution/LDAC- -> /~{ADC_CS1}
- U3 pad 4: /FPGA Board, Signal Distribution/LDAC+ -> GND
- U3 pad 5: +3V3 -> /Amp board 1 interface/~{ADC_CS-}
- U3 pad 6: GND -> /Amp board 1 interface/~{ADC_CS+}
- U3 pad 7: GND -> /Amp board 1 interface/ADC_MOSI-
- U3 pad 8: Net-(U3-ITTP) -> /Amp board 1 interface/ADC_MOSI+
- U34 pad 5: Net-(U34-Clk) -> /FPGA Board, Signal Distribution/Scanner_Clk
- U6 pad 16: +2.5V -> +3V3
Routing:
- net +3V3: track 807.5 -> 324.7 mm, vias 47 -> 79
- net /~{LDAC-6}: track 261.3 -> 0.00 mm, vias 2 -> 0
- net /~{LDAC+6}: track 258.2 -> 0.00 mm, vias 2 -> 0
- net /SCKI-6: track 249.5 -> 0.00 mm, vias 1 -> 0
- net /~{LDAC-7}: track 248.2 -> 0.00 mm, vias 3 -> 0
- net /SCKI+6: track 246.6 -> 0.00 mm, vias 1 -> 0
- net /~{LDAC+7}: track 243.7 -> 0.00 mm, vias 3 -> 0
- net /SCK6: track 0.00 -> 227.1 mm, vias 0 -> 1
- net /SCKI+7: track 222.2 -> 0.00 mm, vias 2 -> 0
- net /~{DAC_CS6}: track 0.00 -> 222.0 mm, vias 0 -> 1
- net /~{DAC_CS+6}: track 221.4 -> 0.00 mm
- net /SCKI-7: track 220.7 -> 0.00 mm, vias 2 -> 0
- net /~{ADC_CS+7}: track 220.2 -> 0.00 mm
- net /DAC_MOSI-6: track 219.6 -> 0.00 mm
- net /~{LDAC6}: track 0.00 -> 219.3 mm, vias 0 -> 1
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- added copper zone on In3.Cu, net +3V3
- removed copper zone on In3.Cu, net +2.5V
- removed copper zone on In2.Cu, net +3V3
Other:
- board text added: "+VDC"
- board text added: "Don Straney 2026-07"
- board text added: "Inverted"
- board text added: "Not inverted"
- board text added: "Rev. D3"
- board text added: "SCLK_LB:"
- board text added: "Shutdown Force"
- board text added: "Shutdown Reset"
- board text added: "Trigger"
- board text removed: "+2.5V"
- board text removed: "30 Mhz (2.5V)"
- board text removed: "Don Straney 2025-04"
- board text removed: "Expected stackup: 6 layers, 1.6 mm thickness - Top silkscreen - Top soldermask - 1 oz copper (top layer) - 0.15 mm pre-preg - 1 oz copper (layer 2) - 0.43 mm core - 1 oz copper (layer 3) - 0.15 mm pre-preg - 1 oz copper (layer 4) - 0.43 mm core - 1 oz copper (layer 5) - 0.15 mm pre-preg - 1 oz copper (bottom layer) - Bottom soldermask - Bottom silkscreen"
- board text removed: "Reset"
- board text removed: "Rev. D2"
- board text removed: "Trigger (2.5V)"
