File: pcbs/backplane/backplane.kicad_pcb (KiCad board)
At the start: 6 copper layers, 145 x 355 mm, 486 parts, among them J1 Conn_01x02, J10 AFBR-2624Z, J11 AFBR-2624Z, J12 AFBR-1624Z, J13 RJ45_Shielded, J14 Conn_01x02, J15 RJ45_Shielded, J16 RJ45_Shielded, J17 Conn_01x02, J18 RJ45_Shielded, J19 Conn_01x02, J2 Conn_02x15_Odd_Even, J20 RJ45_Shielded, J21 RJ45_Shielded, J22 Conn_01x02, J23 RJ45_Shielded, J24 Conn_01x02, J25 RJ45_Shielded, J26 RJ45_Shielded, J27 Conn_01x02, J28 RJ45_Shielded, J29 Conn_01x02, J3 Conn_02x20_Odd_Even, J30 RJ45_Shielded, J31 RJ45_Shielded, J32 Conn_01x02, J33 RJ45_Shielded, J34 Conn_01x02, J35 RJ45_Shielded, J36 RJ45_Shielded, J37 Conn_01x02, J38 RJ45_Shielded, J39 Conn_01x02, J4 RJ45_Shielded, J40 RJ45_Shielded, J41 RJ45_Shielded, J42 Conn_01x02, J43 RJ45_Shielded, J44 Conn_01x02, J45 RJ45_Shielded, J46 RJ45_Shielded, J47 Conn_01x02, J48 Conn_01x02, J5 AFBR-2624Z, J6 RJ45_Shielded, J7 RJ45_Shielded, J8 Conn_01x02, J9 AFBR-2624Z, Q1 MMBT3904, Q10 MMBT3906, Q11 MMBT3906, Q12 MMBT3904, Q13 MMBT3904, Q2 MMBT3904, Q3 MMBT3904, Q4 MMBT3904, Q5 MMBT3904, Q6 MMBT3904, Q7 MMBT3904, Q8 MMBT3904, Q9 D44H11G, U1 74LVC1G14, U10 74LVC2T45, U12 74LVC1G14, U13 74LVC2G02, U14 74LVC1G14, U15 74LVC2G02, U16 74LVC2G02, U17 74LVC1G14, U18 74LVC2G02, U19 74LVC1G14, U2 FIN1027, U20 74LVC2G02, U21 74LVC1G14, U22 74LVC2G02, U23 74LVC1G14, U24 74LVC2G02, U25 74LVC1G14, U26 74LVC2G02, U27 74LVC1G14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

Commit message: Optical Ethernet, closed-loop response prediction
Backplane: added optical Ethernet interface with transceiver AFBR-5972Z, updated pinout (fixes #44)
Backplane: cleaned up schematic readability slightly (assigned sheet background colors)
Docs: added closed-loop response plotting to compensation script
Parts:
- added C121: 10uF 6.3V X7R, Capacitor_SMD:C_0805_2012Metric, F.Cu at (65.1, 245.2)
- added C122: 100nF 50V X7R, Capacitor_SMD:C_0603_1608Metric, F.Cu at (57.9, 224.2)
- added C125: 100nF 50V X7R, Capacitor_SMD:C_0603_1608Metric, F.Cu at (55.6, 229.2)
- added C25: 1uF 50V X7R, Capacitor_SMD:C_0805_2012Metric, F.Cu at (52.8, 240.2)
- added C27: 1uF 50V X7R, Capacitor_SMD:C_0805_2012Metric, F.Cu at (52.8, 236.7)
- added C29: 10uF 6.3V X7R, Capacitor_SMD:C_0805_2012Metric, F.Cu at (54.8, 240.2)
- added C30: 10uF 6.3V X7R, Capacitor_SMD:C_0805_2012Metric, F.Cu at (54.8, 236.7)
- added C36: 100nF 50V X7R, Capacitor_SMD:C_0603_1608Metric, F.Cu at (58.1, 242.8)
- added C37: 100nF 50V X7R, Capacitor_SMD:C_0603_1608Metric, F.Cu at (58.1, 241.2)
- added C65: 100nF 50V X7R, Capacitor_SMD:C_0603_1608Metric, F.Cu at (58.1, 235.0)
- added C77: 100nF 50V X7R, Capacitor_SMD:C_0603_1608Metric, F.Cu at (58.1, 236.5)
- added C78: 1uF 50V X7R, Capacitor_SMD:C_0805_2012Metric, F.Cu at (61.6, 245.2)
- added JP34: Jumper_NC_Small, Jumper:SolderJumper-2_P1.3mm_Bridged_RoundedPad1.0x1.5mm, F.Cu at (65.4, 234.8)
- added JP56: Jumper_NC_Small, Jumper:SolderJumper-2_P1.3mm_Bridged_RoundedPad1.0x1.5mm, F.Cu at (67.9, 234.8)
- added R12: 1, Resistor_SMD:R_0805_2012Metric, F.Cu at (54.8, 243.7)
- added R48: 1, Resistor_SMD:R_0805_2012Metric, F.Cu at (54.8, 233.2)
- added R49: 150, Resistor_SMD:R_0805_2012Metric, F.Cu at (58.1, 238.5)
- added R51: 150, Resistor_SMD:R_0805_2012Metric, F.Cu at (58.1, 233.2)
- added R52: 100, Resistor_SMD:R_0805_2012Metric, F.Cu at (61.9, 237.8)
- added R53: 10, Resistor_SMD:R_0805_2012Metric, F.Cu at (68.6, 245.2)
- added R54: 15K, Resistor_SMD:R_0805_2012Metric, F.Cu at (58.1, 230.2)
- added R55: 10K, Resistor_SMD:R_0805_2012Metric, F.Cu at (60.1, 230.2)
- added R56: 10K, Resistor_SMD:R_0805_2012Metric, F.Cu at (55.4, 247.0)
- added R57: 10K, Resistor_SMD:R_0805_2012Metric, F.Cu at (60.6, 226.8)
- added R85: 20K, Resistor_SMD:R_0805_2012Metric, F.Cu at (62.9, 235.0)
- added R86: 20K, Resistor_SMD:R_0805_2012Metric, F.Cu at (60.9, 235.0)
- added TP28: TestPoint, TestPoint:TestPoint_Pad_D1.0mm, F.Cu at (69.5, 241.0)
- added TP31: TestPoint, TestPoint:TestPoint_Pad_D2.0mm, F.Cu at (65.0, 228.5)
- added TP32: TestPoint, TestPoint:TestPoint_Pad_D1.0mm, F.Cu at (69.5, 243.2)
- added U11: AFBR-5972Z, shim:AFBR-5972Z, F.Cu at (40.8, 238.7)
- added U32: LMV331, Package_TO_SOT_SMD:SOT-23-5, F.Cu at (57.4, 226.8)
- moved U7 103.1 mm to (63.9, 241.5), turned to 180 degrees
- moved JP25 4.51 mm to (72.2, 228.2)
- moved JP14 3.95 mm to (72.2, 237.5)
- moved JP22 3.78 mm to (72.2, 223.2)
- moved JP17 3.76 mm to (72.2, 242.5)
- moved JP26 3.51 mm to (72.2, 230.8)
- moved JP13 2.02 mm to (72.2, 235.0)
- moved JP18 1.52 mm to (72.2, 245.0)
- moved JP23 1.52 mm to (72.2, 225.8)
- moved JP21 0.56 mm to (72.2, 220.8)
- moved JP15 0.35 mm to (72.2, 240.0)
Connections:
- JC1 pad 29: unconnected-(JC1-Pin_29-Pad29) -> /Eth_SD
- JC1 pad 35: unconnected-(JC1-Pin_35-Pad35) -> /Eth_Rx
- JC1 pad 37: unconnected-(JC1-Pin_37-Pad37) -> /Eth_Tx
- U7 pad 1: unconnected-(U7-DE-Pad1) -> Net-(U7-DE)
- U7 pad 10: unconnected-(U7-RI+-Pad10) -> Net-(U7-RI+)
- U7 pad 11: unconnected-(U7-DO--Pad11) -> Net-(U7-DO-)
- U7 pad 12: unconnected-(U7-DO+-Pad12) -> Net-(U7-DO+)
- U7 pad 14: unconnected-(U7-VCC-Pad14) -> Net-(U7-VCC)
- U7 pad 2: unconnected-(U7-DI-Pad2) -> /Eth_Tx
- U7 pad 4: unconnected-(U7-RO-Pad4) -> /Eth_Rx
- U7 pad 7: unconnected-(U7-GND-Pad7) -> GND
- U7 pad 8: unconnected-(U7-~{RE}-Pad8) -> Net-(U7-~{RE})
- U7 pad 9: unconnected-(U7-RI--Pad9) -> Net-(U7-RI-)
Routing:
- net /Eth_SD: track 0.00 -> 69.0 mm, vias 0 -> 1
- net /Eth_Rx: track 0.00 -> 52.2 mm, vias 0 -> 1
- net /Eth_Tx: track 0.00 -> 52.1 mm, vias 0 -> 1
- net /SD: track 0.00 -> 33.8 mm, vias 0 -> 1
- net Net-(U11-RData+): track 0.00 -> 24.4 mm, vias 0 -> 1
- net Net-(U7-VCC): track 0.00 -> 21.1 mm
- net Net-(U11-RData-): track 0.00 -> 20.6 mm, vias 0 -> 1
- net Net-(U11-TData+): track 0.00 -> 14.0 mm, vias 0 -> 1
- net +3V3: track 322.2 -> 334.5 mm, vias 83 -> 89
- net Net-(U7-DE): track 0.00 -> 10.8 mm
- net Net-(U7-RI+): track 0.00 -> 10.5 mm
- net Net-(U7-~{RE}): track 0.00 -> 10.5 mm, vias 0 -> 2
- net Net-(U11-TData-): track 0.00 -> 10.1 mm, vias 0 -> 1
- net Net-(U11-RX_Vcc): track 0.00 -> 10.0 mm
- net Net-(U11-TX_Vcc): track 0.00 -> 9.72 mm
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Other:
- board text added: "Eth SD"
- board text added: "Optical Ethernet"
- board text added: "Rx Tx"
