File: pcbs/backplane/fanout_buffer.kicad_sch (KiCad schematic)
At the start: 16 parts, among them U2 CDCUN1208LP

Commit message: Backplane comms updates, manufacturing renaming
Removed misspelled "maunfacturing" folder, fixed gitignore rule to remove manufacturing folders within individual PCB folders too
Changed SCKI/SCKO terminology to SCK, SCK_LB (loopback) for clarity
Added ADC_CS loopback signal between amp ctrl board & backplane for better fast-clock timing (#38)
Backplane: changed LVDS FPGA outputs to single-ended FPGA outputs to gain more I/O pins, added external LVDS transceivers (#38)
Backplane: replaced global clock & ~LDAC buffers with a separate FPGA pin for each amp ctrl board (#38)
Backplane: removed +2.5V power supply and level translations, no longer needed without FPGA I/O pins using LVDS_25 I/O configuration
Backplane: replaced +VDC-input resistor with solder jumper (on by default)
Backplane: changed field names (Part Number to MPN) to match Aisler's naming convention for automatic recognition
Amp ctrl: fixed optional level-shifter circuit on each channel for voltage inputs (#9) schematic & channel-1 layout
Parts:
- C36: MPN (none) -> C0805C105K3RACTU; Part Number C0805C105K3RACTU -> (none)
- C5, C6, C7, C8, C9: MPN (none) -> C0603C104K5RACTU; Part Number C0603C104K5RACTU -> (none)
- R1: MPN (none) -> RK73H1ETTP1000F; Part Number RK73H1ETTP1000F -> (none)
- R84, R86: MPN (none) -> RK73H1ETTP1002F; Part Number RK73H1ETTP1002F -> (none)
- U2: MPN (none) -> CDCUN1208LPRHBT; MPN Alt. (none) -> CDCUN1208LPRHBR; Part Number CDCUN1208LPRHBT -> (none); Part Number Alt. CDCUN1208LPRHBR -> (none)
