File: pcbs/backplane/amp_board_interface.kicad_sch (KiCad schematic)
At the start: 19 parts, among them J4 RJ45_Shielded, J6 RJ45_Shielded, J7 RJ45_Shielded, Q1 MMBT3904, U1 74LVC1G14, U16 74LVC2G02

Commit message: Backplane comms updates, manufacturing renaming
Removed misspelled "maunfacturing" folder, fixed gitignore rule to remove manufacturing folders within individual PCB folders too
Changed SCKI/SCKO terminology to SCK, SCK_LB (loopback) for clarity
Added ADC_CS loopback signal between amp ctrl board & backplane for better fast-clock timing (#38)
Backplane: changed LVDS FPGA outputs to single-ended FPGA outputs to gain more I/O pins, added external LVDS transceivers (#38)
Backplane: replaced global clock & ~LDAC buffers with a separate FPGA pin for each amp ctrl board (#38)
Backplane: removed +2.5V power supply and level translations, no longer needed without FPGA I/O pins using LVDS_25 I/O configuration
Backplane: replaced +VDC-input resistor with solder jumper (on by default)
Backplane: changed field names (Part Number to MPN) to match Aisler's naming convention for automatic recognition
Amp ctrl: fixed optional level-shifter circuit on each channel for voltage inputs (#9) schematic & channel-1 layout
Parts:
- removed TP21: TestPoint, TestPoint:TestPoint_Pad_D2.0mm, symbol Connector:TestPoint
- added C104, C112: 22pF 50V NP0, shim:C_Array_0612_1632Metric, symbol shim:C_Array_4
- added C5, C80, C88, C96: 1uF 16V X7R, Capacitor_SMD:C_0603_1608Metric, symbol Device:C
- added JP1, JP9: Jumper_2_Open, Jumper:SolderJumper-2_P1.3mm_Open_RoundedPad1.0x1.5mm, symbol Jumper:Jumper_2_Open
- added JP39, JP47: Jumper_2_Bridged, Jumper:SolderJumper-2_P1.3mm_Bridged_RoundedPad1.0x1.5mm, symbol Jumper:Jumper_2_Bridged
- added RN12, RN20, RN28, RN4: 100 5%, Resistor_SMD:R_Array_Concave_4x0603, symbol Device:R_Pack04
- added U2, U56, U64: FIN1027, Package_SO:SOIC-8_3.9x4.9mm_P1.27mm, symbol shim:FIN1027
- added U72: FIN1048, Package_SO:TSSOP-16_4.4x5mm_P0.65mm, symbol shim:FIN1048
- C1, C38: MPN (none) -> C0603C104K5RACTU; Part Number C0603C104K5RACTU -> (none)
- C39: MPN (none) -> C0805C105K3RACTU; Part Number C0805C105K3RACTU -> (none)
- D4: MPN (none) -> LTST-C170KRKT; Part Number LTST-C170KRKT -> (none)
- J4, J6, J7: MPN (none) -> RJE061881120; MPN Alt. (none) -> RJE061881120H; Part Number RJE061881120 -> (none); Part Number Alt. RJE061881120H -> (none)
- Q1: MPN (none) -> MMBT3904-7-F; MPN Alt. (none) -> MMBT3904,215; Part Number MMBT3904-7-F -> (none); Part Number Alt. MMBT3904,215 -> (none)
- R16, R66: MPN (none) -> RK73H2ATTD1001F; Part Number RK73H2ATTD1001F -> (none)
- R17: MPN (none) -> RK73H2ATTD3301F; Part Number RK73H2ATTD3301F -> (none)
- R63, R64: MPN (none) -> RK73H2ATTD2002F; Part Number RK73H2ATTD2002F -> (none)
- TP19: MPN (none) -> 5019; Part Number 5019 -> (none)
- U1: MPN (none) -> SN74LVC1G14DBVR; MPN Alt. (none) -> 74LVC1G14GV,125; Part Number SN74LVC1G14DBVR -> (none); Part Number Alt. 74LVC1G14GV,125 -> (none)
- U16: MPN (none) -> SN74LVC2G02DCTR; MPN Alt. (none) -> 74LVC2G02DP,125; Part Number SN74LVC2G02DCTR -> (none); Part Number Alt. 74LVC2G02DP,125 -> (none)
Connections:
- net +2.5V is gone; now on net +3V3: C1.1, C38.1, C39.2, U1.5 (VCC), U16.8 (VCC)
- net +3V3: now also C5.2, C80.2, C88.2, C96.2, U2.1 (VDD), U56.1 (VDD), U64.1 (VDD), U72.13 (VDD), U72.16 (EN)
- net ADC_MISO+: now also RN4.3 (R3.1), U72.6 (A3)
- net ADC_MISO-: now also RN4.6 (R3.2), U72.5 (B3)
- net ADC_MOSI+: now also U2.8 (A1)
- net ADC_MOSI-: now also U2.7 (B1)
- net DAC_MISO+: now also RN4.1 (R1.1), U72.2 (A1)
- net DAC_MISO-: now also RN4.8 (R1.2), U72.1 (B1)
- net DAC_MOSI+: now also U56.6 (A2)
- net DAC_MOSI-: now also U56.5 (B2)
- net GND: now also C104.2, C104.4, C104.6, C104.8, C112.2, C112.4, C112.6, C112.8, C5.1, C80.1, C88.1, C96.1, U2.4 (GND), U56.4 (GND), U64.4 (GND), U72.12 (GND), U72.9 (~{EN}); no longer J4.2
- net ~{ADC_CS+}: now also U2.6 (A2)
- net ~{ADC_CS-}: now also U2.5 (B2)
- net ~{DAC_CS+}: now also U64.8 (A1)
- net ~{DAC_CS-}: now also U64.7 (B1)
- net ~{LDAC+}: now also U56.8 (A1)
- net ~{LDAC-}: now also U56.7 (B1)
- net ~{Shutdown}: now also J6.6; no longer J4.1
- net SCKI+ renamed SCK+
- net SCK+: now also U64.6 (A2)
- net SCKI- renamed SCK-
- net SCK-: now also U64.5 (B2)
- net SCKO+ renamed SCK_LB+
- net SCK_LB+: now also JP1.1 (A), JP39.1 (A), RN4.2 (R2.1)
- net SCKO- renamed SCK_LB-
- net SCK_LB-: now also JP47.1 (A), JP9.1 (A), RN4.7 (R2.2)
- new net: RN12.4 (R4.1), U72.10 (Out4)
- new net: RN12.3 (R3.1), U72.11 (Out3)
- new net: RN12.2 (R2.1), U72.14 (Out2)
- new net: RN12.1 (R1.1), U72.15 (Out1)
- new net: JP1.2 (B), JP47.2 (B), U72.3 (A2)
- new net: JP39.2 (B), JP9.2 (B), U72.4 (B2)
- new net: C104.1, RN20.5 (R4.2)
- new net: C104.3, RN20.6 (R3.2)
- new net: C104.5, RN20.7 (R2.2)
- new net: C104.7, RN20.8 (R1.2)
- new net: C112.1, RN28.5 (R4.2)
- new net: C112.3, RN28.6 (R3.2)
- new net: C112.5, RN28.7 (R2.2)
- new net: C112.7, RN28.8 (R1.2)
- new net ADC_MISO: RN12.6 (R3.2)
- new net ADC_MOSI: RN20.4 (R4.1), U2.2 (In1)
- new net DAC_MISO: RN12.8 (R1.2)
- new net DAC_MOSI: RN20.2 (R2.1), U56.3 (In2)
- new net SCK: RN28.3 (R3.1), U64.3 (In2)
- new net SCK_LB: RN12.7 (R2.2)
- new net ~{ADC_CS_LB+}: J4.2, RN4.4 (R4.1), U72.7 (A4)
- new net ~{ADC_CS_LB-}: J4.1, RN4.5 (R4.2), U72.8 (B4)
- new net ~{ADC_CS_LB}: RN12.5 (R4.2)
- new net ~{ADC_CS}: RN20.3 (R3.1), U2.3 (In2)
- new net ~{DAC_CS}: RN28.4 (R4.1), U64.2 (In1)
- new net ~{LDAC}: RN20.1 (R1.1), U56.2 (In1)
- no-connect marks 3 -> 4
Other:
- note added: "A"
- note added: "B"
- note added: "C"
- note added: "SCK_LB polarity inverted by default"
- moved on the sheet: C1, C38, C39, D4, J4, J6, J7, Q1, R16, R17, R63, R64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

Commit message: Optical Ethernet, closed-loop response prediction
Backplane: added optical Ethernet interface with transceiver AFBR-5972Z, updated pinout (fixes #44)
Backplane: cleaned up schematic readability slightly (assigned sheet background colors)
Docs: added closed-loop response plotting to compensation script
Other:
- note added: "15 mA max."
- note added: "17 mA max."
Changed lines of the file:
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@@
+		)
+	)
+	(text "17 mA max."
+		(exclude_from_sim no)
+		(at 219.71 106.68 0)
+		(effects
+			(font
+				(size 1.27 1.27)
+			)
+			(justify left)
 		)
 	)
@@
 		)
 	)
+	(text "15 mA max."
+		(exclude_from_sim no)
+		(at 82.55 162.56 0)
+		(effects
+			(font
+				(size 1.27 1.27)
+			)
+			(justify right)
+		)
+	)
 	(text "SCK_LB polarity inverted by default"
 		(exclude_from_sim no)
@@
 			)
 			(justify right bottom)
+		)
+	)
+	(text "17 mA max."
+		(exclude_from_sim no)
+		(at 218.44 157.48 0)
+		(effects
+			(font
+				(size 1.27 1.27)
+			)
+			(justify left)
 		)
 	)
@@
 		)
 	)
+	(text "17 mA max."
+		(exclude_from_sim no)
+		(at 218.44 210.82 0)
+		(effects
+			(font
+				(size 1.27 1.27)
+			)
+			(justify left)
+		)
+	)
