File: pcbs/backplane/backplane.kicad_sch (KiCad schematic)
At the start: 103 parts, among them J1 Conn_01x02, J10 AFBR-2624Z, J11 AFBR-2624Z, J12 AFBR-1624Z, J14 Conn_01x02, J17 Conn_01x02, J19 Conn_01x02, J22 Conn_01x02, J24 Conn_01x02, J27 Conn_01x02, J29 Conn_01x02, J32 Conn_01x02, J34 Conn_01x02, J37 Conn_01x02, J39 Conn_01x02, J42 Conn_01x02, J44 Conn_01x02, J47 Conn_01x02, J48 Conn_01x02, J5 AFBR-2624Z, J8 Conn_01x02, J9 AFBR-2624Z, Q12 MMBT3904, Q13 MMBT3904, U27 74LVC1G14, U29 74LVC1G14

Commit message: Backplane comms updates, manufacturing renaming
Removed misspelled "maunfacturing" folder, fixed gitignore rule to remove manufacturing folders within individual PCB folders too
Changed SCKI/SCKO terminology to SCK, SCK_LB (loopback) for clarity
Added ADC_CS loopback signal between amp ctrl board & backplane for better fast-clock timing (#38)
Backplane: changed LVDS FPGA outputs to single-ended FPGA outputs to gain more I/O pins, added external LVDS transceivers (#38)
Backplane: replaced global clock & ~LDAC buffers with a separate FPGA pin for each amp ctrl board (#38)
Backplane: removed +2.5V power supply and level translations, no longer needed without FPGA I/O pins using LVDS_25 I/O configuration
Backplane: replaced +VDC-input resistor with solder jumper (on by default)
Backplane: changed field names (Part Number to MPN) to match Aisler's naming convention for automatic recognition
Amp ctrl: fixed optional level-shifter circuit on each channel for voltage inputs (#9) schematic & channel-1 layout
Parts:
- removed D5: Green, LED_SMD:LED_0805_2012Metric, symbol Device:LED
- removed R12: 560, Resistor_SMD:R_0805_2012Metric, symbol Device:R
- removed R5: 1 0.25W, Resistor_SMD:R_2010_5025Metric, symbol Device:R
- removed R88: 20K, Resistor_SMD:R_0805_2012Metric, symbol Device:R
- removed R89: 10K, Resistor_SMD:R_0805_2012Metric, symbol Device:R
- added JP55: Jumper_2_Bridged, Jumper:SolderJumper-2_P1.3mm_Bridged_RoundedPad1.0x1.5mm, symbol Jumper:Jumper_2_Bridged
- added TP21, TP23, TP24, TP25, TP27: TestPoint, TestPoint:TestPoint_Pad_D2.0mm, symbol Connector:TestPoint
- C10, C2, C20, C3, C61, C62, C68, C70, C71, C72, C73, C74, C75: MPN (none) -> C0603C104K5RACTU; Part Number C0603C104K5RACTU -> (none)
- C16, C17, C18, C19, C31, C34, C69: MPN (none) -> C0805C105K3RACTU; Part Number C0805C105K3RACTU -> (none)
- C4: MPN (none) -> 865080545012; Part Number 865080545012 -> (none)
- D1: MPN (none) -> PMEG6010CEH,115; Part Number PMEG6010CEH,115 -> (none)
- D2, D3: MPN (none) -> LTST-C171KGKT; Part Number LTST-C171KGKT -> (none)
- D20, D21: MPN (none) -> LTST-C170KRKT; Part Number LTST-C170KRKT -> (none)
- J10, J11, J5, J9: MPN (none) -> AFBR-2624Z; Part Number AFBR-2624Z -> (none)
- J12: MPN (none) -> AFBR-1624Z; Part Number AFBR-1624Z -> (none)
- J14, J19, J24, J29, J34, J39, J44, J48: MPN (none) -> 1190363; Part Number 1190363 -> (none)
- J17, J22, J27, J32, J37, J42, J47, J8: MPN (none) -> 1792229; Part Number 1792229 -> (none)
- L1: MPN (none) -> 2929SQ-501JEC; MPN Alt. (none) -> 2929SQ-501GEC; Part Number 2929SQ-501JEC -> (none); Part Number Alt. 2929SQ-501GEC -> (none)
- Q12, Q13: MPN (none) -> MMBT3904-7-F; MPN Alt. (none) -> MMBT3904,215; Part Number MMBT3904-7-F -> (none); Part Number Alt. MMBT3904,215 -> (none)
- R10, R11, R3, R4, R77: MPN (none) -> RK73H2ATTD1R00F; Part Number RK73H2ATTD1R00F -> (none)
- R13, R81, R82, R90: MPN (none) -> RK73H2ATTD2002F; Part Number RK73H2ATTD2002F -> (none)
- R18: MPN (none) -> RK73H2HTTE1R00F; Part Number RK73H2HTTE1R00F -> (none)
- R6, R7: MPN (none) -> RK73H2BTTD1R00F; Part Number RK73H2BTTD1R00F -> (none)
- R78, R79, R80, R83, R91, R92: MPN (none) -> RK73H2ATTD3301F; Part Number RK73H2ATTD3301F -> (none)
- R8: MPN (none) -> RK73H2ATTD1502F; Part Number RK73H2ATTD1502F -> (none)
- R9: MPN (none) -> RK73H2ATTD1001F; Part Number RK73H2ATTD1001F -> (none)
- TP1, TP2, TP3, TP5: MPN (none) -> 5019; Part Number 5019 -> (none)
- U27, U29: MPN (none) -> SN74LVC1G14DBVR; MPN Alt. (none) -> 74LVC1G14GV,125; Part Number SN74LVC1G14DBVR -> (none); Part Number Alt. 74LVC1G14GV,125 -> (none)
Connections:
- net +VDC: now also JP55.1 (A)
- net Activity Indicator (Trigger)/In: now also TP27.1
- net Power_Enable_Ext: now also TP25.1
- net Power_Enable_FPGA: now also TP24.1
- net Shutdown_Force: now also TP23.1
- net Shutdown_Reset: now also TP21.1
- net at D1.2 (A), R6.1: now also JP55.2 (B)
Other:
- sheet Amp board 0 interface ports: added ADC_MISO, ADC_MOSI, DAC_MISO, DAC_MOSI, SCK, SCK_LB, ~{ADC_CS_LB}, ~{ADC_CS}, ~{DAC_CS}, ~{LDAC}; removed ADC_MISO+, ADC_MISO-, ADC_MOSI+, ADC_MOSI-, DAC_MISO+, DAC_MISO-, DAC_MOSI+, DAC_MOSI-, SCKI+, SCKI-, SCKO+, SCKO-, ~{ADC_CS+}, ~{ADC_CS-}, ~{DAC_CS+}, ~{DAC_CS-}, ~{LDAC+}, ~{LDAC-}
- sheet Amp board 1 interface ports: added ADC_MISO, ADC_MOSI, DAC_MISO, DAC_MOSI, SCK, SCK_LB, ~{ADC_CS_LB}, ~{ADC_CS}, ~{DAC_CS}, ~{LDAC}; removed ADC_MISO+, ADC_MISO-, ADC_MOSI+, ADC_MOSI-, DAC_MISO+, DAC_MISO-, DAC_MOSI+, DAC_MOSI-, SCKI+, SCKI-, SCKO+, SCKO-, ~{ADC_CS+}, ~{ADC_CS-}, ~{DAC_CS+}, ~{DAC_CS-}, ~{LDAC+}, ~{LDAC-}
- sheet Amp board 2 interface ports: added ADC_MISO, ADC_MOSI, DAC_MISO, DAC_MOSI, SCK, SCK_LB, ~{ADC_CS_LB}, ~{ADC_CS}, ~{DAC_CS}, ~{LDAC}; removed ADC_MISO+, ADC_MISO-, ADC_MOSI+, ADC_MOSI-, DAC_MISO+, DAC_MISO-, DAC_MOSI+, DAC_MOSI-, SCKI+, SCKI-, SCKO+, SCKO-, ~{ADC_CS+}, ~{ADC_CS-}, ~{DAC_CS+}, ~{DAC_CS-}, ~{LDAC+}, ~{LDAC-}
- sheet Amp board 3 interface ports: added ADC_MISO, ADC_MOSI, DAC_MISO, DAC_MOSI, SCK, SCK_LB, ~{ADC_CS_LB}, ~{ADC_CS}, ~{DAC_CS}, ~{LDAC}; removed ADC_MISO+, ADC_MISO-, ADC_MOSI+, ADC_MOSI-, DAC_MISO+, DAC_MISO-, DAC_MOSI+, DAC_MOSI-, SCKI+, SCKI-, SCKO+, SCKO-, ~{ADC_CS+}, ~{ADC_CS-}, ~{DAC_CS+}, ~{DAC_CS-}, ~{LDAC+}, ~{LDAC-}
- sheet Amp board 4 interface ports: added ADC_MISO, ADC_MOSI, DAC_MISO, DAC_MOSI, SCK, SCK_LB, ~{ADC_CS_LB}, ~{ADC_CS}, ~{DAC_CS}, ~{LDAC}; removed ADC_MISO+, ADC_MISO-, ADC_MOSI+, ADC_MOSI-, DAC_MISO+, DAC_MISO-, DAC_MOSI+, DAC_MOSI-, SCKI+, SCKI-, SCKO+, SCKO-, ~{ADC_CS+}, ~{ADC_CS-}, ~{DAC_CS+}, ~{DAC_CS-}, ~{LDAC+}, ~{LDAC-}
- sheet Amp board 5 interface ports: added ADC_MISO, ADC_MOSI, DAC_MISO, DAC_MOSI, SCK, SCK_LB, ~{ADC_CS_LB}, ~{ADC_CS}, ~{DAC_CS}, ~{LDAC}; removed ADC_MISO+, ADC_MISO-, ADC_MOSI+, ADC_MOSI-, DAC_MISO+, DAC_MISO-, DAC_MOSI+, DAC_MOSI-, SCKI+, SCKI-, SCKO+, SCKO-, ~{ADC_CS+}, ~{ADC_CS-}, ~{DAC_CS+}, ~{DAC_CS-}, ~{LDAC+}, ~{LDAC-}
- sheet Amp board 6 interface ports: added ADC_MISO, ADC_MOSI, DAC_MISO, DAC_MOSI, SCK, SCK_LB, ~{ADC_CS_LB}, ~{ADC_CS}, ~{DAC_CS}, ~{LDAC}; removed ADC_MISO+, ADC_MISO-, ADC_MOSI+, ADC_MOSI-, DAC_MISO+, DAC_MISO-, DAC_MOSI+, DAC_MOSI-, SCKI+, SCKI-, SCKO+, SCKO-, ~{ADC_CS+}, ~{ADC_CS-}, ~{DAC_CS+}, ~{DAC_CS-}, ~{LDAC+}, ~{LDAC-}
- sheet Amp board 7 interface ports: added ADC_MISO, ADC_MOSI, DAC_MISO, DAC_MOSI, SCK, SCK_LB, ~{ADC_CS_LB}, ~{ADC_CS}, ~{DAC_CS}, ~{LDAC}; removed ADC_MISO+, ADC_MISO-, ADC_MOSI+, ADC_MOSI-, DAC_MISO+, DAC_MISO-, DAC_MOSI+, DAC_MOSI-, SCKI+, SCKI-, SCKO+, SCKO-, ~{ADC_CS+}, ~{ADC_CS-}, ~{DAC_CS+}, ~{DAC_CS-}, ~{LDAC+}, ~{LDAC-}
- sheet FPGA Board, Signal Distribution ports: added ADC_MISO[0..7], ADC_MOSI[0..7], DAC_MISO[0..7], DAC_MOSI[0..7], SCK[0..7], SCK_LB[0..7], ~{ADC_CS[0..7]}, ~{ADC_CS_LB[0..7]}, ~{DAC_CS[0..7]}, ~{LDAC[0..7]}; removed ADC_MISO+[0..7], ADC_MISO-[0..7], ADC_MOSI+[0..7], ADC_MOSI-[0..7], DAC_MISO+[0..7], DAC_MISO-[0..7], DAC_MOSI+[0..7], DAC_MOSI-[0..7], SCKI+[0..7], SCKI-[0..7], SCKO+[0..7], SCKO-[0..7], ~{ADC_CS+[0..7]}, ~{ADC_CS-[0..7]}, ~{DAC_CS+[0..7]}, ~{DAC_CS-[0..7]}, ~{LDAC+[0..7]}, ~{LDAC-[0..7]}
- note added: "160 mW @ 400 mA"
- note removed: "22 mW @ 150 mA"
- moved on the sheet: C69, J5, R77

Commit message: Backplane: changed timer ICs to TLC556 (fixes #45)
Parts:
- added C64: 100nF 50V X7R, Capacitor_SMD:C_0603_1608Metric, symbol Device:C
- added U30: 74LVC1G14, Package_TO_SOT_SMD:SOT-23-5, symbol backplane-rescue:74LVC1G14-Martinos
- added U7: FIN1019MTC, Package_SO:TSSOP-14_4.4x5mm_P0.65mm, symbol Interface:FIN1019MTC
Connections:
- net +3V3: now also C64.2, U30.5 (VCC)
- net GND: now also C64.1, U30.3 (GND)
- net Activitiy Indicator (Rx)/In: no longer names the net of J9.1 (Data_Out), U27.2
- net Activity Indicator (Trigger & 10 Mhz)/In renamed Activity Indicator (Trigger & 10 Mhz)/In2
- net Activity Indicator (Trigger)/In renamed FPGA Board, Signal Distribution/Trigger
- net FPGA Board, Signal Distribution/Trigger: now also U30.2
- net Activity Indicator (Tx & Rx)/In: no longer names the net of J12.4 (Data_in), U29.4
- net FPGA Board, Signal Distribution/UART_Rx_FPGA renamed Activity Indicator (Tx & Rx)/In2
- net FPGA Board, Signal Distribution/UART_Tx_FPGA renamed Activity Indicator (Tx & Rx)/In1
- new net Activity Indicator (Trigger & 10 Mhz)/In1: U30.4
Other:
- sheet Activity Indicator (10 Mhz) renamed Activity Indicator (Trigger & 10 Mhz)
- sheet Activity Indicator (Tx) renamed Activity Indicator (Tx & Rx)
- removed sheet Activitiy Indicator (Rx)
- removed sheet Activity Indicator (Trigger)
- sheet Activity Indicator (Trigger & 10 Mhz) ports: added In1, In2; removed In
- sheet Activity Indicator (Tx & Rx) ports: added In1, In2; removed In
- moved on the sheet: C61, U27

Commit message: Optical Ethernet, closed-loop response prediction
Backplane: added optical Ethernet interface with transceiver AFBR-5972Z, updated pinout (fixes #44)
Backplane: cleaned up schematic readability slightly (assigned sheet background colors)
Docs: added closed-loop response plotting to compensation script
Parts:
- added C121, C29, C30: 10uF 6.3V X7R, Capacitor_SMD:C_0805_2012Metric, symbol Device:C
- added C122, C125, C36, C37, C65, C77: 100nF 50V X7R, Capacitor_SMD:C_0603_1608Metric, symbol Device:C
- added C25, C27, C78: 1uF 50V X7R, Capacitor_SMD:C_0805_2012Metric, symbol Device:C
- added JP34, JP56: Jumper_NC_Small, Jumper:SolderJumper-2_P1.3mm_Bridged_RoundedPad1.0x1.5mm, symbol backplane-rescue:Jumper_NC_Small-Device
- added R12, R48: 1, Resistor_SMD:R_0805_2012Metric, symbol Device:R
- added R49, R51: 150, Resistor_SMD:R_0805_2012Metric, symbol Device:R
- added R52: 100, Resistor_SMD:R_0805_2012Metric, symbol Device:R
- added R53: 10, Resistor_SMD:R_0805_2012Metric, symbol Device:R
- added R54: 15K, Resistor_SMD:R_0805_2012Metric, symbol Device:R
- added R55, R56, R57: 10K, Resistor_SMD:R_0805_2012Metric, symbol Device:R
- added R85, R86: 20K, Resistor_SMD:R_0805_2012Metric, symbol Device:R
- added TP28, TP32: TestPoint, TestPoint:TestPoint_Pad_D1.0mm, symbol Connector:TestPoint
- added TP31: TestPoint, TestPoint:TestPoint_Pad_D2.0mm, symbol Connector:TestPoint
- added U11: AFBR-5972Z, shim:AFBR-5972Z, symbol shim:AFBR-5972Z
- added U32: LMV331, Package_TO_SOT_SMD:SOT-23-5, symbol Comparator:LMV331
- U7: Manufacturer (none) -> ON Semi; Part Number (none) -> FIN1019MTCX
Connections:
- net +3V3: now also C122.2, JP56.1, R12.1, R48.1, R53.1, R55.1, R57.1, U32.5 (V+)
- net GND: now also U7.7 (GND), C121.1, C122.1, C125.1, C25.1, C27.1, C29.1, C30.1, C78.1, JP34.1, R49.1, R51.1, R54.2, R56.2, R86.1, U11.4 (Gnd), U11.S (Shield), U32.2 (V-)
- net at U7.1 (DE): now also JP56.2
- net at U7.10 (RI+): now also C65.1, R52.2, R85.1
- net at U7.11 (DO-): now also C37.1
- net at U7.12 (DO+): now also C36.1
- net at U7.14 (VCC): now also C121.2, C78.2, R53.2, R85.2
- net Eth_Tx: now reaches U7.2 (DI)
- net Eth_Tx: now also TP32.1
- net Eth_Rx: now reaches U7.4 (RO)
- net Eth_Rx: now also TP28.1
- net at U7.8 (~{RE}): now also JP34.2
- net at U7.9 (RI-): now also C77.1, R52.1, R86.2
- new net: C27.2, C30.2, R48.2, U11.3 (TX_Vcc)
- new net: C125.2, R54.1, R55.2, U32.3 (-)
- new net: C25.2, C29.2, R12.2, U11.5 (RX_Vcc)
- new net: C37.2, U11.2 (TData-)
- new net: C36.2, U11.1 (TData+)
- new net: C65.2, R51.2, U11.7 (RData+)
- new net: C77.2, R49.2, U11.8 (RData-)
- new net Eth_SD: R57.2, TP31.1, U32.4
- new net SD: R56.1, U11.6 (SD), U32.1 (+)
Other:
- sheet FPGA Board, Signal Distribution ports: added Eth_Rx, Eth_SD, Eth_Tx; removed none
- note added: "110 mA max."
- note added: "13 mA max."
- note added: "220 mVpp min. input"
- note added: "250-450 mV output (500-900 mVpp?)"
- note added: "500 mV min. output"
- note added: "8.2µF @ 3.3V"
- note added: "LEDs light on falling edges as signal-activity indicators"
- note added: "Noise filter, 1.7 kHz LPF"
- note added: "Noise filter, 17 kHz LPF"
- note added: "±100 mV max. thresholds"
- note removed: "LEDs light on rising edges as signal-activity indicators"
- moved on the sheet: C10, C16, C17, C18, C19, C2, C20, C3, C61, C62, C64, C68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
