File: pcbs/output conn ODU 10x9 32ch/output conn ODU 10x9 32ch.kicad_pcb (KiCad board)
At the start: 4 copper layers, 72 x 104 mm, 9 parts, among them J1 ODU-MAC_Zero_10x9, J2 Conn_02x25_Odd_Even, J3 Conn_02x25_Odd_Even, J4 Conn_02x25_Odd_Even, J5 Conn_02x25_Odd_Even

Commit message: Migrated PCB designs to KiCAD 6
Other:
- net class Default removed
- board text added: "~20 mm spacing between ribbon cable connectors to give ribbon cable some bend radius, and avoid putting upwards pressure on the inner connector"
- board text removed: "~~20 mm spacing between ribbon cable connectors to give ribbon cable some bend radius, and avoid putting upwards pressure on the inner connector"

Commit message: Moved all project-specific symbols & footprints into new "shim" libraries Updated projects to reference the new "shim" library
Parts:
- J1: footprint Martinos:ODU-MAC_Zero_10x9 -> shim:ODU-MAC_Zero_10x9
- J2, J3, J4, J5: footprint Martinos_std:PinHeader_2x25_P2.54mm_Vertical_Shrouded -> shim:PinHeader_2x25_P2.54mm_Vertical_Shrouded
Changed lines of the file:
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@@
 	(net 97 "/P8+")
 	(net 98 "/P8-")
-	(footprint "Martinos_std:PinHeader_2x25_P2.54mm_Vertical_Shrouded"
+	(footprint "shim:PinHeader_2x25_P2.54mm_Vertical_Shrouded"
 		(layer "F.Cu")
 		(at 78.54 73.17 90)
@@
 		)
 		(embedded_fonts no)
-		(model ":Martinos_std:PinHeader_2x25_P2.54mm_Vertical_Shrouded_Sullins_SBH11-_ _ _C-D25-ST-_ _.STEP"
+		(model ":shim:PinHeader_2x25_P2.54mm_Vertical_Shrouded_Sullins_SBH11-_ _ _C-D25-ST-_ _.STEP"
 			(offset
 				(xyz 2.75 0 -3)
@@
 		)
 	)
-	(footprint "Martinos_std:PinHeader_2x25_P2.54mm_Vertical_Shrouded"
+	(footprint "shim:PinHeader_2x25_P2.54mm_Vertical_Shrouded"
 		(layer "F.Cu")
 		(at 78.54 100.79 90)
@@
 		)
 		(embedded_fonts no)
-		(model ":Martinos_std:PinHeader_2x25_P2.54mm_Vertical_Shrouded_Sullins_SBH11-_ _ _C-D25-ST-_ _.STEP"
+		(model ":shim:PinHeader_2x25_P2.54mm_Vertical_Shrouded_Sullins_SBH11-_ _ _C-D25-ST-_ _.STEP"
 			(offset
 				(xyz 2.75 0 -3)
@@
 		)
 	)
-	(footprint "Martinos_std:PinHeader_2x25_P2.54mm_Vertical_Shrouded"
+	(footprint "shim:PinHeader_2x25_P2.54mm_Vertical_Shrouded"
 		(layer "F.Cu")
 		(at 139.5 140.21 -90)
@@
 		)
 		(embedded_fonts no)
-		(model ":Martinos_std:PinHeader_2x25_P2.54mm_Vertical_Shrouded_Sullins_SBH11-_ _ _C-D25-ST-_ _.STEP"
+		(model ":shim:PinHeader_2x25_P2.54mm_Vertical_Shrouded_Sullins_SBH11-_ _ _C-D25-ST-_ _.STEP"
 			(offset
 				(xyz 2.75 0 -3)
@@
 		(embedded_fonts no)
 	)
-	(footprint "Martinos_std:PinHeader_2x25_P2.54mm_Vertical_Shrouded"
+	(footprint "shim:PinHeader_2x25_P2.54mm_Vertical_Shrouded"
 		(layer "F.Cu")
 		(at 139.5 165 -90)
@@
 		)
 		(embedded_fonts no)
-		(model ":Martinos_std:PinHeader_2x25_P2.54mm_Vertical_Shrouded_Sullins_SBH11-_ _ _C-D25-ST-_ _.STEP"
+		(model ":shim:PinHeader_2x25_P2.54mm_Vertical_Shrouded_Sullins_SBH11-_ _ _C-D25-ST-_ _.STEP"
 			(offset
 				(xyz 2.75 0 -3)
@@
 		)
 	)
-	(footprint "Martinos:ODU-MAC_Zero_10x9"
+	(footprint "shim:ODU-MAC_Zero_10x9"
 		(locked yes)
 		(layer "B.Cu")
