File: pcbs/output conn ODU 10x9 32ch/output conn ODU 10x9 32ch.kicad_sch (KiCad schematic)
At the start: 17 parts

Commit message: Updated KiCAD file versions to 9.0
Parts:
- gave numbers to parts that had none: 5

Commit message: Moved all project-specific symbols & footprints into new "shim" libraries Updated projects to reference the new "shim" library
Parts:
- J1: footprint Martinos:ODU-MAC_Zero_10x9 -> shim:ODU-MAC_Zero_10x9
- J2, J3, J4, J5: footprint Martinos_std:PinHeader_2x25_P2.54mm_Vertical_Shrouded -> shim:PinHeader_2x25_P2.54mm_Vertical_Shrouded
Changed lines of the file:
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@@
 			)
 		)
-		(property "Footprint" "Martinos:ODU-MAC_Zero_10x9"
+		(property "Footprint" "shim:ODU-MAC_Zero_10x9"
 			(at 218.44 43.18 0)
 			(effects
@@
 			)
 		)
-		(property "Footprint" "Martinos_std:PinHeader_2x25_P2.54mm_Vertical_Shrouded"
+		(property "Footprint" "shim:PinHeader_2x25_P2.54mm_Vertical_Shrouded"
 			(at 220.98 121.92 0)
 			(effects
@@
 			)
 		)
-		(property "Footprint" "Martinos:ODU-MAC_Zero_10x9"
+		(property "Footprint" "shim:ODU-MAC_Zero_10x9"
 			(at 31.75 43.18 0)
 			(effects
@@
 			)
 		)
-		(property "Footprint" "Martinos:ODU-MAC_Zero_10x9"
+		(property "Footprint" "shim:ODU-MAC_Zero_10x9"
 			(at 58.42 43.18 0)
 			(effects
@@
 			)
 		)
-		(property "Footprint" "Martinos:ODU-MAC_Zero_10x9"
+		(property "Footprint" "shim:ODU-MAC_Zero_10x9"
 			(at 85.09 43.18 0)
 			(effects
@@
 			)
 		)
-		(property "Footprint" "Martinos:ODU-MAC_Zero_10x9"
+		(property "Footprint" "shim:ODU-MAC_Zero_10x9"
 			(at 111.76 43.18 0)
 			(effects
@@
 			)
 		)
-		(property "Footprint" "Martinos:ODU-MAC_Zero_10x9"
+		(property "Footprint" "shim:ODU-MAC_Zero_10x9"
 			(at 138.43 43.18 0)
 			(effects
@@
 			)
 		)
-		(property "Footprint" "Martinos:ODU-MAC_Zero_10x9"
+		(property "Footprint" "shim:ODU-MAC_Zero_10x9"
 			(at 165.1 43.18 0)
 			(effects
@@
 			)
 		)
-		(property "Footprint" "Martinos:ODU-MAC_Zero_10x9"
+		(property "Footprint" "shim:ODU-MAC_Zero_10x9"
 			(at 191.77 43.18 0)
 			(effects
@@
 			)
 		)
-		(property "Footprint" "Martinos:ODU-MAC_Zero_10x9"
+		(property "Footprint" "shim:ODU-MAC_Zero_10x9"
 			(at 245.11 43.18 0)
 			(effects
@@
 			)
 		)
-		(property "Footprint" "Martinos_std:PinHeader_2x25_P2.54mm_Vertical_Shrouded"
+		(property "Footprint" "shim:PinHeader_2x25_P2.54mm_Vertical_Shrouded"
 			(at 72.39 121.92 0)
 			(effects
@@
 			)
 		)
-		(property "Footprint" "Martinos_std:PinHeader_2x25_P2.54mm_Vertical_Shrouded"
+		(property "Footprint" "shim:PinHeader_2x25_P2.54mm_Vertical_Shrouded"
 			(at 123.19 121.92 0)
 			(effects
@@
 			)
 		)
-		(property "Footprint" "Martinos_std:PinHeader_2x25_P2.54mm_Vertical_Shrouded"
+		(property "Footprint" "shim:PinHeader_2x25_P2.54mm_Vertical_Shrouded"
 			(at 172.72 121.92 0)
 			(effects
