File: pcbs/output conn ODU 7x6 16ch fwd/output conn ODU 7x6 16ch fwd.kicad_pcb (KiCad board)
At the start: 4 copper layers, 72 x 114 mm, 43 parts, among them J1 ODU-MAC_Zero_6x7, J2 Conn_02x25_Odd_Even, J3 Conn_02x25_Odd_Even

Commit message: Moved all project-specific symbols & footprints into new "shim" libraries Updated projects to reference the new "shim" library
Parts:
- J1: footprint Don:ODU-MAC_Zero_6x7 -> shim:ODU-MAC_Zero_6x7
- J2, J3: footprint Martinos_std:PinHeader_2x25_P2.54mm_Vertical_Shrouded -> shim:PinHeader_2x25_P2.54mm_Vertical_Shrouded
Changed lines of the file:
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@@
 	(net 46 "unconnected-(J3-Pad26)")
 	(net 47 "unconnected-(J3-Pad25)")
-	(footprint "Martinos_std:PinHeader_2x25_P2.54mm_Vertical_Shrouded"
+	(footprint "shim:PinHeader_2x25_P2.54mm_Vertical_Shrouded"
 		(layer "F.Cu")
 		(at 78.54 79.17 90)
@@
 		)
 		(embedded_fonts no)
-		(model ":Martinos_std:PinHeader_2x25_P2.54mm_Vertical_Shrouded_Sullins_SBH11-_ _ _C-D25-ST-_ _.STEP"
+		(model ":shim:PinHeader_2x25_P2.54mm_Vertical_Shrouded_Sullins_SBH11-_ _ _C-D25-ST-_ _.STEP"
 			(offset
 				(xyz 2.75 0 -3)
@@
 		)
 	)
-	(footprint "Martinos_std:PinHeader_2x25_P2.54mm_Vertical_Shrouded"
+	(footprint "shim:PinHeader_2x25_P2.54mm_Vertical_Shrouded"
 		(layer "F.Cu")
 		(at 139.48 161.71 -90)
@@
 		)
 		(embedded_fonts no)
-		(model ":Martinos_std:PinHeader_2x25_P2.54mm_Vertical_Shrouded_Sullins_SBH11-_ _ _C-D25-ST-_ _.STEP"
+		(model ":shim:PinHeader_2x25_P2.54mm_Vertical_Shrouded_Sullins_SBH11-_ _ _C-D25-ST-_ _.STEP"
 			(offset
 				(xyz 2.75 0 -3)
@@
 		)
 	)
-	(footprint "Don:ODU-MAC_Zero_6x7"
+	(footprint "shim:ODU-MAC_Zero_6x7"
 		(layer "B.Cu")
 		(at 109 119 180)
