File: pcbs/output conn ODU 7x6 16ch fwd/output conn ODU 7x6 16ch fwd.kicad_sch (KiCad schematic)
At the start: 43 parts, among them J1 ODU-MAC_Zero_6x7, J2 Conn_02x25_Odd_Even, J3 Conn_02x25_Odd_Even

Commit message: Moved all project-specific symbols & footprints into new "shim" libraries Updated projects to reference the new "shim" library
Parts:
- J1: footprint Don:ODU-MAC_Zero_6x7 -> shim:ODU-MAC_Zero_6x7; symbol Don:ODU-MAC_Zero_6x7 -> shim:ODU-MAC_Zero_6x7
- J2, J3: footprint Martinos_std:PinHeader_2x25_P2.54mm_Vertical_Shrouded -> shim:PinHeader_2x25_P2.54mm_Vertical_Shrouded
Changed lines of the file:
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@@
 	)
 	(symbol
-		(lib_id "Don:ODU-MAC_Zero_6x7")
+		(lib_id "shim:ODU-MAC_Zero_6x7")
 		(at 29.21 52.07 0)
 		(unit 1)
@@
 			)
 		)
-		(property "Footprint" "Don:ODU-MAC_Zero_6x7"
+		(property "Footprint" "shim:ODU-MAC_Zero_6x7"
 			(at 29.21 53.34 0)
 			(effects
@@
 	)
 	(symbol
-		(lib_id "Don:ODU-MAC_Zero_6x7")
+		(lib_id "shim:ODU-MAC_Zero_6x7")
 		(at 68.58 52.07 0)
 		(unit 2)
@@
 			)
 		)
-		(property "Footprint" "Don:ODU-MAC_Zero_6x7"
+		(property "Footprint" "shim:ODU-MAC_Zero_6x7"
 			(at 68.58 53.34 0)
 			(effects
@@
 	)
 	(symbol
-		(lib_id "Don:ODU-MAC_Zero_6x7")
+		(lib_id "shim:ODU-MAC_Zero_6x7")
 		(at 106.68 52.07 0)
 		(unit 3)
@@
 			)
 		)
-		(property "Footprint" "Don:ODU-MAC_Zero_6x7"
+		(property "Footprint" "shim:ODU-MAC_Zero_6x7"
 			(at 106.68 53.34 0)
 			(effects
@@
 			)
 		)
-		(property "Footprint" "Martinos_std:PinHeader_2x25_P2.54mm_Vertical_Shrouded"
+		(property "Footprint" "shim:PinHeader_2x25_P2.54mm_Vertical_Shrouded"
 			(at 45.72 120.65 0)
 			(effects
@@
 			)
 		)
-		(property "Footprint" "Martinos_std:PinHeader_2x25_P2.54mm_Vertical_Shrouded"
+		(property "Footprint" "shim:PinHeader_2x25_P2.54mm_Vertical_Shrouded"
 			(at 96.52 120.65 0)
 			(effects
