File: pcbs/amp pwr/amp pwr.kicad_pcb (KiCad board)
At the start: 2 copper layers, 290 x 110 mm, 382 parts, among them J1 Conn_02x10_Odd_Even, J10 Conn_02x02_Odd_Even, J11 Conn_02x10_Odd_Even, J12 Conn_02x02_Odd_Even, J13 Conn_02x10_Odd_Even, J14 Conn_02x02_Odd_Even, J15 Conn_02x10_Odd_Even, J16 Conn_02x02_Odd_Even, J17 Conn_02x02_Odd_Even, J18 Conn_02x02_Odd_Even, J19 Conn_02x02_Odd_Even, J2 Conn_02x02_Odd_Even, J20 Conn_02x02_Odd_Even, J3 Conn_02x10_Odd_Even, J4 Conn_02x02_Odd_Even, J5 Conn_02x10_Odd_Even, J6 Conn_02x02_Odd_Even, J7 Conn_02x10_Odd_Even, J8 Conn_02x02_Odd_Even, J9 Conn_02x10_Odd_Even, U1 OPA548, U10 OPA548, U11 OPA548, U12 OPA548, U13 OPA548, U14 OPA548, U15 OPA548, U16 OPA548, U17 TPS7A60, U2 OPA548, U3 OPA548, U4 OPA548, U5 OPA548, U6 OPA548, U7 OPA548, U8 OPA548, U9 OPA548

Commit message: Migrated PCB designs to KiCAD 6
Connections:
- net /Channel 1/~Shutdown1 renamed /Channel 1/~{Shutdown1}
- net /Channel 1/~Shutdown2 renamed /Channel 1/~{Shutdown2}
- net /Channel 2/~Shutdown1 renamed /Channel 2/~{Shutdown1}
- net /Channel 2/~Shutdown2 renamed /Channel 2/~{Shutdown2}
- net /Channel 3/~Shutdown1 renamed /Channel 3/~{Shutdown1}
- net /Channel 3/~Shutdown2 renamed /Channel 3/~{Shutdown2}
- net /Channel 4/~Shutdown1 renamed /Channel 4/~{Shutdown1}
- net /Channel 4/~Shutdown2 renamed /Channel 4/~{Shutdown2}
- net /Channel 5/~Shutdown1 renamed /Channel 5/~{Shutdown1}
- net /Channel 5/~Shutdown2 renamed /Channel 5/~{Shutdown2}
- net /Channel 6/~Shutdown1 renamed /Channel 6/~{Shutdown1}
- net /Channel 6/~Shutdown2 renamed /Channel 6/~{Shutdown2}
- net /Channel 7/~Shutdown1 renamed /Channel 7/~{Shutdown1}
- net /Channel 7/~Shutdown2 renamed /Channel 7/~{Shutdown2}
- net /Channel 8/~Shutdown1 renamed /Channel 8/~{Shutdown1}
- net /Channel 8/~Shutdown2 renamed /Channel 8/~{Shutdown2}
Other:
- net class Default removed
- board text added: "~{Shutdown}"
- board text removed: "~Shutdown"

Commit message: Manufacturing fixes for amp control board
Arranged *.Fab text for assembly drawings
Minor stiffener outline fixes, silkscreen fixes
Fixed missing BOM fields on some parts
Removed exported manufacturing files from version control
Other:
- rule pad_to_mask_clearance: 0.051 -> 0
Changed lines of the file:
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@@
   (title_block
     (title "Shim amplifier, power board")
+    (date "2023-05-04")
     (rev "D2")
     (company "Martinos Center @ MGH")
@@
   )
   (setup
-    (pad_to_mask_clearance 0.051)
-    (solder_mask_min_width 0.25)
+    (stackup
+      (layer "F.SilkS" (type "Top Silk Screen"))
+      (layer "F.Paste" (type "Top Solder Paste"))
+      (layer "F.Mask" (type "Top Solder Mask") (thickness 0.01))
+      (layer "F.Cu" (type "copper") (thickness 0.035))
+      (layer "dielectric 1" (type "core") (thickness 1.51) (material "FR4") (epsilon_r 4.5) (loss_tangent 0.02))
+      (layer "B.Cu" (type "copper") (thickness 0.035))
+      (layer "B.Mask" (type "Bottom Solder Mask") (thickness 0.01))
+      (layer "B.Paste" (type "Bottom Solder Paste"))
+      (layer "B.SilkS" (type "Bottom Silk Screen"))
+      (copper_finish "None")
+      (dielectric_constraints no)
+    )
+    (pad_to_mask_clearance 0)
     (pcbplotparams
-      (layerselection 0x00010a8_7fffffff)
+      (layerselection 0x0020000_7ffffffe)
       (disableapertmacros false)
-      (usegerberextensions false)
+      (usegerberextensions true)
       (usegerberattributes false)
       (usegerberadvancedattributes false)
@@
       (svguseinch false)
       (svgprecision 6)
-      (excludeedgelayer true)
-      (plotframeref false)
+      (excludeedgelayer false)
+      (plotframeref true)
       (viasonmask false)
       (mode 1)
@@
       (plotvalue false)
       (plotinvisibletext false)
-      (sketchpadsonfab false)
+      (sketchpadsonfab true)
       (subtractmaskfromsilk true)
-      (outputformat 1)
+      (outputformat 4)
       (mirror false)
       (drillshape 0)
@@
   (zone (net 155) (net_name "GND") (layer "F.Cu") (hatch edge 0.508)
     (connect_pads (clearance 0.508))
-    (min_thickness 0.254)
+    (min_thickness 0.254) (filled_areas_thickness no)
     (fill yes (thermal_gap 0.508) (thermal_bridge_width 0.508))
     (polygon
@@
     (priority 2)
     (connect_pads yes (clearance 0.4))
-    (min_thickness 0.254)
+    (min_thickness 0.254) (filled_areas_thickness no)
     (fill yes (thermal_gap 0.508) (thermal_bridge_width 0.508))
     (polygon
@@
     (priority 2)
     (connect_pads yes (clearance 0.4))
-    (min_thickness 0.254)
+    (min_thickness 0.254) (filled_areas_thickness no)
     (fill yes (thermal_gap 0.508) (thermal_bridge_width 0.508))
     (polygon
@@
     (priority 2)
     (connect_pads yes (clearance 0.4))
-    (min_thickness 0.254)
+    (min_thickness 0.254) (filled_areas_thickness no)
     (fill yes (thermal_gap 0.508) (thermal_bridge_width 0.508))
     (polygon
@@
     (priority 2)
     (connect_pads yes (clearance 0.4))
-    (min_thickness 0.254)
+    (min_thickness 0.254) (filled_areas_thickness no)
     (fill yes (thermal_gap 0.508) (thermal_bridge_width 0.508))
     (polygon
@@
     (priority 2)
     (connect_pads yes (clearance 0.4))
-    (min_thickness 0.254)
+    (min_thickness 0.254) (filled_areas_thickness no)
     (fill yes (thermal_gap 0.508) (thermal_bridge_width 0.508))
     (polygon
@@
     (priority 2)
     (connect_pads yes (clearance 0.4))
-    (min_thickness 0.254)
+    (min_thickness 0.254) (filled_areas_thickness no)
     (fill yes (thermal_gap 0.508) (thermal_bridge_width 0.508))
     (polygon
@@
     (priority 2)
     (connect_pads yes (clearance 0.4))
-    (min_thickness 0.254)
+    (min_thickness 0.254) (filled_areas_thickness no)
     (fill yes (thermal_gap 0.508) (thermal_bridge_width 0.508))
     (polygon
@@
     (priority 2)
     (connect_pads yes (clearance 0.4))
-    (min_thickness 0.254)
+    (min_thickness 0.254) (filled_areas_thickness no)
     (fill yes (thermal_gap 0.508) (thermal_bridge_width 0.508))
     (polygon
@@
     (priority 2)
     (connect_pads yes (clearance 0.4))
-    (min_thickness 0.254)
+    (min_thickness 0.254) (filled_areas_thickness no)
     (fill yes (thermal_gap 0.508) (thermal_bridge_width 0.508))
     (polygon
@@
     (priority 2)
     (connect_pads yes (clearance 0.4))
-    (min_thickness 0.254)
+    (min_thickness 0.254) (filled_areas_thickness no)
     (fill yes (thermal_gap 0.508) (thermal_bridge_width 0.508))
     (polygon
@@
     (priority 2)
     (connect_pads yes (clearance 0.508))
-    (min_thickness 0.254)
+    (min_thickness 0.254) (filled_areas_thickness no)
     (fill yes (thermal_gap 0.508) (thermal_bridge_width 0.508))
     (polygon
@@
     (priority 2)
     (connect_pads yes (clearance 0.4))
-    (min_thickness 0.254)
+    (min_thickness 0.254) (filled_areas_thickness no)
     (fill yes (thermal_gap 0.508) (thermal_bridge_width 0.508))
     (polygon
@@
     (priority 2)
     (connect_pads yes (clearance 0.4))
-    (min_thickness 0.254)
+    (min_thickness 0.254) (filled_areas_thickness no)
     (fill yes (thermal_gap 0.508) (thermal_bridge_width 0.508))
     (polygon
@@
     (priority 2)
     (connect_pads yes (clearance 0.4))
-    (min_thickness 0.254)
+    (min_thickness 0.254) (filled_areas_thickness no)
     (fill yes (thermal_gap 0.508) (thermal_bridge_width 0.508))
     (polygon
@@
     (priority 2)
     (connect_pads yes (clearance 0.4))
-    (min_thickness 0.254)
+    (min_thickness 0.254) (filled_areas_thickness no)
     (fill yes (thermal_gap 0.508) (thermal_bridge_width 0.508))
     (polygon
@@
     (priority 2)
     (connect_pads yes (clearance 0.4))
-    (min_thickness 0.254)
+    (min_thickness 0.254) (filled_areas_thickness no)
     (fill yes (thermal_gap 0.508) (thermal_bridge_width 0.508))
     (polygon
@@
     (priority 1)
     (connect_pads (clearance 0.4))
-    (min_thickness 0.16)
+    (min_thickness 0.16) (filled_areas_thickness no)
     (fill yes (thermal_gap 0.254) (thermal_bridge_width 0.254))
     (polygon

Commit message: Moved all project-specific symbols & footprints into new "shim" libraries Updated projects to reference the new "shim" library
Parts:
- R17, R18, R27, R28, R37, R38, R47, R48, R57, R58, R67, R68, R7, R77, R78, R8: footprint Martinos:R_Shunt_Vishay_WSR5_KelvinConnection -> shim:R_Shunt_Vishay_WSR5_KelvinConnection
Changed lines of the file:
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@@
 		)
 		(embedded_fonts no)
-		(model ":Martinos:C_Elec_8x12_Nichicon_Polymer.stp"
+		(model ":shim:C_Elec_8x12_Nichicon_Polymer.stp"
 			(offset
 				(xyz 0 0 0)
@@
 		)
 		(embedded_fonts no)
-		(model ":Martinos:C_Elec_8x12_Nichicon_Polymer.stp"
+		(model ":shim:C_Elec_8x12_Nichicon_Polymer.stp"
 			(offset
 				(xyz 0 0 0)
@@
 		)
 	)
-	(footprint "Martinos:R_Shunt_Vishay_WSR5_KelvinConnection"
+	(footprint "shim:R_Shunt_Vishay_WSR5_KelvinConnection"
 		(layer "F.Cu")
 		(at 149.54 63.425 90)
@@
 		)
 		(embedded_fonts no)
-		(model ":Martinos:PinHeader_02x02_Vertical_SMT_Samtec_TSM-102-03-F-DV.stp"
+		(model ":shim:PinHeader_02x02_Vertical_SMT_Samtec_TSM-102-03-F-DV.stp"
 			(offset
 				(xyz 0 0 2.55)
@@
 		)
 		(embedded_fonts no)
-		(model ":Martinos:PinHeader_02x10_Vertical_SMT_Samtec_TSM-110-03-F-DV.stp"
+		(model ":shim:PinHeader_02x10_Vertical_SMT_Samtec_TSM-110-03-F-DV.stp"
 			(offset
 				(xyz 0 0 2.55)
@@
 		)
 	)
-	(footprint "Martinos:R_Shunt_Vishay_WSR5_KelvinConnection"
+	(footprint "shim:R_Shunt_Vishay_WSR5_KelvinConnection"
 		(layer "F.Cu")
 		(at 137.25 102.25 -90)
@@
 		)
 		(embedded_fonts no)
-		(model ":Martinos:C_Elec_8x12_Nichicon_Polymer.stp"
+		(model ":shim:C_Elec_8x12_Nichicon_Polymer.stp"
 			(offset
 				(xyz 0 0 0)
@@
 		)
 		(embedded_fonts no)
-		(model ":Martinos:C_Elec_8x12_Nichicon_Polymer.stp"
+		(model ":shim:C_Elec_8x12_Nichicon_Polymer.stp"
 			(offset
 				(xyz 0 0 0)
@@
 		)
 		(embedded_fonts no)
-		(model ":Martinos:C_Elec_8x12_Nichicon_Polymer.stp"
+		(model ":shim:C_Elec_8x12_Nichicon_Polymer.stp"
 			(offset
 				(xyz 0 0 0)
@@
 		)
 		(embedded_fonts no)
-		(model ":Martinos:C_Elec_8x12_Nichicon_Polymer.stp"
+		(model ":shim:C_Elec_8x12_Nichicon_Polymer.stp"
 			(offset
 				(xyz 0 0 0)
@@
 		)
 		(embedded_fonts no)
-		(model ":Martinos:C_Elec_8x12_Nichicon_Polymer.stp"
+		(model ":shim:C_Elec_8x12_Nichicon_Polymer.stp"
 			(offset
 				(xyz 0 0 0)
@@
 		)
 		(embedded_fonts no)
-		(model ":Martinos:C_Elec_8x12_Nichicon_Polymer.stp"
+		(model ":shim:C_Elec_8x12_Nichicon_Polymer.stp"
 			(offset
 				(xyz 0 0 0)
@@
 		)
 		(embedded_fonts no)
-		(model ":Martinos:C_Elec_8x12_Nichicon_Polymer.stp"
+		(model ":shim:C_Elec_8x12_Nichicon_Polymer.stp"
 			(offset
 				(xyz 0 0 0)
@@
 		)
 		(embedded_fonts no)
-		(model ":Martinos:C_Elec_8x12_Nichicon_Polymer.stp"
+		(model ":shim:C_Elec_8x12_Nichicon_Polymer.stp"
 			(offset
 				(xyz 0 0 0)
@@
 		)
 		(embedded_fonts no)
-		(model ":Martinos:C_Elec_8x12_Nichicon_Polymer.stp"
+		(model ":shim:C_Elec_8x12_Nichicon_Polymer.stp"
 			(offset
 				(xyz 0 0 0)
@@
 		)
 		(embedded_fonts no)
-		(model ":Martinos:C_Elec_8x12_Nichicon_Polymer.stp"
+		(model ":shim:C_Elec_8x12_Nichicon_Polymer.stp"
 			(offset
 				(xyz 0 0 0)
@@
 		)
 		(embedded_fonts no)
-		(model ":Martinos:C_Elec_8x12_Nichicon_Polymer.stp"
+		(model ":shim:C_Elec_8x12_Nichicon_Polymer.stp"
 			(offset
 				(xyz 0 0 0)
@@
 		)
 		(embedded_fonts no)
-		(model ":Martinos:C_Elec_8x12_Nichicon_Polymer.stp"
+		(model ":shim:C_Elec_8x12_Nichicon_Polymer.stp"
 			(offset
 				(xyz 0 0 0)
@@
 		)
 		(embedded_fonts no)
-		(model ":Martinos:C_Elec_8x12_Nichicon_Polymer.stp"
+		(model ":shim:C_Elec_8x12_Nichicon_Polymer.stp"
 			(offset
 				(xyz 0 0 0)
@@
 		)
 		(embedded_fonts no)
-		(model ":Martinos:C_Elec_8x12_Nichicon_Polymer.stp"
+		(model ":shim:C_Elec_8x12_Nichicon_Polymer.stp"
 			(offset
 				(xyz 0 0 0)
@@
 		)
 		(embedded_fonts no)
-		(model ":Martinos:PinHeader_02x10_Vertical_SMT_Samtec_TSM-110-03-F-DV.stp"
+		(model ":shim:PinHeader_02x10_Vertical_SMT_Samtec_TSM-110-03-F-DV.stp"
 			(offset
 				(xyz 0 0 2.55)
@@
 		)
 		(embedded_fonts no)
-		(model ":Martinos:PinHeader_02x02_Vertical_SMT_Samtec_TSM-102-03-F-DV.stp"
+		(model ":shim:PinHeader_02x02_Vertical_SMT_Samtec_TSM-102-03-F-DV.stp"
 			(offset
 				(xyz 0 0 2.55)
@@
 		)
 		(embedded_fonts no)
-		(model ":Martinos:PinHeader_02x10_Vertical_SMT_Samtec_TSM-110-03-F-DV.stp"
+		(model ":shim:PinHeader_02x10_Vertical_SMT_Samtec_TSM-110-03-F-DV.stp"
 			(offset
 				(xyz 0 0 2.55)
@@
 		)
 		(embedded_fonts no)
-		(model ":Martinos:PinHeader_02x02_Vertical_SMT_Samtec_TSM-102-03-F-DV.stp"
+		(model ":shim:PinHeader_02x02_Vertical_SMT_Samtec_TSM-102-03-F-DV.stp"
 			(offset
 				(xyz 0 0 2.55)
@@
 		)
 		(embedded_fonts no)
-		(model ":Martinos:PinHeader_02x10_Vertical_SMT_Samtec_TSM-110-03-F-DV.stp"
+		(model ":shim:PinHeader_02x10_Vertical_SMT_Samtec_TSM-110-03-F-DV.stp"
 			(offset
 				(xyz 0 0 2.55)
@@
 		)
 		(embedded_fonts no)
-		(model ":Martinos:PinHeader_02x02_Vertical_SMT_Samtec_TSM-102-03-F-DV.stp"
+		(model ":shim:PinHeader_02x02_Vertical_SMT_Samtec_TSM-102-03-F-DV.stp"
 			(offset
 				(xyz 0 0 2.55)
@@
 		)
 		(embedded_fonts no)
-		(model ":Martinos:PinHeader_02x10_Vertical_SMT_Samtec_TSM-110-03-F-DV.stp"
+		(model ":shim:PinHeader_02x10_Vertical_SMT_Samtec_TSM-110-03-F-DV.stp"
 			(offset
 				(xyz 0 0 2.55)
@@
 		)
 		(embedded_fonts no)
-		(model ":Martinos:PinHeader_02x02_Vertical_SMT_Samtec_TSM-102-03-F-DV.stp"
+		(model ":shim:PinHeader_02x02_Vertical_SMT_Samtec_TSM-102-03-F-DV.stp"
 			(offset
 				(xyz 0 0 2.55)
@@
 		)
 		(embedded_fonts no)
-		(model ":Martinos:PinHeader_02x10_Vertical_SMT_Samtec_TSM-110-03-F-DV.stp"
+		(model ":shim:PinHeader_02x10_Vertical_SMT_Samtec_TSM-110-03-F-DV.stp"
 			(offset
 				(xyz 0 0 2.55)
@@
 		)
 		(embedded_fonts no)
-		(model ":Martinos:PinHeader_02x02_Vertical_SMT_Samtec_TSM-102-03-F-DV.stp"
+		(model ":shim:PinHeader_02x02_Vertical_SMT_Samtec_TSM-102-03-F-DV.stp"
 			(offset
 				(xyz 0 0 2.55)
@@
 		)
 		(embedded_fonts no)
-		(model ":Martinos:PinHeader_02x10_Vertical_SMT_Samtec_TSM-110-03-F-DV.stp"
+		(model ":shim:PinHeader_02x10_Vertical_SMT_Samtec_TSM-110-03-F-DV.stp"
 			(offset
 				(xyz 0 0 2.55)
@@
 		)
 		(embedded_fonts no)
-		(model ":Martinos:PinHeader_02x02_Vertical_SMT_Samtec_TSM-102-03-F-DV.stp"
+		(model ":shim:PinHeader_02x02_Vertical_SMT_Samtec_TSM-102-03-F-DV.stp"
 			(offset
 				(xyz 0 0 2.55)
@@
 		)
 		(embedded_fonts no)
-		(model ":Martinos:PinHeader_02x10_Vertical_SMT_Samtec_TSM-110-03-F-DV.stp"
+		(model ":shim:PinHeader_02x10_Vertical_SMT_Samtec_TSM-110-03-F-DV.stp"
 			(offset
 				(xyz 0 0 2.55)
@@
 		)
 		(embedded_fonts no)
-		(model ":Martinos:PinHeader_02x02_Vertical_SMT_Samtec_TSM-102-03-F-DV.stp"
+		(model ":shim:PinHeader_02x02_Vertical_SMT_Samtec_TSM-102-03-F-DV.stp"
 			(offset
 				(xyz 0 0 2.55)
@@
 		)
 	)
-	(footprint "Martinos:R_Shunt_Vishay_WSR5_KelvinConnection"
+	(footprint "shim:R_Shunt_Vishay_WSR5_KelvinConnection"
 		(layer "F.Cu")
 		(at 164.5 102.25 -90)
@@
 		)
 	)
-	(footprint "Martinos:R_Shunt_Vishay_WSR5_KelvinConnection"
+	(footprint "shim:R_Shunt_Vishay_WSR5_KelvinConnection"
 		(layer "F.Cu")
 		(at 178.79 63.425 90)
@@
 		)
 	)
-	(footprint "Martinos:R_Shunt_Vishay_WSR5_KelvinConnection"
+	(footprint "shim:R_Shunt_Vishay_WSR5_KelvinConnection"
 		(layer "F.Cu")
 		(at 203.25 102.25 -90)
@@
 		)
 	)
-	(footprint "Martinos:R_Shunt_Vishay_WSR5_KelvinConnection"
+	(footprint "shim:R_Shunt_Vishay_WSR5_KelvinConnection"
 		(layer "F.Cu")
 		(at 215.54 63.425 90)
@@
 		)
 	)
-	(footprint "Martinos:R_Shunt_Vishay_WSR5_KelvinConnection"
+	(footprint "shim:R_Shunt_Vishay_WSR5_KelvinConnection"
 		(layer "F.Cu")
 		(at 230.5 102.25 -90)
@@
 		)
 	)
-	(footprint "Martinos:R_Shunt_Vishay_WSR5_KelvinConnection"
+	(footprint "shim:R_Shunt_Vishay_WSR5_KelvinConnection"
 		(layer "F.Cu")
 		(at 244.79 63.425 90)
@@
 		)
 	)
-	(footprint "Martinos:R_Shunt_Vishay_WSR5_KelvinConnection"
+	(footprint "shim:R_Shunt_Vishay_WSR5_KelvinConnection"
 		(layer "F.Cu")
 		(at 269.25 102.25 -90)
@@
 		)
 	)
-	(footprint "Martinos:R_Shunt_Vishay_WSR5_KelvinConnection"
+	(footprint "shim:R_Shunt_Vishay_WSR5_KelvinConnection"
 		(layer "F.Cu")
 		(at 281.54 63.425 90)
@@
 		)
 	)
-	(footprint "Martinos:R_Shunt_Vishay_WSR5_KelvinConnection"
+	(footprint "shim:R_Shunt_Vishay_WSR5_KelvinConnection"
 		(layer "F.Cu")
 		(at 296.5 102.25 -90)
@@
 		)
 	)
-	(footprint "Martinos:R_Shunt_Vishay_WSR5_KelvinConnection"
+	(footprint "shim:R_Shunt_Vishay_WSR5_KelvinConnection"
 		(layer "F.Cu")
 		(at 310.79 63.425 90)
@@
 		)
 	)
-	(footprint "Martinos:R_Shunt_Vishay_WSR5_KelvinConnection"
+	(footprint "shim:R_Shunt_Vishay_WSR5_KelvinConnection"
 		(layer "F.Cu")
 		(at 335.25 102.25 -90)
@@
 		)
 	)
-	(footprint "Martinos:R_Shunt_Vishay_WSR5_KelvinConnection"
+	(footprint "shim:R_Shunt_Vishay_WSR5_KelvinConnection"
 		(layer "F.Cu")
 		(at 347.54 63.425 90)
@@
 		)
 	)
-	(footprint "Martinos:R_Shunt_Vishay_WSR5_KelvinConnection"
+	(footprint "shim:R_Shunt_Vishay_WSR5_KelvinConnection"
 		(layer "F.Cu")
 		(at 362.5 102.25 -90)
@@
 		)
 	)
-	(footprint "Martinos:R_Shunt_Vishay_WSR5_KelvinConnection"
+	(footprint "shim:R_Shunt_Vishay_WSR5_KelvinConnection"
 		(layer "F.Cu")
 		(at 376.79 63.425 90)
@@
 		)
 		(embedded_fonts no)
-		(model ":Martinos:PinHeader_02x02_Vertical_SMT_Samtec_TSM-102-03-F-DV.stp"
+		(model ":shim:PinHeader_02x02_Vertical_SMT_Samtec_TSM-102-03-F-DV.stp"
 			(offset
 				(xyz 0 0 2.55)
@@
 		)
 		(embedded_fonts no)
-		(model ":Martinos:PinHeader_02x02_Vertical_SMT_Samtec_TSM-102-03-F-DV.stp"
+		(model ":shim:PinHeader_02x02_Vertical_SMT_Samtec_TSM-102-03-F-DV.stp"
 			(offset
 				(xyz 0 0 2.55)
@@
 		)
 		(embedded_fonts no)
-		(model ":Martinos:PinHeader_02x02_Vertical_SMT_Samtec_TSM-102-03-F-DV.stp"
+		(model ":shim:PinHeader_02x02_Vertical_SMT_Samtec_TSM-102-03-F-DV.stp"
 			(offset
 				(xyz 0 0 2.55)
@@
 		)
 		(embedded_fonts no)
-		(model ":Martinos:PinHeader_02x02_Vertical_SMT_Samtec_TSM-102-03-F-DV.stp"
+		(model ":shim:PinHeader_02x02_Vertical_SMT_Samtec_TSM-102-03-F-DV.stp"
 			(offset
 				(xyz 0 0 2.55)

Commit message: Finished migrating footprint names
Parts:
- TP1, TP14, TP38, TP62, TP86: footprint TestPoint:TestPoint_Keystone_5019_Minature -> TestPoint:TestPoint_Keystone_5019_Miniature
Changed lines of the file:
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@@
 		)
 	)
-	(footprint "TestPoint:TestPoint_Keystone_5019_Minature"
+	(footprint "TestPoint:TestPoint_Keystone_5019_Miniature"
 		(layer "F.Cu")
 		(at 125.25 123 180)
@@
 		(embedded_fonts no)
 	)
-	(footprint "TestPoint:TestPoint_Keystone_5019_Minature"
+	(footprint "TestPoint:TestPoint_Keystone_5019_Miniature"
 		(layer "F.Cu")
 		(at 258.25 122.75)
@@
 		(embedded_fonts no)
 	)
-	(footprint "TestPoint:TestPoint_Keystone_5019_Minature"
+	(footprint "TestPoint:TestPoint_Keystone_5019_Miniature"
 		(layer "F.Cu")
 		(at 324.75 122.75)
@@
 		(embedded_fonts no)
 	)
-	(footprint "TestPoint:TestPoint_Keystone_5019_Minature"
+	(footprint "TestPoint:TestPoint_Keystone_5019_Miniature"
 		(layer "F.Cu")
 		(at 391.5 122.75)
@@
 		)
 	)
-	(footprint "TestPoint:TestPoint_Keystone_5019_Minature"
+	(footprint "TestPoint:TestPoint_Keystone_5019_Miniature"
 		(layer "F.Cu")
 		(at 192.75 122.75)
