File: pcbs/amp pwr/amp pwr.kicad_pcb (KiCad board)
At the start: 2 copper layers, 290 x 110 mm, 382 parts, among them J1 Conn_02x10_Odd_Even, J10 Conn_02x02_Odd_Even, J11 Conn_02x10_Odd_Even, J12 Conn_02x02_Odd_Even, J13 Conn_02x10_Odd_Even, J14 Conn_02x02_Odd_Even, J15 Conn_02x10_Odd_Even, J16 Conn_02x02_Odd_Even, J17 Conn_02x02_Odd_Even, J18 Conn_02x02_Odd_Even, J19 Conn_02x02_Odd_Even, J2 Conn_02x02_Odd_Even, J20 Conn_02x02_Odd_Even, J3 Conn_02x10_Odd_Even, J4 Conn_02x02_Odd_Even, J5 Conn_02x10_Odd_Even, J6 Conn_02x02_Odd_Even, J7 Conn_02x10_Odd_Even, J8 Conn_02x02_Odd_Even, J9 Conn_02x10_Odd_Even, U1 OPA548, U10 OPA548, U11 OPA548, U12 OPA548, U13 OPA548, U14 OPA548, U15 OPA548, U16 OPA548, U17 TPS7A60, U2 OPA548, U3 OPA548, U4 OPA548, U5 OPA548, U6 OPA548, U7 OPA548, U8 OPA548, U9 OPA548

Commit message: Amp power board cleanup
Amp power: updated to KiCAD 10
Library: corrected 3D model path for Vishay WSR5 footprint(s)
Library: added Vishay WSR5 footprint variant w/o Kelvin connections as add'l pads
Amp power: removed alignment pin "-A" from male header part numbers (fixes #8)
Amp power: removed vestigial Kelvin connections on resistor footprints
Parts:
- R17, R18, R27, R28, R37, R38, R47, R48, R57, R58, R67, R68, R7, R77, R78, R8: footprint shim:R_Shunt_Vishay_WSR5_KelvinConnection -> shim:R_Shunt_Vishay_WSR5
Connections:
- J18 pad 1: Net-(J18-Pad1) -> unconnected-(J18-Pin_1-Pad1)
- J18 pad 3: Net-(J18-Pad3) -> unconnected-(J18-Pin_3-Pad3)
- J19 pad 1: Net-(J19-Pad1) -> unconnected-(J19-Pin_1-Pad1)
- J19 pad 3: Net-(J19-Pad3) -> unconnected-(J19-Pin_3-Pad3)
- J20 pad 1: Net-(J20-Pad1) -> unconnected-(J20-Pin_1-Pad1)
- J20 pad 3: Net-(J20-Pad3) -> unconnected-(J20-Pin_3-Pad3)
- U17 pad 2: Net-(U17-Pad2) -> unconnected-(U17-~{RST}-Pad2)
- U17 pad 4: Net-(U17-Pad4) -> unconnected-(U17-RDELAY-Pad4)
Routing:
- net Net-(U16-Vo): track 55.1 -> 53.6 mm
- net Net-(U14-Vo): track 54.4 -> 52.9 mm
- net Net-(U12-Vo): track 55.1 -> 53.6 mm
- net Net-(U10-Vo): track 54.4 -> 52.9 mm
- net Net-(U8-Vo): track 55.1 -> 53.6 mm
- net Net-(U6-Vo): track 54.4 -> 52.9 mm
- net Net-(U2-Vo): track 54.6 -> 53.2 mm
- net Net-(U4-Vo): track 55.1 -> 53.6 mm
- net /Channel 8/Out+: track 47.9 -> 47.0 mm
- net /Channel 5/Out+: track 47.9 -> 47.0 mm
- net /Channel 6/Out+: track 47.9 -> 47.1 mm
- net /Channel 4/Out+: track 47.9 -> 47.1 mm
- net /Channel 2/Out+: track 47.9 -> 47.1 mm
- net /Channel 1/Out+: track 47.9 -> 47.1 mm
Other:
- board text added: "Don Straney 2026-08 Martinos Center @ MGH"
- board text added: "Shim Amplifier, Power Board Rev. D3"
- board text removed: "Don Straney 2022-02 Martinos Center @ MGH"
- board text removed: "Shim Amplifier, Power Board Rev. D2"

Commit message: Amp power board re-arrangement for spring pins
Moved channel circuitry, particularly bulk caps, closer to board edge to make room for spring pin arrangement
Updated 3D model assignments
Parts:
- removed R10, R19, R20, R29, R30, R39, R40, R49, R50, R59, R60, R69, R70, R79, R80, R9: 0, Resistor_SMD:R_0603_1608Metric
- removed R14, R24, R34, R4, R44, R54, R64, R74: 0, Resistor_SMD:R_1206_3216Metric
- moved D10 18.6 mm to (220.8, 72.5), turned to 0 degrees
- moved D14 18.6 mm to (250.0, 72.5), turned to 0 degrees
- moved D18 18.6 mm to (286.8, 72.5), turned to 0 degrees
- moved D2 18.6 mm to (154.8, 72.5), turned to 0 degrees
- moved D22 18.6 mm to (316.0, 72.5), turned to 0 degrees
- moved D26 18.6 mm to (352.8, 72.5), turned to 0 degrees
- moved D30 18.6 mm to (382.0, 72.5), turned to 0 degrees
- moved D6 18.6 mm to (184.0, 72.5), turned to 0 degrees
- moved C12 17.6 mm to (140.5, 53.8)
- moved C24 17.6 mm to (169.8, 53.8)
- moved C36 17.6 mm to (206.5, 53.8)
- moved C48 17.6 mm to (235.8, 53.8)
- moved C60 17.6 mm to (272.5, 53.8)
- moved C72 17.6 mm to (301.8, 53.8)
- moved C84 17.6 mm to (338.5, 53.8)
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Connections:
- C15 pad 1: Net-(U4-Vo) -> /Channel 2/CS+
- C27 pad 1: Net-(U6-Vo) -> /Channel 3/CS+
- C3 pad 1: Net-(U2-Vo) -> /Channel 1/CS+
- C39 pad 1: Net-(U8-Vo) -> /Channel 4/CS+
- C51 pad 1: Net-(U10-Vo) -> /Channel 5/CS+
- C63 pad 1: Net-(U12-Vo) -> /Channel 6/CS+
- C75 pad 1: Net-(U14-Vo) -> /Channel 7/CS+
- C87 pad 1: Net-(U16-Vo) -> /Channel 8/CS+
- D1 pad 2: /Channel 1/Out+ -> /Channel 1/CS-
- D10 pad 1: /Channel 3/Out+ -> /Channel 3/CS-
- D13 pad 2: /Channel 4/Out+ -> /Channel 4/CS-
- D14 pad 1: /Channel 4/Out+ -> /Channel 4/CS-
- D17 pad 2: /Channel 5/Out+ -> /Channel 5/CS-
- D18 pad 1: /Channel 5/Out+ -> /Channel 5/CS-
- D2 pad 1: /Channel 1/Out+ -> /Channel 1/CS-
- D21 pad 2: /Channel 6/Out+ -> /Channel 6/CS-
- D22 pad 1: /Channel 6/Out+ -> /Channel 6/CS-
- D25 pad 2: /Channel 7/Out+ -> /Channel 7/CS-
- D26 pad 1: /Channel 7/Out+ -> /Channel 7/CS-
- D29 pad 2: /Channel 8/Out+ -> /Channel 8/CS-
- D30 pad 1: /Channel 8/Out+ -> /Channel 8/CS-
- D5 pad 2: /Channel 2/Out+ -> /Channel 2/CS-
- D6 pad 1: /Channel 2/Out+ -> /Channel 2/CS-
- D9 pad 2: /Channel 3/Out+ -> /Channel 3/CS-
- J1 pad 16: /Channel 1/Out+ -> /Channel 1/CS-
- J1 pad 18: /Channel 1/Out+ -> /Channel 1/CS-
- J11 pad 16: /Channel 6/Out+ -> /Channel 6/CS-
- J11 pad 18: /Channel 6/Out+ -> /Channel 6/CS-
- J13 pad 16: /Channel 7/Out+ -> /Channel 7/CS-
- J13 pad 18: /Channel 7/Out+ -> /Channel 7/CS-
- J15 pad 16: /Channel 8/Out+ -> /Channel 8/CS-
- J15 pad 18: /Channel 8/Out+ -> /Channel 8/CS-
- J3 pad 16: /Channel 2/Out+ -> /Channel 2/CS-
- J3 pad 18: /Channel 2/Out+ -> /Channel 2/CS-
- J5 pad 16: /Channel 3/Out+ -> /Channel 3/CS-
- J5 pad 18: /Channel 3/Out+ -> /Channel 3/CS-
- J7 pad 16: /Channel 4/Out+ -> /Channel 4/CS-
- J7 pad 18: /Channel 4/Out+ -> /Channel 4/CS-
- J9 pad 16: /Channel 5/Out+ -> /Channel 5/CS-
- J9 pad 18: /Channel 5/Out+ -> /Channel 5/CS-
- R15 pad 1: Net-(U4-Vo) -> /Channel 2/CS+
- R18 pad 1: /Channel 2/Out+ -> /Channel 2/CS-
- R18 pad 2: Net-(U4-Vo) -> /Channel 2/CS+
- R25 pad 1: Net-(U6-Vo) -> /Channel 3/CS+
- R28 pad 1: /Channel 3/Out+ -> /Channel 3/CS-
- R28 pad 2: Net-(U6-Vo) -> /Channel 3/CS+
- R35 pad 1: Net-(U8-Vo) -> /Channel 4/CS+
- R38 pad 1: /Channel 4/Out+ -> /Channel 4/CS-
- R38 pad 2: Net-(U8-Vo) -> /Channel 4/CS+
- R45 pad 1: Net-(U10-Vo) -> /Channel 5/CS+
- R48 pad 1: /Channel 5/Out+ -> /Channel 5/CS-
- R48 pad 2: Net-(U10-Vo) -> /Channel 5/CS+
- R5 pad 1: Net-(U2-Vo) -> /Channel 1/CS+
- R55 pad 1: Net-(U12-Vo) -> /Channel 6/CS+
- R58 pad 1: /Channel 6/Out+ -> /Channel 6/CS-
- R58 pad 2: Net-(U12-Vo) -> /Channel 6/CS+
- R65 pad 1: Net-(U14-Vo) -> /Channel 7/CS+
- R68 pad 1: /Channel 7/Out+ -> /Channel 7/CS-
- R68 pad 2: Net-(U14-Vo) -> /Channel 7/CS+
- R75 pad 1: Net-(U16-Vo) -> /Channel 8/CS+
- R78 pad 1: /Channel 8/Out+ -> /Channel 8/CS-
- R78 pad 2: Net-(U16-Vo) -> /Channel 8/CS+
- R8 pad 1: /Channel 1/Out+ -> /Channel 1/CS-
- R8 pad 2: Net-(U2-Vo) -> /Channel 1/CS+
- R82 pad 2: Net-(U2-Vo) -> /Channel 1/CS+
- R84 pad 2: Net-(U4-Vo) -> /Channel 2/CS+
- R86 pad 2: Net-(U6-Vo) -> /Channel 3/CS+
- R88 pad 2: Net-(U8-Vo) -> /Channel 4/CS+
- R90 pad 2: Net-(U10-Vo) -> /Channel 5/CS+
- R92 pad 2: Net-(U12-Vo) -> /Channel 6/CS+
- R94 pad 2: Net-(U14-Vo) -> /Channel 7/CS+
- R96 pad 2: Net-(U16-Vo) -> /Channel 8/CS+
- TP12 pad 1: Net-(U2-Vo) -> /Channel 1/CS+
- TP24 pad 1: Net-(U4-Vo) -> /Channel 2/CS+
- TP36 pad 1: Net-(U6-Vo) -> /Channel 3/CS+
- TP48 pad 1: Net-(U8-Vo) -> /Channel 4/CS+
- TP60 pad 1: Net-(U10-Vo) -> /Channel 5/CS+
- TP72 pad 1: Net-(U12-Vo) -> /Channel 6/CS+
- TP84 pad 1: Net-(U14-Vo) -> /Channel 7/CS+
- TP96 pad 1: Net-(U16-Vo) -> /Channel 8/CS+
- U10 pad 6: Net-(U10-Vo) -> /Channel 5/CS+
- U10 pad 7: Net-(U10-E/S) -> /Channel 5/~{Shutdown1}
- U12 pad 6: Net-(U12-Vo) -> /Channel 6/CS+
- U12 pad 7: Net-(U12-E/S) -> /Channel 6/~{Shutdown1}
- U14 pad 6: Net-(U14-Vo) -> /Channel 7/CS+
- U14 pad 7: Net-(U14-E/S) -> /Channel 7/~{Shutdown1}
- U16 pad 6: Net-(U16-Vo) -> /Channel 8/CS+
- U16 pad 7: Net-(U16-E/S) -> /Channel 8/~{Shutdown1}
- U2 pad 6: Net-(U2-Vo) -> /Channel 1/CS+
- U2 pad 7: Net-(U2-E/S) -> /Channel 1/~{Shutdown1}
- U4 pad 6: Net-(U4-Vo) -> /Channel 2/CS+
- U4 pad 7: Net-(U4-E/S) -> /Channel 2/~{Shutdown1}
- U6 pad 6: Net-(U6-Vo) -> /Channel 3/CS+
- U6 pad 7: Net-(U6-E/S) -> /Channel 3/~{Shutdown1}
- U8 pad 6: Net-(U8-Vo) -> /Channel 4/CS+
- U8 pad 7: Net-(U8-E/S) -> /Channel 4/~{Shutdown1}
Routing:
- net GNDPWR: track 181.7 -> 126.2 mm
- net Net-(U4-Vo): track 53.6 -> 0.00 mm
- net Net-(U8-Vo): track 53.6 -> 0.00 mm
- net Net-(U16-Vo): track 53.6 -> 0.00 mm
- net Net-(U12-Vo): track 53.6 -> 0.00 mm
- net Net-(U2-Vo): track 53.2 -> 0.00 mm
- net Net-(U14-Vo): track 52.9 -> 0.00 mm
- net Net-(U10-Vo): track 52.9 -> 0.00 mm
- net Net-(U6-Vo): track 52.9 -> 0.00 mm
- net /Channel 3/CS+: track 21.3 -> 74.2 mm
- net /Channel 4/CS+: track 21.3 -> 74.2 mm
- net /Channel 2/CS+: track 21.3 -> 74.2 mm
- net /Channel 1/CS+: track 21.3 -> 74.2 mm
- net /Channel 8/CS+: track 21.3 -> 74.2 mm
- net /Channel 6/CS+: track 21.3 -> 74.2 mm
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
Commit message: Added footprints and started layout of interposer board
Parts:
- moved C1 30.5 mm to (128.0, 135.8)
- moved C101 30.5 mm to (180.8, 141.8)
- moved C103 30.5 mm to (210.0, 141.8)
- moved C105 30.5 mm to (246.8, 141.8)
- moved C107 30.5 mm to (276.0, 141.8)
- moved C109 30.5 mm to (312.8, 141.8)
- moved C11 30.5 mm to (121.5, 130.1)
- moved C111 30.5 mm to (342.0, 141.8)
- moved C13 30.5 mm to (157.2, 135.8)
- moved C16 30.5 mm to (161.5, 135.8)
- moved C17 30.5 mm to (152.2, 136.3)
- moved C23 30.5 mm to (150.8, 130.1)
- moved C25 30.5 mm to (194.0, 135.8)
- moved C28 30.5 mm to (198.2, 135.8)
- moved C29 30.5 mm to (189.0, 136.3)
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