File: pcbs/amp pwr/amp pwr.kicad_sch (KiCad schematic)
At the start: 38 parts, among them J17 Conn_02x02_Odd_Even, J18 Conn_02x02_Odd_Even, J19 Conn_02x02_Odd_Even, J20 Conn_02x02_Odd_Even, U17 TPS7A60

Commit message: Amp power board cleanup
Amp power: updated to KiCAD 10
Library: corrected 3D model path for Vishay WSR5 footprint(s)
Library: added Vishay WSR5 footprint variant w/o Kelvin connections as add'l pads
Amp power: removed alignment pin "-A" from male header part numbers (fixes #8)
Amp power: removed vestigial Kelvin connections on resistor footprints
Parts:
- H1, H10, H11, H12, H13, H14, H15, H16, H17, H18, H2, H21, H24, H29, H3, H32, H4, H5, H6, H7, H8, H9: now left out of the parts list
- J17, J18, J19, J20: Part Number TSM-102-03-L-DV-A -> TSM-102-03-L-DV
