File: pcbs/amp pwr/channel.kicad_sch (KiCad schematic)
At the start: 43 parts, among them J1 Conn_02x10_Odd_Even, J2 Conn_02x02_Odd_Even, U1 OPA548, U2 OPA548

Commit message: Amp power board cleanup
Amp power: updated to KiCAD 10
Library: corrected 3D model path for Vishay WSR5 footprint(s)
Library: added Vishay WSR5 footprint variant w/o Kelvin connections as add'l pads
Amp power: removed alignment pin "-A" from male header part numbers (fixes #8)
Amp power: removed vestigial Kelvin connections on resistor footprints
Parts:
- J1: Part Number TSM-110-03-L-DV-A -> TSM-110-03-L-DV
- J2: Part Number TSM-102-03-L-DV-A -> TSM-102-03-L-DV
- R7, R8: footprint shim:R_Shunt_Vishay_WSR5_KelvinConnection -> shim:R_Shunt_Vishay_WSR5
- TP10, TP11, TP12, TP3, TP4, TP5, TP6, TP7, TP8, TP9: now left out of the parts list

Commit message: Amp power board re-arrangement for spring pins
Moved channel circuitry, particularly bulk caps, closer to board edge to make room for spring pin arrangement
Updated 3D model assignments
Parts:
- removed R10, R9: 0, Resistor_SMD:R_0603_1608Metric, symbol Device:R
- removed R4: 0, Resistor_SMD:R_1206_3216Metric, symbol Device:R
Connections:
- net Out+ is gone; now on net CS-: D1.2 (A), D2.1 (K), J1.16 (Pin_16), J1.18 (Pin_18), R8.1
- net CS+: now also C3.1, R5.1, R8.2, R82.2, TP12.1, U2.6 (Vo)
- net ~{Shutdown1}: now also U2.7 (E/S)
Other:
- note removed: "Used as jumper in layout"

Commit message: Spring connector layout updates
Amp ctrl: added spring connectors for current sense, thermistors, +5V regulator
Amp ctrl: changed pass-through screwdriver holes to mounting holes
Amp ctrl: added part number to optional level shifter
Amp pwr: marked DNP components as DNP
Parts:
- C3, C4, R2: now not fitted
Changed lines of the file:
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@@
 		(on_board yes)
 		(in_pos_files yes)
-		(dnp no)
+		(dnp yes)
 		(property "Reference" "R2"
 			(at 207.518 115.6716 0)
@@
 		(on_board yes)
 		(in_pos_files yes)
-		(dnp no)
+		(dnp yes)
 		(property "Reference" "C3"
 			(at 227.33 114.2492 90)
@@
 		(on_board yes)
 		(in_pos_files yes)
-		(dnp no)
+		(dnp yes)
 		(property "Reference" "C4"
 			(at 228.6 214.5792 90)
