File: pcbs/amp_interposer/amp_interposer.kicad_sch (KiCad schematic)
At the start: 0 parts

Commit message: Added footprints and started layout of interposer board
Parts:
- added J74: Conn_02x02, shim:PinSocket_2x02_P2.54mm_Vertical_SMD_BotEntry_Pin, symbol Connector_Generic:Conn_02x02_Odd_Even
- added J75, J76: Conn_01x02, shim:Conn_70AAJ-M_SIB_1x02_P2.54mm_M, symbol Connector_Generic:Conn_01x02
Connections:
- new net +5V: J74.2 (Pin_2), J75.1 (Pin_1)
- new net +VDC: J74.1 (Pin_1), J76.2 (Pin_2)
- new net GND: J74.3 (Pin_3), J74.4 (Pin_4), J75.2 (Pin_2), J76.1 (Pin_1)
Other:
- added sheet Channel 1 (channel.kicad_sch)
- added sheet Channel 2 (channel.kicad_sch)
- added sheet Channel 3 (channel.kicad_sch)
- added sheet Channel 4 (channel.kicad_sch)
- added sheet Channel 5 (channel.kicad_sch)
- added sheet Channel 6 (channel.kicad_sch)
- added sheet Channel 7 (channel.kicad_sch)
- added sheet Channel 8 (channel.kicad_sch)
- added sheet Thermistor 1 (therminstor_conn.kicad_sch)
- added sheet Thermistor 2 (therminstor_conn.kicad_sch)
- added sheet Thermistor 3 (therminstor_conn.kicad_sch)
- note added: "Amp Control"
- note added: "Power Header F (Power Board)"
- note added: "Spring Pins M (Amp Board)"
- note added: "Thermistor Connectors"
