File: pcbs/amp_interposer/amp_interposer.kicad_pcb (KiCad board)
At the start: 2 copper layers, 12 parts

Commit message: Added footprints and started layout of interposer board
Parts:
- added J1: Conn_01x05, shim:Conn_70AAJ-M_SIB_1x05_P2.54mm_M, F.Cu at (111.9, 108.0)
- added J10: Conn_01x05, shim:Conn_70AAJ-M_SIB_1x05_P2.54mm_M, F.Cu at (152.5, 111.7)
- added J11: Conn_01x02, shim:Conn_70AAJ-M_SIB_1x02_P2.54mm_M, F.Cu at (148.3, 46.5)
- added J12: Conn_02x10_Odd_Even, shim:PinSocket_2x10_P2.54mm_Vertical_SMD_BotEntry_Pin, B.Cu at (147.5, 100.8)
- added J13: Conn_02x02, shim:PinSocket_2x02_P2.54mm_Vertical_SMD_BotEntry_Pin, B.Cu at (155.0, 61.8)
- added J14: Conn_01x05, shim:Conn_70AAJ-M_SIB_1x05_P2.54mm_M, F.Cu at (139.6, 89.3)
- added J15: Conn_01x05, shim:Conn_70AAJ-M_SIB_1x05_P2.54mm_M, F.Cu at (152.2, 89.3)
- added J16: Conn_01x02, shim:Conn_70AAJ-M_SIB_1x02_P2.54mm_M, F.Cu at (148.3, 53.4)
- added J17: Conn_01x05, shim:Conn_70AAJ-M_SIB_1x05_P2.54mm_M, F.Cu at (176.8, 111.7)
- added J18: Conn_01x05, shim:Conn_70AAJ-M_SIB_1x05_P2.54mm_M, F.Cu at (189.5, 111.7)
- added J19: Conn_01x02, shim:Conn_70AAJ-M_SIB_1x02_P2.54mm_M, F.Cu at (191.3, 45.7)
- added J2: Conn_01x05, shim:Conn_70AAJ-M_SIB_1x05_P2.54mm_M, F.Cu at (124.6, 108.0)
- added J20: Conn_02x10_Odd_Even, shim:PinSocket_2x10_P2.54mm_Vertical_SMD_BotEntry_Pin, B.Cu at (184.2, 100.8)
- added J21: Conn_02x02, shim:PinSocket_2x02_P2.54mm_Vertical_SMD_BotEntry_Pin, B.Cu at (191.8, 61.8)
- added J22: Conn_01x05, shim:Conn_70AAJ-M_SIB_1x05_P2.54mm_M, F.Cu at (178.6, 88.3)
- added J23: Conn_01x05, shim:Conn_70AAJ-M_SIB_1x05_P2.54mm_M, F.Cu at (191.2, 88.3)
- added J24: Conn_01x02, shim:Conn_70AAJ-M_SIB_1x02_P2.54mm_M, F.Cu at (191.6, 52.8)
- added J25: Conn_01x05, shim:Conn_70AAJ-M_SIB_1x05_P2.54mm_M, F.Cu at (205.8, 111.7)
- added J26: Conn_01x05, shim:Conn_70AAJ-M_SIB_1x05_P2.54mm_M, F.Cu at (218.5, 111.7)
- added J27: Conn_01x02, shim:Conn_70AAJ-M_SIB_1x02_P2.54mm_M, F.Cu at (215.8, 47.5)
- added J28: Conn_02x10_Odd_Even, shim:PinSocket_2x10_P2.54mm_Vertical_SMD_BotEntry_Pin, B.Cu at (213.5, 100.8)
- added J29: Conn_02x02, shim:PinSocket_2x02_P2.54mm_Vertical_SMD_BotEntry_Pin, B.Cu at (221.0, 61.8)
- added J3: Conn_01x02, shim:Conn_70AAJ-M_SIB_1x02_P2.54mm_M, F.Cu at (134.5, 56.9)
- added J30: Conn_01x05, shim:Conn_70AAJ-M_SIB_1x05_P2.54mm_M, F.Cu at (206.6, 88.3)
- added J31: Conn_01x05, shim:Conn_70AAJ-M_SIB_1x05_P2.54mm_M, F.Cu at (219.2, 88.3)
- added J32: Conn_01x02, shim:Conn_70AAJ-M_SIB_1x02_P2.54mm_M, F.Cu at (222.8, 47.5)
- added J33: Conn_01x05, shim:Conn_70AAJ-M_SIB_1x05_P2.54mm_M, F.Cu at (241.8, 112.7)
- added J34: Conn_01x05, shim:Conn_70AAJ-M_SIB_1x05_P2.54mm_M, F.Cu at (254.5, 112.7)
- added J35: Conn_01x02, shim:Conn_70AAJ-M_SIB_1x02_P2.54mm_M, F.Cu at (253.1, 49.5)
- added J36: Conn_02x10_Odd_Even, shim:PinSocket_2x10_P2.54mm_Vertical_SMD_BotEntry_Pin, B.Cu at (250.2, 100.8)
- added J37: Conn_02x02, shim:PinSocket_2x02_P2.54mm_Vertical_SMD_BotEntry_Pin, B.Cu at (257.8, 61.8)
- added J38: Conn_01x05, shim:Conn_70AAJ-M_SIB_1x05_P2.54mm_M, F.Cu at (243.6, 88.3)
- added J39: Conn_01x05, shim:Conn_70AAJ-M_SIB_1x05_P2.54mm_M, F.Cu at (256.2, 88.3)
- added J4: Conn_02x10_Odd_Even, shim:PinSocket_2x10_P2.54mm_Vertical_SMD_BotEntry_Pin, B.Cu at (118.2, 100.8)
- added J40: Conn_01x02, shim:Conn_70AAJ-M_SIB_1x02_P2.54mm_M, F.Cu at (260.0, 49.5)
- added J41: Conn_01x05, shim:Conn_70AAJ-M_SIB_1x05_P2.54mm_M, F.Cu at (271.8, 112.7)
- added J42: Conn_01x05, shim:Conn_70AAJ-M_SIB_1x05_P2.54mm_M, F.Cu at (284.5, 112.7)
- added J43: Conn_01x02, shim:Conn_70AAJ-M_SIB_1x02_P2.54mm_M, F.Cu at (279.7, 49.5)
- added J44: Conn_02x10_Odd_Even, shim:PinSocket_2x10_P2.54mm_Vertical_SMD_BotEntry_Pin, B.Cu at (279.5, 100.8)
- added J45: Conn_02x02, shim:PinSocket_2x02_P2.54mm_Vertical_SMD_BotEntry_Pin, B.Cu at (287.0, 61.8)
- added J46: Conn_01x05, shim:Conn_70AAJ-M_SIB_1x05_P2.54mm_M, F.Cu at (273.6, 89.3)
- added J47: Conn_01x05, shim:Conn_70AAJ-M_SIB_1x05_P2.54mm_M, F.Cu at (286.2, 89.3)
- added J48: Conn_01x02, shim:Conn_70AAJ-M_SIB_1x02_P2.54mm_M, F.Cu at (286.7, 49.5)
- added J49: Conn_01x05, shim:Conn_70AAJ-M_SIB_1x05_P2.54mm_M, F.Cu at (307.8, 112.7)
- added J5: Conn_02x02, shim:PinSocket_2x02_P2.54mm_Vertical_SMD_BotEntry_Pin, B.Cu at (125.8, 61.8)
- added J50: Conn_01x05, shim:Conn_70AAJ-M_SIB_1x05_P2.54mm_M, F.Cu at (320.5, 112.7)
- added J51: Conn_01x02, shim:Conn_70AAJ-M_SIB_1x02_P2.54mm_M, F.Cu at (320.8, 49.5)
- added J52: Conn_02x10_Odd_Even, shim:PinSocket_2x10_P2.54mm_Vertical_SMD_BotEntry_Pin, B.Cu at (316.2, 100.8)
- added J53: Conn_02x02, shim:PinSocket_2x02_P2.54mm_Vertical_SMD_BotEntry_Pin, B.Cu at (323.8, 61.8)
- added J54: Conn_01x05, shim:Conn_70AAJ-M_SIB_1x05_P2.54mm_M, F.Cu at (309.6, 89.3)
- added J55: Conn_01x05, shim:Conn_70AAJ-M_SIB_1x05_P2.54mm_M, F.Cu at (322.2, 89.3)
- added J56: Conn_01x02, shim:Conn_70AAJ-M_SIB_1x02_P2.54mm_M, F.Cu at (327.8, 49.5)
- added J57: Conn_01x05, shim:Conn_70AAJ-M_SIB_1x05_P2.54mm_M, F.Cu at (338.8, 113.7)
- added J58: Conn_01x05, shim:Conn_70AAJ-M_SIB_1x05_P2.54mm_M, F.Cu at (351.5, 113.7)
- added J59: Conn_01x02, shim:Conn_70AAJ-M_SIB_1x02_P2.54mm_M, F.Cu at (348.2, 49.9)
- added J6: Conn_01x05, shim:Conn_70AAJ-M_SIB_1x05_P2.54mm_M, F.Cu at (111.9, 93.6)
- added J60: Conn_02x10_Odd_Even, shim:PinSocket_2x10_P2.54mm_Vertical_SMD_BotEntry_Pin, B.Cu at (345.5, 100.8)
- added J61: Conn_02x02, shim:PinSocket_2x02_P2.54mm_Vertical_SMD_BotEntry_Pin, B.Cu at (353.0, 61.8)
- added J62: Conn_01x05, shim:Conn_70AAJ-M_SIB_1x05_P2.54mm_M, F.Cu at (338.6, 88.3)
- added J63: Conn_01x05, shim:Conn_70AAJ-M_SIB_1x05_P2.54mm_M, F.Cu at (351.2, 88.3)
- added J64: Conn_01x02, shim:Conn_70AAJ-M_SIB_1x02_P2.54mm_M, F.Cu at (355.1, 49.9)
- added J68: Conn_02x02, shim:PinSocket_2x02_P2.54mm_Vertical_SMD_BotEntry_Pin, B.Cu at (100.0, 100.8)
- added J69: Conn_01x02, shim:Conn_70AAJ-M_SIB_1x02_P2.54mm_M, F.Cu at (100.0, 93.6)
- added J7: Conn_01x05, shim:Conn_70AAJ-M_SIB_1x05_P2.54mm_M, F.Cu at (124.7, 93.6)
- added J70: Conn_02x02, shim:PinSocket_2x02_P2.54mm_Vertical_SMD_BotEntry_Pin, B.Cu at (231.8, 100.8)
- added J71: Conn_01x02, shim:Conn_70AAJ-M_SIB_1x02_P2.54mm_M, F.Cu at (231.8, 88.0)
- added J72: Conn_02x02, shim:PinSocket_2x02_P2.54mm_Vertical_SMD_BotEntry_Pin, B.Cu at (363.5, 100.8)
- added J73: Conn_01x02, shim:Conn_70AAJ-M_SIB_1x02_P2.54mm_M, F.Cu at (364.0, 87.7)
- added J74: Conn_02x02, shim:PinSocket_2x02_P2.54mm_Vertical_SMD_BotEntry_Pin, B.Cu at (87.0, 49.5)
- added J75: Conn_01x02, shim:Conn_70AAJ-M_SIB_1x02_P2.54mm_M, F.Cu at (81.7, 58.3)
- added J76: Conn_01x02, shim:Conn_70AAJ-M_SIB_1x02_P2.54mm_M, F.Cu at (92.0, 58.2)
- added J8: Conn_01x02, shim:Conn_70AAJ-M_SIB_1x02_P2.54mm_M, F.Cu at (118.3, 61.8)
- added J9: Conn_01x05, shim:Conn_70AAJ-M_SIB_1x05_P2.54mm_M, F.Cu at (139.8, 111.7)
- moved ? 50.0 mm to (100.0, 151.6)
- moved ? 50.0 mm to (100.0, 50.0)
- moved ? 50.0 mm to (166.0, 50.0)
- moved ? 50.0 mm to (298.0, 100.8)
- moved ? 50.0 mm to (298.0, 50.0)
- moved ? 50.0 mm to (298.0, 151.6)
- moved ? 50.0 mm to (232.0, 50.0)
- moved ? 50.0 mm to (364.0, 151.6)
- moved ? 50.0 mm to (364.0, 50.0)
- moved ? 50.0 mm to (166.0, 100.8)
- moved ? 50.0 mm to (232.0, 151.6)
- moved ? 50.0 mm to (166.0, 151.6)

Commit message: Basic interposer layout done. Borders and choice of which standoffs to use still in the works.
Parts:
- removed J16, J24, J32, J40, J48, J56, J64, J8: Conn_01x02, shim:Conn_70AAJ-M_SIB_1x02_P2.54mm_M
- moved J76 18.4 mm to (79.7, 44.5), turned to 90 degrees
- moved J19 17.5 mm to (184.4, 61.8), turned to 90 degrees
- moved J3 16.8 mm to (118.5, 61.8), turned to 90 degrees
- moved J11 15.3 mm to (147.7, 61.8), turned to 90 degrees
- moved J27 14.5 mm to (213.7, 61.8), turned to 90 degrees
- moved J51 13.1 mm to (316.4, 61.8), turned to 90 degrees
- moved J35 12.6 mm to (250.4, 61.8), turned to 90 degrees
- moved J43 12.3 mm to (279.7, 61.8), turned to 90 degrees
- moved J59 12.2 mm to (345.7, 61.8), turned to 90 degrees
- moved J75 8.96 mm to (79.7, 49.5), turned to 90 degrees
- moved J73 5.80 mm to (363.5, 93.5)
- moved J58 5.62 mm to (351.9, 108.1)
- moved J57 5.62 mm to (339.1, 108.1)
- moved J71 5.50 mm to (231.8, 93.5)
- moved J22 5.25 mm to (177.9, 93.5)
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Routing:
- net /Channel 8/CS+: track 0.00 -> 19.7 mm, vias 0 -> 1
- net /Channel 7/CS+: track 0.00 -> 19.7 mm, vias 0 -> 1
- net /Channel 6/CS+: track 0.00 -> 19.7 mm, vias 0 -> 1
- net /Channel 1/CS+: track 0.00 -> 19.7 mm, vias 0 -> 1
- net /Channel 4/CS+: track 0.00 -> 19.7 mm, vias 0 -> 1
- net /Channel 3/CS+: track 0.00 -> 19.7 mm, vias 0 -> 1
- net /Channel 2/CS+: track 0.00 -> 19.7 mm, vias 0 -> 1
- net /Channel 5/CS+: track 0.00 -> 19.7 mm, vias 0 -> 1
- net /Channel 8/CS-: track 0.00 -> 19.1 mm, vias 0 -> 2
- net /Channel 7/CS-: track 0.00 -> 19.1 mm, vias 0 -> 2
- net /Channel 6/CS-: track 0.00 -> 19.1 mm, vias 0 -> 2
- net /Channel 5/CS-: track 0.00 -> 19.1 mm, vias 0 -> 2
- net /Channel 4/CS-: track 0.00 -> 19.1 mm, vias 0 -> 2
- net /Channel 3/CS-: track 0.00 -> 19.1 mm, vias 0 -> 2
- net /Channel 2/CS-: track 0.00 -> 19.1 mm, vias 0 -> 2
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