File: pcbs/amp_interposer/channel.kicad_sch (KiCad schematic)
At the start: 8 parts, among them J1 Conn_01x05, J2 Conn_01x05, J3 Conn_01x02, J4 Conn_02x10_Odd_Even, J5 Conn_02x02, J6 Conn_01x05, J7 Conn_01x05, J8 Conn_01x02

Commit message: Basic interposer layout done. Borders and choice of which standoffs to use still in the works.
Parts:
- removed J8: Conn_01x02, shim:Conn_70AAJ-M_SIB_1x02_P2.54mm_M, symbol Connector_Generic:Conn_01x02
Changed lines of the file:
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@@
-	)
-	(symbol
-		(lib_id "Connector_Generic:Conn_01x02")
-		(at 170.18 100.33 0)
-		(unit 1)
-		(body_style 1)
-		(exclude_from_sim no)
-		(in_bom yes)
-		(on_board yes)
-		(in_pos_files yes)
-		(dnp no)
-		(fields_autoplaced yes)
-		(property "Reference" "J8"
-			(at 172.72 100.3299 0)
-			(show_name no)
-			(do_not_autoplace no)
-			(effects
-				(font
-					(size 1.27 1.27)
-				)
-				(justify left)
-			)
-		)
-		(property "Value" "Conn_01x02"
-			(at 172.72 102.8699 0)
-			(show_name no)
-			(do_not_autoplace no)
-			(effects
-				(font
-					(size 1.27 1.27)
-				)
-				(justify left)
-			)
-		)
-		(property "Footprint" "shim:Conn_70AAJ-M_SIB_1x02_P2.54mm_M"
-			(at 170.18 100.33 0)
-			(hide yes)
-			(show_name no)
-			(do_not_autoplace no)
-			(effects
-				(font
-					(size 1.27 1.27)
-				)
-			)
-		)
-		(property "Datasheet" ""
-			(at 170.18 100.33 0)
-			(hide yes)
-			(show_name no)
-			(do_not_autoplace no)
-			(effects
-				(font
-					(size 1.27 1.27)
-				)
-			)
-		)
-		(property "Description" "Generic connector, single row, 01x02, script generated (kicad-library-utils/schlib/autogen/connector/)"
-			(at 170.18 100.33 0)
-			(hide yes)
-			(show_name no)
-			(do_not_autoplace no)
-			(effects
-				(font
-					(size 1.27 1.27)
-				)
-			)
-		)
-		(pin "2"
-		)
-		(pin "1"
-		)
-		(instances
-			(project "amp_interposer"
-				(path "/c8d23550-b570-431c-9f87-c6e7cc90483a/0bfd2173-f5c7-49cd-b60a-2864e281386d"
-					(reference "J24")
-					(unit 1)
-				)
-				(path "/c8d23550-b570-431c-9f87-c6e7cc90483a/4756725f-58fd-4b41-93fc-102ddf024bc9"
-					(reference "J48")
-					(unit 1)
-				)
-				(path "/c8d23550-b570-431c-9f87-c6e7cc90483a/62447b76-7766-4b2e-b543-26ff21a21d57"
-					(reference "J16")
-					(unit 1)
-				)
-				(path "/c8d23550-b570-431c-9f87-c6e7cc90483a/915bfc09-a406-47c2-9a64-29bf999fff3f"
-					(reference "J56")
-					(unit 1)
-				)
-				(path "/c8d23550-b570-431c-9f87-c6e7cc90483a/bb950187-f54c-441b-b347-5a24deeee557"
-					(reference "J64")
-					(unit 1)
-				)
-				(path "/c8d23550-b570-431c-9f87-c6e7cc90483a/d51dbd77-c715-42c2-8f6b-d98e8015d3ba"
-					(reference "J32")
-					(unit 1)
-				)
-				(path "/c8d23550-b570-431c-9f87-c6e7cc90483a/db111a79-ed75-4a66-80e6-0ca737d8c1cc"
-					(reference "J8")
-					(unit 1)
-				)
-				(path "/c8d23550-b570-431c-9f87-c6e7cc90483a/fc93d66d-ac25-4cdf-a540-3c2d6e3f7a6f"
-					(reference "J40")
-					(unit 1)
-				)
-			)
-		)
 	)
 	(symbol
